File: hardware/readout_slice/connectivity.sch (KiCad schematic (older format))
At the start: 11 parts

Commit message: working on readount_slice
Parts:
- added J?: Serial USB, symbol Connector_Generic:Conn_01x04
- added J? (x2): Mounting, symbol Connector_Generic:Conn_01x09
Connections:
- net labels added: SD_io_CD#, SD_io_D0, SD_io_D1, SD_io_D2, SD_io_D3, SD_io_clk, SD_io_cmd, uart_rx, uart_tx
- wire segments 65 -> 84
- no-connect marks 10 -> 28
Other:
- note added: "To sparkfun FT232RL"
- note added: "from\nglobal"
- moved on the sheet: J?, U?C
Changed lines of the file:
@@
 Wire Wire Line
 	7650 3350 7600 3350
-Text Label 7600 3350 2    50   ~ 0
+Text Label 7600 3350 2    50   ~ 10
 VCC_CFG_MIO_B13
 Text Notes 7100 4000 2    50   ~ 10
@@
 	8150 3800 7750 3800
 Wire Wire Line
-	4700 6350 3650 6350
-Wire Wire Line
-	3650 6450 4700 6450
-Wire Wire Line
-	3650 6550 4700 6550
-Wire Wire Line
-	3650 6650 4700 6650
-Wire Wire Line
-	3650 6850 4700 6850
-Wire Wire Line
-	3650 7050 4700 7050
-Text Notes 4550 6350 2    50   ~ 0
+	5200 6250 4150 6250
+Wire Wire Line
+	4150 6350 5200 6350
+Wire Wire Line
+	4150 6450 5200 6450
+Wire Wire Line
+	4150 6550 5200 6550
+Wire Wire Line
+	4150 6750 5200 6750
+Wire Wire Line
+	4150 6950 5200 6950
+Text Notes 4450 5950 2    50   ~ 0
 MIO 40-45 to SD Card
-Text Notes 3300 5900 0    50   ~ 10
+Text Notes 3550 5750 0    50   ~ 10
 MIo 1-6, 8 for QSPI flash??\n
 $Comp
 L Connector:SD_Card J?
 U 1 1 608C0AD2
-P 1800 6650
+P 1850 6300
 AR Path="/608C0AD2" Ref="J?"  Part="1"
 AR Path="/608B2FC0/608C0AD2" Ref="J?"  Part="1"
-F 0 "J?" H 1800 5985 50  0000 C CNN
-F 1 "SD_Card" H 1800 6076 50  0000 C CNN
-F 2 "" H 1800 6650 50  0001 C CNN
-F 3 "http://portal.fciconnect.com/Comergent//fci/drawing/10067847.pdf" H 1800 6650 50  0001 C CNN
-	1    1800 6650
+F 0 "J?" H 1850 5635 50  0000 C CNN
+F 1 "SD_Card" H 1850 5726 50  0000 C CNN
+F 2 "" H 1850 6300 50  0001 C CNN
+F 3 "http://portal.fciconnect.com/Comergent//fci/drawing/10067847.pdf" H 1850 6300 50  0001 C CNN
+	1    1850 6300
 	-1   0    0    1
 $EndComp
 Wire Wire Line
-	2700 6450 2800 6450
-Wire Wire Line
-	2800 6450 2800 6750
-Wire Wire Line
-	2700 6750 2800 6750
-Connection ~ 2800 6750
-Wire Wire Line
-	2800 6750 2800 7200
+	2750 6100 2850 6100
+Wire Wire Line
+	2850 6100 2850 6400
+Wire Wire Line
+	2750 6400 2850 6400
+Connection ~ 2850 6400
+Wire Wire Line
+	2850 6400 2850 6850
 $Comp
 L power:GNDD #PWR?
 U 1 1 608C0ADD
-P 2800 7200
+P 2850 6850
 AR Path="/608C0ADD" Ref="#PWR?"  Part="1"
 AR Path="/608B2FC0/608C0ADD" Ref="#PWR?"  Part="1"
-F 0 "#PWR?" H 2800 6950 50  0001 C CNN
-F 1 "GNDD" H 2804 7045 50  0000 C CNN
-F 2 "" H 2800 7200 50  0001 C CNN
-F 3 "" H 2800 7200 50  0001 C CNN
-	1    2800 7200
-	1    0    0    -1
-$EndComp
-Wire Wire Line
-	2700 6650 2750 6650
-Wire Wire Line
-	2750 6650 2750 6050
+F 0 "#PWR?" H 2850 6600 50  0001 C CNN
+F 1 "GNDD" H 2854 6695 50  0000 C CNN
+F 2 "" H 2850 6850 50  0001 C CNN
+F 3 "" H 2850 6850 50  0001 C CNN
+	1    2850 6850
+	1    0    0    -1
+$EndComp
+Wire Wire Line
+	2750 6300 2800 6300
+Wire Wire Line
+	2800 6300 2800 5700
 $Comp
 L power:+3V3 #PWR?
 U 1 1 608C0AE5
-P 2750 6050
+P 2800 5700
 AR Path="/608C0AE5" Ref="#PWR?"  Part="1"
 AR Path="/608B2FC0/608C0AE5" Ref="#PWR?"  Part="1"
-F 0 "#PWR?" H 2750 5900 50  0001 C CNN
-F 1 "+3V3" H 2750 6200 50  0000 C CNN
-F 2 "" H 2750 6050 50  0001 C CNN
-F 3 "" H 2750 6050 50  0001 C CNN
-	1    2750 6050
-	1    0    0    -1
-$EndComp
-Text Notes 2550 6000 0    50   ~ 10
+F 0 "#PWR?" H 2800 5550 50  0001 C CNN
+F 1 "+3V3" H 2800 5850 50  0000 C CNN
+F 2 "" H 2800 5700 50  0001 C CNN
+F 3 "" H 2800 5700 50  0001 C CNN
+	1    2800 5700
+	1    0    0    -1
+$EndComp
+Text Notes 2600 5650 0    50   ~ 10
 caps?
 $Comp
 L readout:Mars_ZX2 U?
 U 3 1 608C0AEC
-P 5200 6200
+P 5700 6100
 AR Path="/608C0AEC" Ref="U?"  Part="3"
 AR Path="/608B2FC0/608C0AEC" Ref="U?"  Part="3"
-F 0 "U?" H 5037 6365 50  0000 C CNN
-F 1 "Mars_ZX2" H 5037 6274 50  0000 C CNN
-F 2 "" H 5250 6550 50  0001 C CNN
-F 3 "" H 5250 6550 50  0001 C CNN
-	3    5200 6200
+F 0 "U?" H 5537 6265 50  0000 C CNN
+F 1 "Mars_ZX2" H 5537 6174 50  0000 C CNN
+F 2 "" H 5750 6450 50  0001 C CNN
+F 3 "" H 5750 6450 50  0001 C CNN
+	3    5700 6100
 	-1   0    0    -1
 $EndComp
@@
 Text Notes 5450 3500 0    50   ~ 10
 +/- 5%\n
+Wire Wire Line
+	5200 7150 4850 7150
+Wire Wire Line
+	5200 7350 4850 7350
+Text Label 4850 7150 0    50   ~ 10
+uart_rx
+Text Label 4850 7350 0    50   ~ 10
+uart_tx
+$Comp
+L Connector_Generic:Conn_01x04 J?
+U 1 1 604E9FF6
+P 9550 5900
+F 0 "J?" H 9468 6217 50  0000 C CNN
+F 1 "Serial USB" H 9468 6126 50  0000 C CNN
+F 2 "" H 9550 5900 50  0001 C CNN
+F 3 "~" H 9550 5900 50  0001 C CNN
+	1    9550 5900
+	-1   0    0    -1
+$EndComp
+Wire Wire Line
+	9750 5900 10000 5900
+Wire Wire Line
+	9750 6000 10000 6000
+Text Label 10000 6000 2    50   ~ 10
+uart_rx
+Text Label 10000 5900 2    50   ~ 10
+uart_tx
+$Comp
+L power:GNDD #PWR?
+U 1 1 604F6F5D
+P 10000 6200
+AR Path="/604F6F5D" Ref="#PWR?"  Part="1"
+AR Path="/608B2FC0/604F6F5D" Ref="#PWR?"  Part="1"
+F 0 "#PWR?" H 10000 5950 50  0001 C CNN
+F 1 "GNDD" H 10000 6050 50  0000 C CNN
+F 2 "" H 10000 6200 50  0001 C CNN
+F 3 "" H 10000 6200 50  0001 C CNN
+	1    10000 6200
+	1    0    0    -1
+$EndComp
+Wire Wire Line
+	10000 6200 10000 6100
+Wire Wire Line
+	10000 6100 9750 6100
+Wire Wire Line
+	9750 5800 10000 5800
+Wire Wire Line
+	10000 5800 10000 5700
+$Comp
+L power:+3V3 #PWR?
+U 1 1 604FBF11
+P 10000 5700
+AR Path="/604FBF11" Ref="#PWR?"  Part="1"
+AR Path="/608B2FC0/604FBF11" Ref="#PWR?"  Part="1"
+F 0 "#PWR?" H 10000 5550 50  0001 C CNN
+F 1 "+3V3" H 10000 5850 50  0000 C CNN
+F 2 "" H 10000 5700 50  0001 C CNN
+F 3 "" H 10000 5700 50  0001 C CNN
+	1    10000 5700
+	1    0    0    -1
+$EndComp
+Text Notes 9300 5150 0    118  ~ 24
+To sparkfun FT232RL
+$Comp
+L Connector_Generic:Conn_01x09 J?
+U 1 1 605012A1
+P 10850 5950
+F 0 "J?" H 10768 5325 50  0000 C CNN
+F 1 "Mounting" H 10768 5416 50  0000 C CNN
+F 2 "" H 10850 5950 50  0001 C CNN
+F 3 "~" H 10850 5950 50  0001 C CNN
+	1    10850 5950
+	-1   0    0    1
+$EndComp
+Text Label 6650 5900 0    50   ~ 10
+VCC_CFG_MIO_B13
+Wire Wire Line
+	6650 5900 6650 6050
+Wire Wire Line
+	6650 6050 6550 6050
+Wire Wire Line
+	6550 6050 6550 6100
+Connection ~ 6650 6050
+Wire Wire Line
+	6650 6050 6650 6100
+Text Label 4150 6250 0    50   ~ 10
+SD_io_clk
+Text Label 4150 6350 0    50   ~ 10
+SD_io_cmd
+Text Label 4150 6450 0    50   ~ 10
+SD_io_D0
+Text Label 4150 6550 0    50   ~ 10
+SD_io_D1
+Text Label 4150 6750 0    50   ~ 10
+SD_io_D2
+Text Label 4150 6950 0    50   ~ 10
+SD_io_D3
+Text Label 500  6500 0    50   ~ 10
+SD_io_CD#
+Text Label 3300 6700 2    50   ~ 10
+SD_io_D2
+Wire Wire Line
+	3300 6700 2750 6700
+Text Label 3300 6600 2    50   ~ 10
+SD_io_D3
+Wire Wire Line
+	3300 6600 2750 6600
+Text Label 3300 6500 2    50   ~ 10
+SD_io_cmd
+Wire Wire Line
+	3300 6500 2750 6500
+Text Label 3300 6200 2    50   ~ 10
+SD_io_clk
+Wire Wire Line
+	3300 6200 2750 6200
+Text Label 3300 6000 2    50   ~ 10
+SD_io_D0
+Wire Wire Line
+	3300 6000 2750 6000
+Text Label 3300 5900 2    50   ~ 10
+SD_io_D1
+Wire Wire Line
+	3300 5900 2750 5900
+Wire Wire Line
+	500  6500 950  6500
+Text Notes 550  6400 0    50   ~ 10
+from\nglobal
+NoConn ~ 11050 6350
+NoConn ~ 11050 6250
+NoConn ~ 11050 6150
+NoConn ~ 11050 6050
+NoConn ~ 11050 5950
+NoConn ~ 11050 5850
+NoConn ~ 11050 5750
+NoConn ~ 11050 5650
+NoConn ~ 11050 5550
+NoConn ~ 10550 5550
+NoConn ~ 10550 5650
+NoConn ~ 10550 5750
+NoConn ~ 10550 5850
+NoConn ~ 10550 5950
+NoConn ~ 10550 6050
+NoConn ~ 10550 6150
+NoConn ~ 10550 6250
+NoConn ~ 10550 6350
+$Comp
+L Connector_Generic:Conn_01x09 J?
+U 1 1 60502B7C
+P 10350 5950
+F 0 "J?" H 10268 5325 50  0000 C CNN
+F 1 "Mounting" H 10268 5416 50  0000 C CNN
+F 2 "" H 10350 5950 50  0001 C CNN
+F 3 "~" H 10350 5950 50  0001 C CNN
+	1    10350 5950
+	-1   0    0    1
+$EndComp
 $EndSCHEMATC

Commit message: more work on readout_slice
Parts:
- removed R?: 20k, symbol Device:R
- added C?: .1u, symbol Device:C_Small
- R?: Precision (none) -> 5%
Connections:
- net +3V3: now also C?.1
- net GNDD: now also C?.2
- net JTAG_TCK: no longer J?.6 (Pin_6)
- net PS_SRST: now reaches J?.14 (Pin_14)
- net SD_io_CD# renamed SD_id_CD#
- no-connect marks 28 -> 26
Other:
- note added: "ESD diode chip here\nref antmicro"
- note added: "Maybe need level shifter here?"
- note added: "Not sure?"
- note removed: "+/- 5%\n"
- note removed: "from\nglobal"
- moved on the sheet: J?, R?, U?

Commit message: working more on readout_slice schematic
Parts:
- removed R?: 1K, symbol Device:R
- removed R?: 3k3, symbol Device:R
- removed R?: 4k7, symbol Device:R
- removed U?: S25FL52, Package_SO:SOIC-16_4.55x10.3mm_P1.27mm, symbol readout:S25FL52
- removed U?: USB3320-EZK, Package_DFN_QFN:QFN-32-1EP_5x5mm_P0.5mm_EP3.45x3.45mm, symbol readout:USB3320-EZK
- added C?: 47u, symbol Device:C_Small
- added D?: GREEN, symbol Device:LED
- added J?: Digilent JTAG header, readout_slice:87832-1420, symbol Connector_Generic:Conn_02x07_Odd_Even
- added R?: 100, symbol Device:R
- added R?: 330, symbol Device:R
- added R? (x2): 4.7k, symbol Device:R
- added U?: XC7A35T-1FGG484, symbol readout:XC7A35T-1FGG484
Connections:
- net GNDD: now also C?.2, D?.1 (K), J?.1 (Pin_1), J?.11 (Pin_11), J?.13 (Pin_13), J?.3 (Pin_3), J?.5 (Pin_5), J?.7 (Pin_7), J?.9 (Pin_9), U?.E12 (VCCBATT_0), U?.K9 (GNDADC_0), U?.U10 (M1_0), U?.U9 (M2_0)
- net JTAG_TCK: now also J?.6 (Pin_6)
- net at U?.194 (FPGA_DONE): now also R?.1
- new net: D?.2 (A), R?.2
- new net: R?.2, U?.G11 (DONE_0)
- new net: R?.2, U?.N12 (PROGRAM_B_0)
- new net: J?.10 (Pin_10), U?.R13 (TDI_0)
- new net: J?.4 (Pin_4), U?.T13 (TMS_0)
- new net: R?.1, U?.U12 (INIT_B_0)
- new net: J?.8 (Pin_8), U?.U13 (TDO_0)
- new net: J?.6 (Pin_6), U?.V12 (TCK_0)
- new net Vcc_0: C?.1, R?.1, R?.1, R?.2, U?.F12 (VCCO_0), U?.T12 (VCCO_0), U?.U11 (M0_0)
- no-connect marks 26 -> 21
Other:
- note added: "Need to create this"
- note added: "Vref here"
- note added: "and pullups?\n"
- note added: "goes global?"
- note removed: "CAPS?"
- note removed: "VCC_CFG_MIO_B13 needs to be global"
- note removed: "check package on this\n"
- note removed: "to FLASH_IO2"
- note removed: "to FLASH_IO3"
- note removed: "to PS_POR#"
- moved on the sheet: C?, J?, U?B

Commit message: auto push run at Mon Mar 15 12:11:48 EDT 2021
Other:
- moved on the sheet: J?, U?C
Changed lines of the file:
@@
 $Descr A4 11693 8268
 encoding utf-8
-Sheet 3 4
+Sheet 3 5
 Title ""
 Date ""
@@
 	8000 2200 7600 2200
 Wire Wire Line
-	5200 6250 4700 6250
-Wire Wire Line
-	4700 6350 5200 6350
-Wire Wire Line
-	4700 6450 5200 6450
-Wire Wire Line
-	4700 6550 5200 6550
-Wire Wire Line
-	4700 6750 5200 6750
-Wire Wire Line
-	4700 6950 5200 6950
-Text Notes 4450 5950 2    50   ~ 0
+	4900 6450 4400 6450
+Wire Wire Line
+	4400 6550 4900 6550
+Wire Wire Line
+	4400 6650 4900 6650
+Wire Wire Line
+	4400 6750 4900 6750
+Wire Wire Line
+	4400 6950 4900 6950
+Wire Wire Line
+	4400 7150 4900 7150
+Text Notes 4150 6150 2    50   ~ 0
 MIO 40-45 to SD Card
-Text Notes 3550 5750 0    50   ~ 10
+Text Notes 3250 5950 0    50   ~ 10
 MIo 1-6, 8 for QSPI flash??\n
 $Comp
 L Connector:SD_Card J?
 U 1 1 608C0AD2
-P 2400 6750
+P 2100 6950
 AR Path="/608C0AD2" Ref="J?"  Part="1"
 AR Path="/608B2FC0/608C0AD2" Ref="J?"  Part="1"
-F 0 "J?" H 2400 6085 50  0000 C CNN
-F 1 "SD_Card" H 2400 6176 50  0000 C CNN
-F 2 "" H 2400 6750 50  0001 C CNN
-F 3 "http://portal.fciconnect.com/Comergent//fci/drawing/10067847.pdf" H 2400 6750 50  0001 C CNN
-	1    2400 6750
+F 0 "J?" H 2100 6285 50  0000 C CNN
+F 1 "SD_Card" H 2100 6376 50  0000 C CNN
+F 2 "" H 2100 6950 50  0001 C CNN
+F 3 "http://portal.fciconnect.com/Comergent//fci/drawing/10067847.pdf" H 2100 6950 50  0001 C CNN
+	1    2100 6950
 	-1   0    0    1
 $EndComp
 Wire Wire Line
-	3300 6550 3400 6550
-Wire Wire Line
-	3400 6550 3400 6850
-Wire Wire Line
-	3300 6850 3400 6850
-Connection ~ 3400 6850
-Wire Wire Line
-	3400 6850 3400 7300
+	3000 6750 3100 6750
+Wire Wire Line
+	3100 6750 3100 7050
+Wire Wire Line
+	3000 7050 3100 7050
+Connection ~ 3100 7050
+Wire Wire Line
+	3100 7050 3100 7500
 $Comp
 L power:GNDD #PWR?
 U 1 1 608C0ADD
-P 3400 7300
+P 3100 7500
 AR Path="/608C0ADD" Ref="#PWR?"  Part="1"
 AR Path="/608B2FC0/608C0ADD" Ref="#PWR?"  Part="1"
-F 0 "#PWR?" H 3400 7050 50  0001 C CNN
-F 1 "GNDD" H 3404 7145 50  0000 C CNN
-F 2 "" H 3400 7300 50  0001 C CNN
-F 3 "" H 3400 7300 50  0001 C CNN
-	1    3400 7300
-	1    0    0    -1
-$EndComp
-Wire Wire Line
-	3300 6750 3350 6750
-Wire Wire Line
-	3350 6750 3350 6150
+F 0 "#PWR?" H 3100 7250 50  0001 C CNN
+F 1 "GNDD" H 3104 7345 50  0000 C CNN
+F 2 "" H 3100 7500 50  0001 C CNN
+F 3 "" H 3100 7500 50  0001 C CNN
+	1    3100 7500
+	1    0    0    -1
+$EndComp
+Wire Wire Line
+	3000 6950 3050 6950
+Wire Wire Line
+	3050 6950 3050 6350
 $Comp
 L power:+3V3 #PWR?
 U 1 1 608C0AE5
-P 3350 6150
+P 3050 6350
 AR Path="/608C0AE5" Ref="#PWR?"  Part="1"
 AR Path="/608B2FC0/608C0AE5" Ref="#PWR?"  Part="1"
-F 0 "#PWR?" H 3350 6000 50  0001 C CNN
-F 1 "+3V3" H 3350 6300 50  0000 C CNN
-F 2 "" H 3350 6150 50  0001 C CNN
-F 3 "" H 3350 6150 50  0001 C CNN
-	1    3350 6150
-	1    0    0    -1
-$EndComp
-Text Notes 3150 6100 0    50   ~ 10
+F 0 "#PWR?" H 3050 6200 50  0001 C CNN
+F 1 "+3V3" H 3050 6500 50  0000 C CNN
+F 2 "" H 3050 6350 50  0001 C CNN
+F 3 "" H 3050 6350 50  0001 C CNN
+	1    3050 6350
+	1    0    0    -1
+$EndComp
+Text Notes 2850 6300 0    50   ~ 10
 caps?
 $Comp
 L readout:Mars_ZX2 U?
 U 3 1 608C0AEC
-P 5700 6100
+P 5400 6300
 AR Path="/608C0AEC" Ref="U?"  Part="3"
 AR Path="/608B2FC0/608C0AEC" Ref="U?"  Part="3"
-F 0 "U?" H 5700 6200 50  0000 C CNN
-F 1 "Mars_ZX2" H 5700 6100 50  0000 C CNN
-F 2 "" H 5750 6450 50  0001 C CNN
-F 3 "" H 5750 6450 50  0001 C CNN
-	3    5700 6100
+F 0 "U?" H 5400 6400 50  0000 C CNN
+F 1 "Mars_ZX2" H 5400 6300 50  0000 C CNN
+F 2 "" H 5450 6650 50  0001 C CNN
+F 3 "" H 5450 6650 50  0001 C CNN
+	3    5400 6300
 	-1   0    0    -1
 $EndComp
@@
 $EndComp
 Wire Wire Line
-	5200 7150 4850 7150
-Wire Wire Line
-	5200 7350 4850 7350
-Text Label 4850 7150 0    50   ~ 10
+	4900 7350 4550 7350
+Wire Wire Line
+	4900 7550 4550 7550
+Text Label 4550 7350 0    50   ~ 10
 uart_rx
-Text Label 4850 7350 0    50   ~ 10
+Text Label 4550 7550 0    50   ~ 10
 uart_tx
 $Comp
@@
 	-1   0    0    1
 $EndComp
-Text Label 6650 5900 0    50   ~ 10
+Text Label 6350 6100 0    50   ~ 10
 VCC_CFG_MIO_B13
 Wire Wire Line
-	6650 5900 6650 6050
-Wire Wire Line
-	6650 6050 6550 6050
-Wire Wire Line
-	6550 6050 6550 6100
-Connection ~ 6650 6050
-Wire Wire Line
-	6650 6050 6650 6100
-Text Label 4700 6250 0    50   ~ 10
+	6350 6100 6350 6250
+Wire Wire Line
+	6350 6250 6250 6250
+Wire Wire Line
+	6250 6250 6250 6300
+Connection ~ 6350 6250
+Wire Wire Line
+	6350 6250 6350 6300
+Text Label 4400 6450 0    50   ~ 10
 SD_io_clk
-Text Label 4700 6350 0    50   ~ 10
+Text Label 4400 6550 0    50   ~ 10
 SD_io_cmd
-Text Label 4700 6450 0    50   ~ 10
+Text Label 4400 6650 0    50   ~ 10
 SD_io_D0
-Text Label 4700 6550 0    50   ~ 10
+Text Label 4400 6750 0    50   ~ 10
 SD_io_D1
-Text Label 4700 6750 0    50   ~ 10
+Text Label 4400 6950 0    50   ~ 10
 SD_io_D2
-Text Label 4700 6950 0    50   ~ 10
+Text Label 4400 7150 0    50   ~ 10
 SD_io_D3
-Text Label 3850 7150 2    50   ~ 10
+Text Label 3550 7350 2    50   ~ 10
 SD_io_D2
 Wire Wire Line
-	3850 7150 3300 7150
-Text Label 3850 7050 2    50   ~ 10
+	3550 7350 3000 7350
+Text Label 3550 7250 2    50   ~ 10
 SD_io_D3
 Wire Wire Line
-	3850 7050 3300 7050
-Text Label 3850 6950 2    50   ~ 10
+	3550 7250 3000 7250
+Text Label 3550 7150 2    50   ~ 10
 SD_io_cmd
 Wire Wire Line
-	3850 6950 3300 6950
-Text Label 3850 6650 2    50   ~ 10
+	3550 7150 3000 7150
+Text Label 3550 6850 2    50   ~ 10
 SD_io_clk
 Wire Wire Line
-	3850 6650 3300 6650
-Text Label 3850 6450 2    50   ~ 10
+	3550 6850 3000 6850
+Text Label 3550 6650 2    50   ~ 10
 SD_io_D0
 Wire Wire Line
-	3850 6450 3300 6450
-Text Label 3850 6350 2    50   ~ 10
+	3550 6650 3000 6650
+Text Label 3550 6550 2    50   ~ 10
 SD_io_D1
 Wire Wire Line
-	3850 6350 3300 6350
-Wire Wire Line
-	1300 6950 1500 6950
+	3550 6550 3000 6550
+Wire Wire Line
+	1000 7150 1200 7150
 NoConn ~ 11050 6350
 NoConn ~ 11050 6250
@@
 Text HLabel 6550 2600 2    50   Input ~ 0
 PS_SRST
-Text HLabel 1300 6950 0    50   Input ~ 10
+Text HLabel 1000 7150 0    50   Input ~ 10
 SD_id_CD#
-Text Notes 3350 6800 0    79   ~ 16
+Text Notes 3050 7000 0    79   ~ 16
 Maybe need level shifter here?
 $Comp
@@
 Text HLabel 4000 2350 2    50   Input ~ 10
 Vcc_0
-Text Notes 4000 6450 0    50   ~ 10
+Text Notes 3700 6650 0    50   ~ 10
 and pullups?\n
 $EndSCHEMATC
