File: hardware/readout_slice/Citiroc3V3.sch (KiCad schematic (older format))
At the start: 0 parts

Commit message: more progress on readout_slice
Parts:
- added C?: 47u, symbol Device:C_Small
- added C? (x2): 4.7u, symbol Device:C_Small
- added C? (x4): .47u, symbol Device:C_Small
- added U?: XC7A35T-1FGG484, symbol readout:XC7A35T-1FGG484
Changed lines of the file:
@@
 Comment4 ""
 $EndDescr
+$Comp
+L readout:XC7A35T-1FGG484 U?
+U 6 1 60742FAE
+P 7200 2050
+F 0 "U?" H 7075 -1723 50  0000 C CNN
+F 1 "XC7A35T-1FGG484" H 7075 -1814 50  0000 C CNN
+F 2 "" H 6100 2200 50  0001 C CNN
+F 3 "" H 6100 2200 50  0001 C CNN
+	6    7200 2050
+	1    0    0    -1
+$EndComp
+$Comp
+L Device:C_Small C?
+U 1 1 60742FB4
+P 3950 3600
+F 0 "C?" H 3858 3646 50  0000 R CNN
+F 1 "47u" H 3858 3555 50  0000 R CNB
+F 2 "" H 3950 3600 50  0001 C CNN
+F 3 "~" H 3950 3600 50  0001 C CNN
+	1    3950 3600
+	1    0    0    -1
+$EndComp
+$Comp
+L Device:C_Small C?
+U 1 1 60742FBA
+P 3950 3300
+F 0 "C?" H 4042 3346 50  0000 L CNN
+F 1 "4.7u" H 4042 3255 50  0000 L CNB
+F 2 "" H 3950 3300 50  0001 C CNN
+F 3 "~" H 3950 3300 50  0001 C CNN
+	1    3950 3300
+	1    0    0    -1
+$EndComp
+$Comp
+L Device:C_Small C?
+U 1 1 60742FC0
+P 3600 3300
+F 0 "C?" H 3692 3346 50  0000 L CNN
+F 1 "4.7u" H 3692 3255 50  0000 L CNB
+F 2 "" H 3600 3300 50  0001 C CNN
+F 3 "~" H 3600 3300 50  0001 C CNN
+	1    3600 3300
+	1    0    0    -1
+$EndComp
+$Comp
+L Device:C_Small C?
+U 1 1 60742FC6
+P 3250 2950
+F 0 "C?" H 3342 2996 50  0000 L CNN
+F 1 ".47u" H 3342 2905 50  0000 L CNB
+F 2 "" H 3250 2950 50  0001 C CNN
+F 3 "~" H 3250 2950 50  0001 C CNN
+	1    3250 2950
+	1    0    0    -1
+$EndComp
+$Comp
+L Device:C_Small C?
+U 1 1 60742FCC
+P 3600 2950
+F 0 "C?" H 3692 2996 50  0000 L CNN
+F 1 ".47u" H 3692 2905 50  0000 L CNB
+F 2 "" H 3600 2950 50  0001 C CNN
+F 3 "~" H 3600 2950 50  0001 C CNN
+	1    3600 2950
+	1    0    0    -1
+$EndComp
+$Comp
+L Device:C_Small C?
+U 1 1 60742FD2
+P 3950 2950
+F 0 "C?" H 4042 2996 50  0000 L CNN
+F 1 ".47u" H 4042 2905 50  0000 L CNB
+F 2 "" H 3950 2950 50  0001 C CNN
+F 3 "~" H 3950 2950 50  0001 C CNN
+	1    3950 2950
+	1    0    0    -1
+$EndComp
+$Comp
+L Device:C_Small C?
+U 1 1 60742FD8
+P 4300 2950
+F 0 "C?" H 4392 2996 50  0000 L CNN
+F 1 ".47u" H 4392 2905 50  0000 L CNB
+F 2 "" H 4300 2950 50  0001 C CNN
+F 3 "~" H 4300 2950 50  0001 C CNN
+	1    4300 2950
+	1    0    0    -1
+$EndComp
 $EndSCHEMATC
