File: hardware/readout_slice/ZX2-connectivity.sch (KiCad schematic (older format))
At the start: 11 parts

Commit message: readout_slice is more ordered now
Connections:
- net labels added: SD_io_CD#
- net labels removed: SD_id_CD#
Other:
- moved on the sheet: D?, J?, R?, U?B, U?C

Commit message: added notes to schematics for readout_slice
Other:
- note added: "magjack for eth rj45 connector with transformer modled into it\n"
- note added: "still need some caps\n"
Changed lines of the file:
@@
 Text HLabel 9300 4600 2    50   Input ~ 10
 Vcc_cfg_MIO_B13
+Text Notes 8550 2850 0    157  ~ 31
+magjack for eth rj45 connector with transformer modled into it\n
+Text Notes 8550 3100 0    157  ~ 31
+still need some caps\n
 $EndSCHEMATC

Commit message: working on readout_slice
Parts:
- removed J?: RJ45, symbol Connector:RJ45
- added J?: RJ45_Amphenol_RJMG1BD3B8K1ANR, Connector_RJ:RJ45_Amphenol_RJMG1BD3B8K1ANR, symbol Connector:RJ45_Amphenol_RJMG1BD3B8K1ANR
- added R? (x2): 150, symbol Device:R
Connections:
- net labels added: ETH_LED1, ETH_LED2
- wire segments 72 -> 84
Changed lines of the file:
@@
 $Descr A4 11693 8268
 encoding utf-8
-Sheet 10 10
+Sheet 7 16
 Title ""
 Date ""
@@
 AR Path="/608B2FC0/608B92E4" Ref="J?"  Part="1"
 AR Path="/60AD0200/60B2D848/608B92E4" Ref="J?"  Part="1"
+AR Path="/607155C8/608B92E4" Ref="J?"  Part="1"
 F 0 "J?" H 1000 2800 50  0000 C CNN
 F 1 "Digilent JTAG header" H 1250 2900 50  0000 C CNN
@@
 	1    0    0    -1
 $EndComp
-$Comp
-L Connector:RJ45 J?
-U 1 1 608B92EA
-P 8500 1750
-AR Path="/608B92EA" Ref="J?"  Part="1"
-AR Path="/608B2FC0/608B92EA" Ref="J?"  Part="1"
-AR Path="/60AD0200/60B2D848/608B92EA" Ref="J?"  Part="1"
-F 0 "J?" H 8557 2417 50  0000 C CNN
-F 1 "RJ45" H 8557 2326 50  0000 C CNN
-F 2 "" V 8500 1775 50  0001 C CNN
-F 3 "~" V 8500 1775 50  0001 C CNN
-	1    8500 1750
-	-1   0    0    1
-$EndComp
-Text Notes 7350 2050 0    50   ~ 0
+Text Notes 7800 2000 0    50   ~ 0
 Hmmmm?
 Wire Wire Line
@@
 AR Path="/608B2FC0/608B930D" Ref="#PWR?"  Part="1"
 AR Path="/60AD0200/60B2D848/608B930D" Ref="#PWR?"  Part="1"
+AR Path="/607155C8/608B930D" Ref="#PWR?"  Part="1"
 F 0 "#PWR?" H 1350 2500 50  0001 C CNN
 F 1 "+3V3" H 1350 2800 50  0000 C CNN
@@
 AR Path="/608B2FC0/608B9327" Ref="U?"  Part="2"
 AR Path="/60AD0200/60B2D848/608B9327" Ref="U?"  Part="2"
+AR Path="/607155C8/608B9327" Ref="U?"  Part="2"
 F 0 "U?" H 6575 1475 50  0000 C CNN
 F 1 "Mars_ZX2" H 6575 1384 50  0000 C CNN
@@
 AR Path="/608B2FC0/608C0AD2" Ref="J?"  Part="1"
 AR Path="/60AD0200/60B2D848/608C0AD2" Ref="J?"  Part="1"
+AR Path="/607155C8/608C0AD2" Ref="J?"  Part="1"
 F 0 "J?" H 4900 4635 50  0000 C CNN
 F 1 "SD_Card" H 4900 4726 50  0000 C CNN
@@
 AR Path="/608B2FC0/608C0ADD" Ref="#PWR?"  Part="1"
 AR Path="/60AD0200/60B2D848/608C0ADD" Ref="#PWR?"  Part="1"
+AR Path="/607155C8/608C0ADD" Ref="#PWR?"  Part="1"
 F 0 "#PWR?" H 5900 5600 50  0001 C CNN
 F 1 "GNDD" H 5904 5695 50  0000 C CNN
@@
 AR Path="/608B2FC0/608C0AE5" Ref="#PWR?"  Part="1"
 AR Path="/60AD0200/60B2D848/608C0AE5" Ref="#PWR?"  Part="1"
+AR Path="/607155C8/608C0AE5" Ref="#PWR?"  Part="1"
 F 0 "#PWR?" H 5850 4550 50  0001 C CNN
 F 1 "+3V3" H 5850 4850 50  0000 C CNN
@@
 AR Path="/608B2FC0/608C0AEC" Ref="U?"  Part="3"
 AR Path="/60AD0200/60B2D848/608C0AEC" Ref="U?"  Part="3"
+AR Path="/607155C8/608C0AEC" Ref="U?"  Part="3"
 F 0 "U?" H 8200 4750 50  0000 C CNN
 F 1 "Mars_ZX2" H 8200 4650 50  0000 C CNN
@@
 AR Path="/608B2FC0/608B92F1" Ref="#PWR?"  Part="1"
 AR Path="/60AD0200/60B2D848/608B92F1" Ref="#PWR?"  Part="1"
+AR Path="/607155C8/608B92F1" Ref="#PWR?"  Part="1"
 F 0 "#PWR?" H 700 3450 50  0001 C CNN
 F 1 "GNDD" H 704 3545 50  0000 C CNN
@@
 AR Path="/608B2FC0/604E9FF6" Ref="J?"  Part="1"
 AR Path="/60AD0200/60B2D848/604E9FF6" Ref="J?"  Part="1"
+AR Path="/607155C8/604E9FF6" Ref="J?"  Part="1"
 F 0 "J?" H 1018 1967 50  0000 C CNN
 F 1 "Serial USB" H 1018 1876 50  0000 C CNN
@@
 AR Path="/608B2FC0/604F6F5D" Ref="#PWR?"  Part="1"
 AR Path="/60AD0200/60B2D848/604F6F5D" Ref="#PWR?"  Part="1"
+AR Path="/607155C8/604F6F5D" Ref="#PWR?"  Part="1"
 F 0 "#PWR?" H 1550 1700 50  0001 C CNN
 F 1 "GNDD" H 1550 1800 50  0000 C CNN
@@
 AR Path="/608B2FC0/604FBF11" Ref="#PWR?"  Part="1"
 AR Path="/60AD0200/60B2D848/604FBF11" Ref="#PWR?"  Part="1"
+AR Path="/607155C8/604FBF11" Ref="#PWR?"  Part="1"
 F 0 "#PWR?" H 1550 1300 50  0001 C CNN
 F 1 "+3V3" H 1550 1600 50  0000 C CNN
@@
 AR Path="/608B2FC0/605012A1" Ref="J?"  Part="1"
 AR Path="/60AD0200/60B2D848/605012A1" Ref="J?"  Part="1"
+AR Path="/607155C8/605012A1" Ref="J?"  Part="1"
 F 0 "J?" H 2318 1075 50  0000 C CNN
 F 1 "Mounting" H 2318 1166 50  0000 C CNN
@@
 AR Path="/608B2FC0/60502B7C" Ref="J?"  Part="1"
 AR Path="/60AD0200/60B2D848/60502B7C" Ref="J?"  Part="1"
+AR Path="/607155C8/60502B7C" Ref="J?"  Part="1"
 F 0 "J?" H 1818 1075 50  0000 C CNN
 F 1 "Mounting" H 1818 1166 50  0000 C CNN
@@
 AR Path="/608B2FC0/604EB839" Ref="C?"  Part="1"
 AR Path="/60AD0200/60B2D848/604EB839" Ref="C?"  Part="1"
+AR Path="/607155C8/604EB839" Ref="C?"  Part="1"
 F 0 "C?" V 800 2750 50  0000 C CNN
 F 1 ".1u" V 900 2750 50  0000 C CNN
@@
 AR Path="/608B2FC0/61905C3D" Ref="D?"  Part="1"
 AR Path="/60AD0200/60B2D848/61905C3D" Ref="D?"  Part="1"
+AR Path="/607155C8/61905C3D" Ref="D?"  Part="1"
 F 0 "D?" V 5450 2950 50  0000 C CNN
 F 1 "GREEN" V 5350 2900 50  0000 C CNN
@@
 AR Path="/608B2FC0/61905C43" Ref="R?"  Part="1"
 AR Path="/60AD0200/60B2D848/61905C43" Ref="R?"  Part="1"
+AR Path="/607155C8/61905C43" Ref="R?"  Part="1"
 F 0 "R?" V 5550 2800 50  0000 L CNN
 F 1 "100" V 5650 2800 50  0000 L CNN
@@
 AR Path="/608B2FC0/61919E41" Ref="#PWR?"  Part="1"
 AR Path="/60AD0200/60B2D848/61919E41" Ref="#PWR?"  Part="1"
+AR Path="/607155C8/61919E41" Ref="#PWR?"  Part="1"
 F 0 "#PWR?" H 5400 3000 50  0001 C CNN
 F 1 "GNDD" H 5404 3095 50  0000 C CNN
@@
 Text HLabel 9300 4600 2    50   Input ~ 10
 Vcc_cfg_MIO_B13
-Text Notes 8550 2850 0    157  ~ 31
+Text Notes 4850 150  0    157  ~ 31
 magjack for eth rj45 connector with transformer modled into it\n
-Text Notes 8550 3100 0    157  ~ 31
+Text Notes 7550 450  0    157  ~ 31
 still need some caps\n
+$Comp
+L Connector:RJ45_Amphenol_RJMG1BD3B8K1ANR J?
+U 1 1 60ECCBA3
+P 9650 2000
+F 0 "J?" H 9650 2725 50  0000 C CNN
+F 1 "RJ45_Amphenol_RJMG1BD3B8K1ANR" H 9650 2634 50  0000 C CNN
+F 2 "Connector_RJ:RJ45_Amphenol_RJMG1BD3B8K1ANR" H 9650 2700 50  0001 C CNN
+F 3 "https://cdn.amphenol-icc.com/media/wysiwyg/files/documentation/datasheet/inputoutput/io_rjmag.pdf?__cf_chl_jschl_tk__=54a32f8a488397d94d3ded030830f585ee31ab3b-1616385693-0-AXGuwXvDAGbbe1nf5I-Xde7AJy63eLNl1z_hsh-Rvb99UTV3DGG9YQ5RW2x0FGxxB00lARUWcldbQfdTiBGnIhuPN6p4EacKdRY865A9mrZHu-SkMg_65fA8pQV82VqIluafGpMZ4oSnJULTpptDPmpyXEDzyQ9GRFnnPxp66lVWrUfE9B7R_cKfC9TwB8TaIVgP3TYnNZndjC2XKsqeWDTwuoXJxPD57KykX_7zZq4JiNDiD7RJLHgdYR6XmSaNqsXGuy9V_eWl0AiADh1niMpDoVqdZxgR2GKpTo5Z1xXX6GGm8YWv9Mc-gXZxRsx7X7y_zTS_giemPFgYQjrHiKC1BShuwP5XMrNmYJWiGjdhzN7x5mzbfc-ImI0ese86FNxeNXYYxDX07YqkwTUw2gEbf-nL9AMfjQ6AiglSUR5IUw-48_yeF4G9VzuhAG1ucip3nkM6rlMa4W0_lj9dKr7QmwbqKCm5RoCbsjj942Zl" H 9650 2800 50  0001 C CNN
+F 4 "Digi-Key" H 9650 2000 50  0001 C CNN "Supplier"
+F 5 "RJMG1BD3B8K1ANR-ND" H 9650 2000 50  0001 C CNN "Supplier P/N"
+F 6 "RJMG1BD3B8K1ANR" H 9650 2000 50  0001 C CNN "MFN"
+F 7 "4.16" H 9650 2000 50  0001 C CNN "Item Cost"
+	1    9650 2000
+	1    0    0    -1
+$EndComp
+$Comp
+L power:GNDD #PWR?
+U 1 1 60EE4CD2
+P 9650 2700
+AR Path="/60EE4CD2" Ref="#PWR?"  Part="1"
+AR Path="/608B2FC0/60EE4CD2" Ref="#PWR?"  Part="1"
+AR Path="/60AD0200/60B2D848/60EE4CD2" Ref="#PWR?"  Part="1"
+AR Path="/607155C8/60EE4CD2" Ref="#PWR?"  Part="1"
+F 0 "#PWR?" H 9650 2450 50  0001 C CNN
+F 1 "GNDD" H 9654 2545 50  0000 C CNN
+F 2 "" H 9650 2700 50  0001 C CNN
+F 3 "" H 9650 2700 50  0001 C CNN
+	1    9650 2700
+	1    0    0    -1
+$EndComp
+$Comp
+L Device:R R?
+U 1 1 60EF1438
+P 8650 1200
+F 0 "R?" H 8720 1246 50  0000 L CNN
+F 1 "150" V 8650 1150 50  0000 L CNN
+F 2 "" V 8580 1200 50  0001 C CNN
+F 3 "~" H 8650 1200 50  0001 C CNN
+	1    8650 1200
+	1    0    0    -1
+$EndComp
+$Comp
+L power:+3V3 #PWR?
+U 1 1 60EF373F
+P 8650 950
+AR Path="/60EF373F" Ref="#PWR?"  Part="1"
+AR Path="/608B2FC0/60EF373F" Ref="#PWR?"  Part="1"
+AR Path="/60AD0200/60B2D848/60EF373F" Ref="#PWR?"  Part="1"
+AR Path="/607155C8/60EF373F" Ref="#PWR?"  Part="1"
+F 0 "#PWR?" H 8650 800 50  0001 C CNN
+F 1 "+3V3" H 8650 1100 50  0000 C CNN
+F 2 "" H 8650 950 50  0001 C CNN
+F 3 "" H 8650 950 50  0001 C CNN
+	1    8650 950
+	1    0    0    -1
+$EndComp
+$Comp
+L Device:R R?
+U 1 1 60EF451F
+P 8550 1200
+F 0 "R?" H 8620 1246 50  0000 L CNN
+F 1 "150" V 8550 1150 50  0000 L CNN
+F 2 "" V 8480 1200 50  0001 C CNN
+F 3 "~" H 8550 1200 50  0001 C CNN
+	1    8550 1200
+	-1   0    0    -1
+$EndComp
+Wire Wire Line
+	8550 1050 8550 1000
+Wire Wire Line
+	8550 1000 8650 1000
+Wire Wire Line
+	8650 1000 8650 950
+Wire Wire Line
+	8650 1000 8650 1050
+Connection ~ 8650 1000
+Wire Wire Line
+	8750 2200 8650 2200
+Wire Wire Line
+	8650 2200 8650 1350
+Wire Wire Line
+	8750 2400 8550 2400
+Wire Wire Line
+	8550 2400 8550 1350
+Wire Wire Line
+	7250 1650 7650 1650
+Text Label 7650 1650 2    50   ~ 10
+ETH_LED1
+Text Label 7650 1750 2    50   ~ 10
+ETH_LED2
+Wire Wire Line
+	7650 1750 7250 1750
+Text Label 8150 2300 0    50   ~ 10
+ETH_LED1
+Text Label 8150 2500 0    50   ~ 10
+ETH_LED2
+Wire Wire Line
+	8150 2500 8750 2500
+Wire Wire Line
+	8150 2300 8750 2300
 $EndSCHEMATC

Commit message: more progress on readout_slice
Changed lines of the file:
@@
 Text Notes 4850 150  0    157  ~ 31
 magjack for eth rj45 connector with transformer modled into it\n
-Text Notes 7550 450  0    157  ~ 31
+Text Notes 7550 650  0    157  ~ 31
 still need some caps\n
 $Comp

Commit message: auto push run at Fri Apr  9 14:02:10 EDT 2021
Connections:
- net GNDD: now also J?.13 (SHIELD)
Changed lines of the file:
@@
 $Descr A4 11693 8268
 encoding utf-8
-Sheet 5 16
+Sheet 4 15
 Title ""
 Date ""
@@
 L power:GNDD #PWR?
 U 1 1 60EE4CD2
-P 9650 2700
+P 9650 2800
 AR Path="/60EE4CD2" Ref="#PWR?"  Part="1"
 AR Path="/608B2FC0/60EE4CD2" Ref="#PWR?"  Part="1"
 AR Path="/60AD0200/60B2D848/60EE4CD2" Ref="#PWR?"  Part="1"
 AR Path="/607155C8/60EE4CD2" Ref="#PWR?"  Part="1"
-F 0 "#PWR?" H 9650 2450 50  0001 C CNN
-F 1 "GNDD" H 9654 2545 50  0000 C CNN
-F 2 "" H 9650 2700 50  0001 C CNN
-F 3 "" H 9650 2700 50  0001 C CNN
-	1    9650 2700
+F 0 "#PWR?" H 9650 2550 50  0001 C CNN
+F 1 "GNDD" H 9654 2645 50  0000 C CNN
+F 2 "" H 9650 2800 50  0001 C CNN
+F 3 "" H 9650 2800 50  0001 C CNN
+	1    9650 2800
 	1    0    0    -1
 $EndComp
@@
 Wire Wire Line
 	8150 2300 8750 2300
+Wire Wire Line
+	9650 2800 9650 2750
+Wire Wire Line
+	9650 2750 10600 2750
+Wire Wire Line
+	10600 2750 10600 2400
+Wire Wire Line
+	10600 2400 10550 2400
+Connection ~ 9650 2750
+Wire Wire Line
+	9650 2750 9650 2700
 $EndSCHEMATC

Commit message: auto push run at Fri Apr  9 16:59:37 EDT 2021
Other:
- note added: "Stare at it a lil\nthen zoom andrew"
Changed lines of the file:
@@
 $Descr A4 11693 8268
 encoding utf-8
-Sheet 4 15
+Sheet 3 15
 Title ""
 Date ""
@@
 Wire Wire Line
 	9650 2750 9650 2700
+Text Notes 9250 1200 0    79   ~ 16
+Stare at it a lil\nthen zoom andrew
 $EndSCHEMATC
