File: hardware/readout_slice/ADC_LVDS.sch (KiCad schematic (older format))
At the start: 0 parts

Commit message: moving some things on readout slice
Parts:
- added U?: Mars_ZX2, Package_QFP:LQFP-160_24x24mm_P0.5mm, symbol readout:Mars_ZX2
Connections:
- new net +3V3: U?.117 (VCC_IO_B35), U?.126 (VCC_IO_B35), U?.82 (VCC_IO_B35)
Other:
- note added: "LVDS Bank"
Changed lines of the file:
@@
 Comment4 ""
 $EndDescr
+$Comp
+L readout:Mars_ZX2 U?
+U 5 1 606D4507
+P 3000 2500
+AR Path="/606D4507" Ref="U?"  Part="5"
+AR Path="/605605C8/606D4507" Ref="U?"  Part="5"
+AR Path="/60767BB3/606D4507" Ref="U?"  Part="5"
+F 0 "U?" H 2600 2650 50  0000 C CNN
+F 1 "Mars_ZX2" H 2650 2550 50  0000 C CNN
+F 2 "Package_QFP:LQFP-160_24x24mm_P0.5mm" H 3050 2850 50  0001 C CNN
+F 3 "http://gauss.bu.edu/svn/emphatic-doco/Docs/CITIROC1A%20-%20Datasheet%20V2.5.pdf" H 3050 2850 50  0001 C CNN
+	5    3000 2500
+	1    0    0    -1
+$EndComp
+Wire Wire Line
+	3000 2400 3000 2300
+Wire Wire Line
+	3000 2300 3100 2300
+Wire Wire Line
+	3200 2300 3200 2400
+Connection ~ 3000 2300
+Wire Wire Line
+	3000 2300 3000 2150
+Wire Wire Line
+	3100 2400 3100 2300
+Connection ~ 3100 2300
+Wire Wire Line
+	3100 2300 3200 2300
+$Comp
+L power:+3V3 #PWR?
+U 1 1 606D8143
+P 3000 2150
+F 0 "#PWR?" H 3000 2000 50  0001 C CNN
+F 1 "+3V3" H 3015 2323 50  0000 C CNN
+F 2 "" H 3000 2150 50  0001 C CNN
+F 3 "" H 3000 2150 50  0001 C CNN
+	1    3000 2150
+	1    0    0    -1
+$EndComp
+Text Notes 3300 2050 0    50   ~ 0
+LVDS Bank
 $EndSCHEMATC

Commit message: auto push run at Fri Apr  9 14:02:10 EDT 2021
Connections:
- net labels added: Raz_Chn_n, Raz_Chn_p, Val_Evt_n, Val_Evt_p
Other:
- note added: "2.5V"
- note added: "should be FPGA"
Changed lines of the file:
@@
 $Descr A4 11693 8268
 encoding utf-8
-Sheet 8 16
+Sheet 6 15
 Title ""
 Date ""
@@
 Wire Wire Line
 	3200 2300 3200 2400
-Connection ~ 3000 2300
 Wire Wire Line
-	3000 2300 3000 2150
+	3250 1500 3250 1350
 Wire Wire Line
 	3100 2400 3100 2300
@@
 L power:+3V3 #PWR?
 U 1 1 606D8143
-P 3000 2150
-F 0 "#PWR?" H 3000 2000 50  0001 C CNN
-F 1 "+3V3" H 3015 2323 50  0000 C CNN
-F 2 "" H 3000 2150 50  0001 C CNN
-F 3 "" H 3000 2150 50  0001 C CNN
-	1    3000 2150
+P 3250 1350
+F 0 "#PWR?" H 3250 1200 50  0001 C CNN
+F 1 "+3V3" H 3265 1523 50  0000 C CNN
+F 2 "" H 3250 1350 50  0001 C CNN
+F 3 "" H 3250 1350 50  0001 C CNN
+	1    3250 1350
 	1    0    0    -1
 $EndComp
 Text Notes 3300 2050 0    50   ~ 0
 LVDS Bank
+Text Notes 2900 2100 0    50   ~ 0
+2.5V
+Text Notes 2950 2200 0    50   ~ 0
+should be FPGA
+Text HLabel 6800 2050 0    50   Input ~ 0
+Raz_Chn_p
+Text HLabel 6800 2150 0    50   Input ~ 0
+Raz_Chn_n
+Text HLabel 6800 2250 0    50   Input ~ 0
+Val_Evt_p
+Text HLabel 6800 2350 0    50   Input ~ 0
+Val_Evt_n
 $EndSCHEMATC

Commit message: auto push run at Fri Apr  9 14:13:27 EDT 2021
Connections:
- net labels removed: Raz_Chn_n, Raz_Chn_p, Val_Evt_n, Val_Evt_p
Changed lines of the file:
@@
 Text Notes 2950 2200 0    50   ~ 0
 should be FPGA
-Text HLabel 6800 2050 0    50   Input ~ 0
-Raz_Chn_p
-Text HLabel 6800 2150 0    50   Input ~ 0
-Raz_Chn_n
-Text HLabel 6800 2250 0    50   Input ~ 0
-Val_Evt_p
-Text HLabel 6800 2350 0    50   Input ~ 0
-Val_Evt_n
 $EndSCHEMATC

Commit message: auto push run at Wed Apr 14 09:17:01 EDT 2021
Parts:
- removed U?: Mars_ZX2, Package_QFP:LQFP-160_24x24mm_P0.5mm, symbol readout:Mars_ZX2
Connections:
- net labels removed: +3V3
- wire segments 6 -> 0
Other:
- note removed: "2.5V"
- note removed: "LVDS Bank"
- note removed: "should be FPGA"
Changed lines of the file:
@@
 Comment4 ""
 $EndDescr
-$Comp
-L readout:Mars_ZX2 U?
-U 5 1 606D4507
-P 3000 2500
-AR Path="/606D4507" Ref="U?"  Part="5"
-AR Path="/605605C8/606D4507" Ref="U?"  Part="5"
-AR Path="/60767BB3/606D4507" Ref="U?"  Part="5"
-F 0 "U?" H 2600 2650 50  0000 C CNN
-F 1 "Mars_ZX2" H 2650 2550 50  0000 C CNN
-F 2 "Package_QFP:LQFP-160_24x24mm_P0.5mm" H 3050 2850 50  0001 C CNN
-F 3 "http://gauss.bu.edu/svn/emphatic-doco/Docs/CITIROC1A%20-%20Datasheet%20V2.5.pdf" H 3050 2850 50  0001 C CNN
-	5    3000 2500
-	1    0    0    -1
-$EndComp
-Wire Wire Line
-	3000 2400 3000 2300
-Wire Wire Line
-	3000 2300 3100 2300
-Wire Wire Line
-	3200 2300 3200 2400
-Wire Wire Line
-	3250 1500 3250 1350
-Wire Wire Line
-	3100 2400 3100 2300
-Connection ~ 3100 2300
-Wire Wire Line
-	3100 2300 3200 2300
-$Comp
-L power:+3V3 #PWR?
-U 1 1 606D8143
-P 3250 1350
-F 0 "#PWR?" H 3250 1200 50  0001 C CNN
-F 1 "+3V3" H 3265 1523 50  0000 C CNN
-F 2 "" H 3250 1350 50  0001 C CNN
-F 3 "" H 3250 1350 50  0001 C CNN
-	1    3250 1350
-	1    0    0    -1
-$EndComp
-Text Notes 3300 2050 0    50   ~ 0
-LVDS Bank
-Text Notes 2900 2100 0    50   ~ 0
-2.5V
-Text Notes 2950 2200 0    50   ~ 0
-should be FPGA
 $EndSCHEMATC
