File: hardware/readout_slice/citiroc-FPGA-1.sch (KiCad schematic (older format))
At the start: 9 parts

Commit message: need to fix one rescure in readout_slice
Parts:
- U?: symbol readout_slice-rescue:CITIROC1A-readout -> readout_slice-rescue:CITIROC1A-readout-readout_slice-rescue
Changed lines of the file:
@@
 $EndDescr
 $Comp
-L readout_slice-rescue:CITIROC1A-readout U?
+L readout_slice-rescue:CITIROC1A-readout-readout_slice-rescue U?
 U 2 1 606347B4
 P 2250 2300
 AR Path="/60548503/606347B4" Ref="U?"  Part="2"
 AR Path="/605DF89A/606347B4" Ref="U?"  Part="2"
+AR Path="/606347B4" Ref="U?"  Part="2"
 F 0 "U?" H 2175 -1923 50  0000 C CNN
 F 1 "CITIROC1A" H 2175 -2014 50  0000 C CNN

Commit message: getting rid of readout_slice rescue
Parts:
- U?: symbol readout_slice-rescue:CITIROC1A-readout-readout_slice-rescue -> readout:CITIROC1A
- U?: value XC7A35T-1FGG484 -> CITIROC1A; footprint (none) -> Package_QFP:LQFP-160_24x24mm_P0.5mm
Changed lines of the file:
@@
 $EndDescr
 $Comp
-L readout_slice-rescue:CITIROC1A-readout-readout_slice-rescue U?
+L readout:CITIROC1A U?
 U 2 1 606347B4
 P 2250 2300
@@
 AR Path="/605DF89A/606347BA" Ref="U?"  Part="8"
 F 0 "U?" H 5775 -1873 50  0000 C CNN
-F 1 "XC7A35T-1FGG484" H 5775 -1964 50  0000 C CNN
-F 2 "" H 5050 2050 50  0001 C CNN
-F 3 "" H 5050 2050 50  0001 C CNN
+F 1 "CITIROC1A" H 5775 -1964 50  0000 C CNN
+F 2 "Package_QFP:LQFP-160_24x24mm_P0.5mm" H 5050 2050 50  0001 C CNN
+F 3 "http://gauss.bu.edu/svn/emphatic-doco/Docs/CITIROC1A%20-%20Datasheet%20V2.5.pdf" H 5050 2050 50  0001 C CNN
 	8    6150 1900
 	1    0    0    -1

Commit message: more progress on readout_slice
Parts:
- added R? (x2): 100, symbol Device:R
- added TP?: probe, symbol Connector:TestPoint_2Pole
Connections:
- net GNDD: now also U?.73 (Raz_Chn_p), U?.76 (Val_Evt_n), R?.1, R?.1, TP?.2
- net T15: now reaches U?.103 (T<15>)
- net T15: now also U?.H3 (IO_L11P_T1_SRCC_35)
- net T14: now reaches U?.104 (T<14>)
- net T14: now also U?.H4 (IO_L12P_T1_MRCC_35)
- net T13: now reaches U?.105 (T<13>)
- net T13: now also U?.J1 (IO_L7N_T1_AD6N_35)
- net T12: now reaches U?.106 (T<12>)
- net T12: now also U?.J2 (IO_L9N_T1_DQS_AD7N_35)
- net T11: now reaches U?.107 (T<11>)
- net T11: now also U?.K1 (IO_L7P_T1_AD6P_35)
- net T10: now reaches U?.108 (T<10>)
- net T10: now also U?.K2 (IO_L9P_T1_DQS_AD7P_35)
- net T9: now reaches U?.109 (T<9>)
- net T9: now also U?.K3 (IO_L14N_T2_SRCC_35)
- net T8: now reaches U?.110 (T<8>)
- net T8: now also U?.L1 (IO_L15N_T2_DQS_35)
- net T7: now reaches U?.111 (T<7>)
- net T7: now also U?.L3 (IO_L14P_T2_SRCC_35)
- net T6: now reaches U?.112 (T<6>)
- net T6: now also U?.M1 (IO_L15P_T2_DQS_35)
- net T5: now reaches U?.113 (T<5>)
- net T5: now also U?.M2 (IO_L16N_T2_35)
- net T4: now reaches U?.114 (T<4>)
- net T4: now also U?.M3 (IO_L16P_T2_35)
- net T3: now reaches U?.115 (T<3>)
- net T3: now also U?.N2 (IO_L22N_T3_35)
- net T2: now reaches U?.116 (T<2>)
- net T2: now also U?.P1 (IO_L20N_T3_35)
- net T1: now reaches U?.117 (T<1>)
- net T1: now also U?.P2 (IO_L22P_T3_35)
- net T0: now reaches U?.118 (T<0>)
- net T0: now also U?.R1 (IO_L20P_T3_35)
- net at U?.119 (digital_probe): now also TP?.1
- net PS_modeb_ext: now reaches U?.120 (PS_modeb_ext)
- net load_sc_1: now reaches U?.124 (load_sc)
- net srout_sc_1: now reaches U?.125 (srout_sc)
- net srin_sc_1: now reaches U?.126 (srin_sc)
- net clk_sr_1: now reaches U?.127 (clk_sr)
- net rstb_sr_1: now reaches U?.128 (rstb_sr)
- net hold_lg: now reaches U?.131 (hold_lg)
- net resetb_read_1: now reaches U?.132 (resetb_read)
- net srout_read_1: now reaches U?.133 (srout_read)
- net srin_read_1: now reaches U?.134 (srin_read)
- net clk_read_1: now reaches U?.135 (clk_read)
- net hold_hg: now reaches U?.136 (hold_hg)
- net resetb_pa: now reaches U?.70 (resetb_pa)
- net rstb_PSC: now reaches U?.71 (rstb_PSC)
- net pwr_on: now reaches U?.72 (pwr_on)
- net +3V3: now reaches U?.74 (Raz_Chn_n)
- net +3V3: now also U?.75 (Val_Evt_p), R?.2, R?.2
- net dig_out_1: now reaches U?.77 (digital_output/hit_mux)
- net select_1: now reaches U?.79 (select)
- net PS_global_trig: now reaches U?.82 (PS_global_trig)
- net T31: now reaches U?.84 (T<31>)
- net T31: now also U?.A1 (IO_L1N_T0_AD4N_35)
- net T30: now reaches U?.85 (T<30>)
- net T30: now also U?.B1 (IO_L1P_T0_AD4P_35)
- net T29: now reaches U?.86 (T<29>)
- net T29: now also U?.B2 (IO_L2N_T0_AD12N_35)
- net T28: now reaches U?.87 (T<28>)
- net T28: now also U?.C2 (IO_L2P_T0_AD12P_35)
- net T27: now reaches U?.88 (T<27>)
- net T27: now also U?.D1 (IO_L3N_T0_DQS_AD5N_35)
- net T26: now reaches U?.89 (T<26>)
- net T26: now also U?.D2 (IO_L4N_T0_35)
- net T25: now reaches U?.90 (T<25>)
- net T25: now also U?.E1 (IO_L3P_T0_DQS_AD5P_35)
- net T24: now reaches U?.91 (T<24>)
- net T24: now also U?.E2 (IO_L4P_T0_35)
- net T23: now reaches U?.92 (T<23>)
- net T23: now also U?.F1 (IO_L5N_T0_AD13N_35)
- net T22: now reaches U?.93 (T<22>)
- net T22: now also U?.F3 (IO_L6P_T0_35)
- net T21: now reaches U?.94 (T<21>)
- net T21: now also U?.F4 (IO_0_35)
- net T20: now reaches U?.95 (T<20>)
- net T20: now also U?.G1 (IO_L5P_T0_AD13P_35)
- net T19: now reaches U?.96 (T<19>)
- net T19: now also U?.G2 (IO_L8N_T1_AD14N_35)
- net T18: now reaches U?.97 (T<18>)
- net T18: now also U?.G3 (IO_L11N_T1_SRCC_35)
- net T17: now reaches U?.98 (T<17>)
- net T17: now also U?.G4 (IO_L12N_T1_MRCC_35)
- net T16: now reaches U?.99 (T<16>)
- net T16: now also U?.H2 (IO_L8P_T1_AD14P_35)
- no-connect marks 0 -> 21
Other:
- note added: "LVDS Logic 0"
- note added: "LVDS Logic 1"
- note added: "Not Needed"
- note added: "from bank?"
- note added: "page 13 of\nCitiroc1A\ndatasheet"
- moved on the sheet: C?, U?B, U?H

Commit message: auto push run at Fri Apr  9 14:02:10 EDT 2021
Connections:
- net GNDD: no longer R?.1, R?.1, U?.73 (Raz_Chn_p), U?.76 (Val_Evt_n)
- net OR32_1: now reaches U?.78 (OR32)
- net NOR32_oc_1: now reaches U?.80 (NOR32_oc)
- net NOR32T_oc_1: now reaches U?.83 (NOR32T_oc)
- net Raz_Chn_n: now reaches U?.J4 (IO_L13N_T2_MRCC_35)
- net Raz_Chn_n: now also R?.1, U?.74 (Raz_Chn_n)
- net Val_Ext_n: now reaches U?.J6 (IO_L17N_T2_35)
- net Val_Ext_n: now also R?.1, U?.76 (Val_Evt_n)
- net Raz_Chn_p: now reaches U?.K4 (IO_L13P_T2_MRCC_35)
- net Raz_Chn_p: now also R?.2, U?.73 (Raz_Chn_p)
- net Val_Ext_p: now reaches U?.K6 (IO_L17P_T2_35)
- net Val_Ext_p: now also R?.2, U?.75 (Val_Evt_p)
- removed net +3V3: R?.2, R?.2, U?.74 (Raz_Chn_n), U?.75 (Val_Evt_p)
- no-connect marks 21 -> 14
Other:
- note added: "LEDS!!!"
- note added: "and GPIOs\n"
- note added: "make sure signals don’t just disapper\nmake accessable on outer layer\n"
- note added: "note open collectors from data sheet"
- note removed: "LVDS Logic 0"
- note removed: "LVDS Logic 1"
- note removed: "Not Needed"
- note removed: "page 13 of\nCitiroc1A\ndatasheet"
- moved on the sheet: R?
Changed lines of the file:
@@
 $Descr A4 11693 8268
 encoding utf-8
-Sheet 4 16
+Sheet 14 15
 Title ""
 Date ""
@@
 Text HLabel 2700 3700 0    50   Input ~ 0
 load_sc_1
-NoConn ~ 4200 5900
-NoConn ~ 4200 6100
-NoConn ~ 4200 6000
-Text Notes 4250 6000 0    50   ~ 0
-Not Needed
-Text Notes 1700 2650 0    50   ~ 0
-LVDS Logic 0
 $Comp
 L Device:R R?
 U 1 1 608CECB3
 P 2500 2900
-F 0 "R?" V 2600 2850 50  0000 L CNN
+F 0 "R?" V 2550 3000 50  0000 L CNN
 F 1 "100" V 2500 2800 50  0000 L CNN
 F 2 "" V 2430 2900 50  0001 C CNN
@@
 	0    -1   -1   0
 $EndComp
-$Comp
-L Device:R R?
-U 1 1 608D2690
-P 2500 2700
-F 0 "R?" V 2650 2650 50  0000 L CNN
-F 1 "100" V 2500 2600 50  0000 L CNN
-F 2 "" V 2430 2700 50  0001 C CNN
-F 3 "~" H 2500 2700 50  0001 C CNN
-	1    2500 2700
-	0    -1   -1   0
-$EndComp
-$Comp
-L power:+3V3 #PWR?
-U 1 1 608D5CA2
-P 2750 2000
-F 0 "#PWR?" H 2750 1850 50  0001 C CNN
-F 1 "+3V3" H 2750 2150 50  0000 C CNN
-F 2 "" H 2750 2000 50  0001 C CNN
-F 3 "" H 2750 2000 50  0001 C CNN
-	1    2750 2000
-	1    0    0    -1
-$EndComp
-Wire Wire Line
-	2850 2900 2750 2900
-Wire Wire Line
-	2750 2900 2750 2700
-Wire Wire Line
-	2850 2700 2750 2700
-Connection ~ 2750 2700
-Wire Wire Line
-	2750 2700 2750 2000
-Wire Wire Line
-	2750 2900 2650 2900
-Connection ~ 2750 2900
-Wire Wire Line
-	2750 2700 2650 2700
-Wire Wire Line
-	2850 2600 2250 2600
-Wire Wire Line
-	2250 2600 2250 2700
-Wire Wire Line
-	2250 2700 2350 2700
-Wire Wire Line
-	2850 3000 2250 3000
-Wire Wire Line
-	2250 3000 2250 2900
-Wire Wire Line
-	2250 2900 2350 2900
-Wire Wire Line
-	2250 2900 2250 2700
-Connection ~ 2250 2900
-Connection ~ 2250 2700
-Wire Wire Line
-	2250 3000 2250 3100
-Connection ~ 2250 3000
-$Comp
-L power:GNDD #PWR?
-U 1 1 608E1AE4
-P 2250 3100
-AR Path="/605605C8/608E1AE4" Ref="#PWR?"  Part="1"
-AR Path="/60548503/608E1AE4" Ref="#PWR?"  Part="1"
-AR Path="/605DF89A/608E1AE4" Ref="#PWR?"  Part="1"
-F 0 "#PWR?" H 2250 2850 50  0001 C CNN
-F 1 "GNDD" H 2250 2950 50  0000 C CNB
-F 2 "" H 2250 3100 50  0001 C CNN
-F 3 "" H 2250 3100 50  0001 C CNN
-	1    2250 3100
-	1    0    0    -1
-$EndComp
 Text HLabel 2750 3200 0    50   Input ~ 0
 select_1
-Text Notes 1700 2900 0    50   ~ 0
-LVDS Logic 1
-Text Notes 1450 2850 2    50   ~ 0
-page 13 of\nCitiroc1A\ndatasheet
 Wire Wire Line
 	7850 2000 7850 2100
@@
 Wire Wire Line
 	8900 5300 9100 5300
-NoConn ~ 6150 4100
-NoConn ~ 6150 4200
-NoConn ~ 6150 4700
-NoConn ~ 6150 4800
 NoConn ~ 6150 5000
 NoConn ~ 6150 5100
@@
 Wire Wire Line
 	3650 1700 3650 2000
+Text Notes 1000 2200 0    50   ~ 0
+make sure signals don’t just disapper\nmake accessable on outer layer\n
+Text Notes 4400 6550 0    50   ~ 0
+note open collectors from data sheet
+Text Notes 3800 7000 0    157  ~ 31
+LEDS!!!
+Text Notes 1750 7000 0    157  ~ 31
+and GPIOs\n
+Wire Wire Line
+	4200 5900 4350 5900
+Wire Wire Line
+	4200 6000 4350 6000
+Wire Wire Line
+	4200 6100 4350 6100
+Text HLabel 4350 5900 2    50   Input ~ 0
+NOR32T_oc_1
+Text HLabel 4350 6000 2    50   Input ~ 0
+NOR32_oc_1
+Text HLabel 4350 6100 2    50   Input ~ 0
+OR32_1
+$Comp
+L Device:R R?
+U 1 1 608D2690
+P 2500 2600
+F 0 "R?" V 2550 2700 50  0000 L CNN
+F 1 "100" V 2500 2500 50  0000 L CNN
+F 2 "" V 2430 2600 50  0001 C CNN
+F 3 "~" H 2500 2600 50  0001 C CNN
+	1    2500 2600
+	0    -1   -1   0
+$EndComp
+Wire Wire Line
+	2850 2600 2750 2600
+Wire Wire Line
+	2850 2900 2750 2900
+Wire Wire Line
+	2750 2600 2750 2500
+Wire Wire Line
+	2750 2500 2200 2500
+Connection ~ 2750 2600
+Wire Wire Line
+	2750 2600 2650 2600
+Wire Wire Line
+	2750 2900 2750 2800
+Wire Wire Line
+	2750 2800 2200 2800
+Connection ~ 2750 2900
+Wire Wire Line
+	2750 2900 2650 2900
+Wire Wire Line
+	2350 2900 2300 2900
+Wire Wire Line
+	2300 2900 2300 3000
+Wire Wire Line
+	2300 3000 2850 3000
+Wire Wire Line
+	2300 3000 2200 3000
+Connection ~ 2300 3000
+Wire Wire Line
+	2200 2700 2300 2700
+Wire Wire Line
+	2350 2600 2300 2600
+Wire Wire Line
+	2300 2600 2300 2700
+Connection ~ 2300 2700
+Wire Wire Line
+	2300 2700 2850 2700
+Text Label 2200 2500 2    50   ~ 0
+Raz_Chn_p
+Text Label 2200 2700 2    50   ~ 0
+Raz_Chn_n
+Text Label 2200 2800 2    50   ~ 0
+Val_Ext_p
+Text Label 2200 3000 2    50   ~ 0
+Val_Ext_n
+Text Label 5650 4100 0    50   ~ 0
+Raz_Chn_p
+Text Label 5650 4200 0    50   ~ 0
+Raz_Chn_n
+Wire Wire Line
+	6150 4100 5650 4100
+Wire Wire Line
+	5650 4200 6150 4200
+Text Label 5700 4700 0    50   ~ 0
+Val_Ext_p
+Text Label 5700 4800 0    50   ~ 0
+Val_Ext_n
+Wire Wire Line
+	6150 4700 5700 4700
+Wire Wire Line
+	5700 4800 6150 4800
 $EndSCHEMATC

Commit message: auto push run at Fri Apr  9 16:59:37 EDT 2021
Other:
- note added: "should be 2.5V"
Changed lines of the file:
@@
 $Descr A4 11693 8268
 encoding utf-8
-Sheet 14 15
+Sheet 13 15
 Title ""
 Date ""
@@
 Wire Wire Line
 	5700 4800 6150 4800
+Text Notes 1150 2700 0    50   ~ 0
+should be 2.5V
 $EndSCHEMATC

Commit message: auto push run at Wed Apr 14 09:17:01 EDT 2021
Connections:
- net Raz_Chn_n: no longer R?.1, U?.74 (Raz_Chn_n)
- new net Raz_chn_n: R?.1, U?.74 (Raz_Chn_n)
Other:
- note added: "Parrallel w/ other chip,\ndoes that change 100R?"
- note removed: "should be 2.5V"
Changed lines of the file:
@@
 $Descr A4 11693 8268
 encoding utf-8
-Sheet 13 15
+Sheet 12 14
 Title ""
 Date ""
@@
 Wire Wire Line
 	2300 2700 2850 2700
-Text Label 2200 2500 2    50   ~ 0
-Raz_Chn_p
-Text Label 2200 2700 2    50   ~ 0
-Raz_Chn_n
-Text Label 2200 2800 2    50   ~ 0
-Val_Ext_p
-Text Label 2200 3000 2    50   ~ 0
-Val_Ext_n
 Text Label 5650 4100 0    50   ~ 0
 Raz_Chn_p
@@
 Wire Wire Line
 	5700 4800 6150 4800
-Text Notes 1150 2700 0    50   ~ 0
-should be 2.5V
+Text Notes 750  2800 0    50   ~ 10
+Parrallel w/ other chip,\ndoes that change 100R?
+Text HLabel 2200 2500 0    50   Input ~ 0
+Raz_Chn_p
+Text HLabel 2200 2700 0    50   Input ~ 0
+Raz_chn_n
+Text HLabel 2200 2800 0    50   Input ~ 0
+Val_Ext_p
+Text HLabel 2200 3000 0    50   Input ~ 0
+Val_Ext_n
 $EndSCHEMATC

Commit message: auto push run at Wed Apr 14 11:00:44 EDT 2021
Parts:
- added R? (x33): R, symbol Device:R
Connections:
- net +1V8: now also R?.1, R?.1, R?.1, R?.1, R?.1, R?.1, R?.1, R?.1, R?.1, R?.1, R?.1, R?.1, R?.1, R?.1, R?.1, R?.1, R?.1, R?.1, R?.1, R?.1, R?.1, R?.1, R?.1, R?.1, R?.1, R?.1, R?.1, R?.1, R?.1, R?.1, R?.1, R?.1, R?.1
- net OR32_1: now also R?.2
- net T0: now also R?.2
- net T1: now also R?.2
- net T10: now also R?.2
- net T11: now also R?.2
- net T12: now also R?.2
- net T13: now also R?.2
- net T14: now also R?.2
- net T15: now also R?.2
- net T16: now also R?.2
- net T17: now also R?.2
- net T18: now also R?.2
- net T19: now also R?.2
- net T2: now also R?.2
- net T20: now also R?.2
- net T21: now also R?.2
- net T22: now also R?.2
- net T23: now also R?.2
- net T24: now also R?.2
- net T25: now also R?.2
- net T26: now also R?.2
- net T27: now also R?.2
- net T28: now also R?.2
- net T29: now also R?.2
- net T3: now also R?.2
- net T30: now also R?.2
- net T31: now also R?.2
- net T4: now also R?.2
- net T5: now also R?.2
- net T6: now also R?.2
- net T7: now also R?.2
- net T8: now also R?.2
- net T9: now also R?.2
Other:
- note added: "r in range 1k to 10k \ndepending on \nspeed of recovery"
- moved on the sheet: R?, TP?, U?B, U?H

Commit message: auto push run at Wed Apr 14 11:08:32 EDT 2021
Connections:
- net 1v8_GPIO2: now reaches U?.L4 (IO_L18N_T2_35)
- net 1v8_GPIO1: now reaches U?.L5 (IO_L18P_T2_35)
- no-connect marks 14 -> 12
Other:
- moved on the sheet: U?H
Changed lines of the file:
@@
 L readout:XC7A35T-1FGG484 U?
 U 8 1 606347BA
-P 9550 2500
+P 8550 2350
 AR Path="/605605C8/606347BA" Ref="U?"  Part="8"
 AR Path="/60548503/606347BA" Ref="U?"  Part="8"
 AR Path="/605DF89A/606347BA" Ref="U?"  Part="8"
-F 0 "U?" H 9175 -1273 50  0000 C CNN
-F 1 "CITIROC1A" H 9175 -1364 50  0000 C CNN
-F 2 "Package_QFP:LQFP-160_24x24mm_P0.5mm" H 8450 2650 50  0001 C CNN
-F 3 "http://gauss.bu.edu/svn/emphatic-doco/Docs/CITIROC1A%20-%20Datasheet%20V2.5.pdf" H 8450 2650 50  0001 C CNN
-	8    9550 2500
+F 0 "U?" H 8175 -1423 50  0000 C CNN
+F 1 "CITIROC1A" H 8175 -1514 50  0000 C CNN
+F 2 "Package_QFP:LQFP-160_24x24mm_P0.5mm" H 7450 2500 50  0001 C CNN
+F 3 "http://gauss.bu.edu/svn/emphatic-doco/Docs/CITIROC1A%20-%20Datasheet%20V2.5.pdf" H 7450 2500 50  0001 C CNN
+	8    8550 2350
 	1    0    0    -1
 $EndComp
@@
 	10050 1200 10300 1200
 Wire Wire Line
-	9500 2400 9500 2350
-Wire Wire Line
-	9400 2400 9400 2350
-Wire Wire Line
-	9400 2350 9500 2350
-Wire Wire Line
-	9300 2400 9300 2350
-Wire Wire Line
-	9300 2350 9400 2350
-Connection ~ 9400 2350
-Wire Wire Line
-	9200 2400 9200 2350
-Connection ~ 9300 2350
-Wire Wire Line
-	9100 2400 9100 2350
-Wire Wire Line
-	9100 2350 9200 2350
-Connection ~ 9200 2350
-Wire Wire Line
-	9200 2350 9300 2350
-Wire Wire Line
-	9000 2400 9000 2350
-Wire Wire Line
-	9000 2350 9100 2350
-Connection ~ 9100 2350
+	8500 2250 8500 2200
+Wire Wire Line
+	8400 2250 8400 2200
+Wire Wire Line
+	8400 2200 8500 2200
+Wire Wire Line
+	8300 2250 8300 2200
+Wire Wire Line
+	8300 2200 8400 2200
+Connection ~ 8400 2200
+Wire Wire Line
+	8200 2250 8200 2200
+Connection ~ 8300 2200
+Wire Wire Line
+	8100 2250 8100 2200
+Wire Wire Line
+	8100 2200 8200 2200
+Connection ~ 8200 2200
+Wire Wire Line
+	8200 2200 8300 2200
+Wire Wire Line
+	8000 2250 8000 2200
+Wire Wire Line
+	8000 2200 8100 2200
+Connection ~ 8100 2200
 $Comp
 L power:+1V8 #PWR?
 U 1 1 6063482B
-P 9500 2250
+P 8500 2100
 AR Path="/60548503/6063482B" Ref="#PWR?"  Part="1"
 AR Path="/605DF89A/6063482B" Ref="#PWR?"  Part="1"
-F 0 "#PWR?" H 9500 2100 50  0001 C CNN
-F 1 "+1V8" H 9500 2400 50  0000 C CNB
-F 2 "" H 9500 2250 50  0001 C CNN
-F 3 "" H 9500 2250 50  0001 C CNN
-	1    9500 2250
+F 0 "#PWR?" H 8500 1950 50  0001 C CNN
+F 1 "+1V8" H 8500 2250 50  0000 C CNB
+F 2 "" H 8500 2100 50  0001 C CNN
+F 3 "" H 8500 2100 50  0001 C CNN
+	1    8500 2100
 	1    0    0    -1
 $EndComp
 Text Notes 700  850  0    157  ~ 31
 3V3 controls?
-Connection ~ 9500 2350
+Connection ~ 8500 2200
 Text Notes 2700 1800 0    50   ~ 0
 from bank?
@@
 select_1
 Wire Wire Line
-	9500 2250 9500 2350
+	8500 2100 8500 2200
 $Comp
 L power:+1V8 #PWR?
@@
 	4250 5200 4050 5200
 Wire Wire Line
-	10550 5450 10750 5450
-Text Label 10750 5450 2    50   ~ 0
+	9550 5300 9750 5300
+Text Label 9750 5300 2    50   ~ 0
 T0
-Text Label 7600 2650 0    50   ~ 0
+Text Label 6600 2500 0    50   ~ 0
 T31
 Wire Wire Line
-	7600 2650 7800 2650
-Text Label 7600 2550 0    50   ~ 0
+	6600 2500 6800 2500
+Text Label 6600 2400 0    50   ~ 0
 T30
-Text Label 10750 2850 2    50   ~ 0
+Text Label 9750 2700 2    50   ~ 0
 T29
-Text Label 10750 2750 2    50   ~ 0
+Text Label 9750 2600 2    50   ~ 0
 T28
-Text Label 7600 2950 0    50   ~ 0
+Text Label 6600 2800 0    50   ~ 0
 T27
-Text Label 10750 3150 2    50   ~ 0
+Text Label 9750 3000 2    50   ~ 0
 T26
-Text Label 7600 2850 0    50   ~ 0
+Text Label 6600 2700 0    50   ~ 0
 T25
-Text Label 10750 3050 2    50   ~ 0
+Text Label 9750 2900 2    50   ~ 0
 T24
-Text Label 7600 3250 0    50   ~ 0
+Text Label 6600 3100 0    50   ~ 0
 T23
-Text Label 10750 3350 2    50   ~ 0
+Text Label 9750 3200 2    50   ~ 0
 T22
-Text Label 10750 2550 2    50   ~ 0
+Text Label 9750 2400 2    50   ~ 0
 T21
-Text Label 7600 3150 0    50   ~ 0
+Text Label 6600 3000 0    50   ~ 0
 T20
-Text Label 10750 3750 2    50   ~ 0
+Text Label 9750 3600 2    50   ~ 0
 T19
-Text Label 7600 4150 0    50   ~ 0
+Text Label 6600 4000 0    50   ~ 0
 T18
-Text Label 10750 4350 2    50   ~ 0
+Text Label 9750 4200 2    50   ~ 0
 T17
-Text Label 10750 3650 2    50   ~ 0
+Text Label 9750 3500 2    50   ~ 0
 T16
-Text Label 7600 4050 0    50   ~ 0
+Text Label 6600 3900 0    50   ~ 0
 T15
-Text Label 10750 4250 2    50   ~ 0
+Text Label 9750 4100 2    50   ~ 0
 T14
-Text Label 7600 3550 0    50   ~ 0
+Text Label 6600 3400 0    50   ~ 0
 T13
-Text Label 7600 3850 0    50   ~ 0
+Text Label 6600 3700 0    50   ~ 0
 T12
-Text Label 7600 3450 0    50   ~ 0
+Text Label 6600 3300 0    50   ~ 0
 T11
-Text Label 7600 3750 0    50   ~ 0
+Text Label 6600 3600 0    50   ~ 0
 T10
-Text Label 10750 4650 2    50   ~ 0
+Text Label 9750 4500 2    50   ~ 0
 T9
-Text Label 7600 4750 0    50   ~ 0
+Text Label 6600 4600 0    50   ~ 0
 T8
-Text Label 10750 4550 2    50   ~ 0
+Text Label 9750 4400 2    50   ~ 0
 T7
-Text Label 7600 4650 0    50   ~ 0
+Text Label 6600 4500 0    50   ~ 0
 T6
-Text Label 10750 4950 2    50   ~ 0
+Text Label 9750 4800 2    50   ~ 0
 T5
-Text Label 10750 4850 2    50   ~ 0
+Text Label 9750 4700 2    50   ~ 0
 T4
-Text Label 10750 5850 2    50   ~ 0
+Text Label 9750 5700 2    50   ~ 0
 T3
-Text Label 10750 5750 2    50   ~ 0
+Text Label 9750 5600 2    50   ~ 0
 T1
 Wire Wire Line
-	10750 5750 10550 5750
-Wire Wire Line
-	10750 5850 10550 5850
-Wire Wire Line
-	10550 4850 10750 4850
-Wire Wire Line
-	10750 4950 10550 4950
-Wire Wire Line
-	7800 4650 7600 4650
-Wire Wire Line
-	10750 4550 10550 4550
-Wire Wire Line
-	7800 4750 7600 4750
-Wire Wire Line
-	10750 4650 10550 4650
-Wire Wire Line
-	7800 3750 7600 3750
-Wire Wire Line
-	7600 3450 7800 3450
-Wire Wire Line
-	7800 3850 7600 3850
-Wire Wire Line
-	7600 3550 7800 3550
-Wire Wire Line
-	10550 4250 10750 4250
-Wire Wire Line
-	7600 4050 7800 4050
-Wire Wire Line
-	10750 3650 10550 3650
-Wire Wire Line
-	10550 4350 10750 4350
-Wire Wire Line
-	7600 4150 7800 4150
-Wire Wire Line
-	10550 3750 10750 3750
-Wire Wire Line
-	7600 3150 7800 3150
-Wire Wire Line
-	10550 2550 10750 2550
-Wire Wire Line
-	10750 3350 10550 3350
-Wire Wire Line
-	7800 3250 7600 3250
-Wire Wire Line
-	10750 3050 10550 3050
-Wire Wire Line
-	7800 2850 7600 2850
-Wire Wire Line
-	10750 3150 10550 3150
-Wire Wire Line
-	7800 2950 7600 2950
-Wire Wire Line
-	10750 2750 10550 2750
-Wire Wire Line
-	10550 2850 10750 2850
-Wire Wire Line
-	7600 2550 7800 2550
-Text Label 10750 5550 2    50   ~ 0
+	9750 5600 9550 5600
+Wire Wire Line
+	9750 5700 9550 5700
+Wire Wire Line
+	9550 4700 9750 4700
+Wire Wire Line
+	9750 4800 9550 4800
+Wire Wire Line
+	6800 4500 6600 4500
+Wire Wire Line
+	9750 4400 9550 4400
+Wire Wire Line
+	6800 4600 6600 4600
+Wire Wire Line
+	9750 4500 9550 4500
+Wire Wire Line
+	6800 3600 6600 3600
+Wire Wire Line
+	6600 3300 6800 3300
+Wire Wire Line
+	6800 3700 6600 3700
+Wire Wire Line
+	6600 3400 6800 3400
+Wire Wire Line
+	9550 4100 9750 4100
+Wire Wire Line
+	6600 3900 6800 3900
+Wire Wire Line
+	9750 3500 9550 3500
+Wire Wire Line
+	9550 4200 9750 4200
+Wire Wire Line
+	6600 4000 6800 4000
+Wire Wire Line
+	9550 3600 9750 3600
+Wire Wire Line
+	6600 3000 6800 3000
+Wire Wire Line
+	9550 2400 9750 2400
+Wire Wire Line
+	9750 3200 9550 3200
+Wire Wire Line
+	6800 3100 6600 3100
+Wire Wire Line
+	9750 2900 9550 2900
+Wire Wire Line
+	6800 2700 6600 2700
+Wire Wire Line
+	9750 3000 9550 3000
+Wire Wire Line
+	6800 2800 6600 2800
+Wire Wire Line
+	9750 2600 9550 2600
+Wire Wire Line
+	9550 2700 9750 2700
+Wire Wire Line
+	6600 2400 6800 2400
+Text Label 9750 5400 2    50   ~ 0
 T2
 Wire Wire Line
-	10550 5550 10750 5550
-NoConn ~ 7800 5250
-NoConn ~ 7800 5350
-NoConn ~ 7800 5550
-NoConn ~ 7800 5650
-NoConn ~ 7800 5850
-NoConn ~ 7800 5950
-NoConn ~ 7800 6150
-NoConn ~ 10550 6150
-NoConn ~ 10550 6050
-NoConn ~ 10550 5250
-NoConn ~ 10550 5150
-NoConn ~ 10550 4050
-NoConn ~ 10550 3950
-NoConn ~ 10550 3450
+	9550 5400 9750 5400
+NoConn ~ 6800 5100
+NoConn ~ 6800 5200
+NoConn ~ 6800 5400
+NoConn ~ 6800 5500
+NoConn ~ 6800 5700
+NoConn ~ 6800 5800
+NoConn ~ 6800 6000
+NoConn ~ 9550 6000
+NoConn ~ 9550 5900
+NoConn ~ 9550 3900
+NoConn ~ 9550 3800
+NoConn ~ 9550 3300
 $Comp
 L Connector:TestPoint_2Pole TP?
@@
 Wire Wire Line
 	2150 2700 2700 2700
-Text Label 7300 4350 0    50   ~ 0
+Text Label 6300 4200 0    50   ~ 0
 Raz_Chn_p
-Text Label 7300 4450 0    50   ~ 0
+Text Label 6300 4300 0    50   ~ 0
 Raz_Chn_n
 Wire Wire Line
-	7800 4350 7300 4350
-Wire Wire Line
-	7300 4450 7800 4450
-Text Label 7350 4950 0    50   ~ 0
+	6800 4200 6300 4200
+Wire Wire Line
+	6300 4300 6800 4300
+Text Label 6350 4800 0    50   ~ 0
 Val_Ext_p
-Text Label 7350 5050 0    50   ~ 0
+Text Label 6350 4900 0    50   ~ 0
 Val_Ext_n
 Wire Wire Line
-	7800 4950 7350 4950
-Wire Wire Line
-	7350 5050 7800 5050
+	6800 4800 6350 4800
+Wire Wire Line
+	6350 4900 6800 4900
 Text Notes 550  2850 0    50   ~ 10
 Parrallel w/ other chip,\ndoes that change 100R?
@@
 Wire Wire Line
 	4150 6100 4200 6100
+Text HLabel 9750 5000 2    50   Input ~ 0
+1v8_GPIO1
+Text HLabel 9750 5100 2    50   Input ~ 0
+1v8_GPIO2
+Wire Wire Line
+	9750 5000 9550 5000
+Wire Wire Line
+	9550 5100 9750 5100
 $EndSCHEMATC
