File: hardware/readout_slice/Citiroc-in-1.sch (KiCad schematic (older format))
At the start: 6 parts

Commit message: need to fix one rescure in readout_slice
Parts:
- U?: symbol readout_slice-rescue:CITIROC1A-readout -> readout_slice-rescue:CITIROC1A-readout-readout_slice-rescue
Changed lines of the file:
@@
 $Descr A4 11693 8268
 encoding utf-8
-Sheet 7 16
+Sheet 6 16
 Title ""
 Date ""
@@
 	9450 1600 3800 1600
 $Comp
-L readout_slice-rescue:CITIROC1A-readout U?
+L readout_slice-rescue:CITIROC1A-readout-readout_slice-rescue U?
 U 3 1 60AFA4EB
 P 10100 900

Commit message: getting rid of readout_slice rescue
Parts:
- U?: symbol readout_slice-rescue:CITIROC1A-readout-readout_slice-rescue -> readout:CITIROC1A
Changed lines of the file:
@@
 	9450 1600 3800 1600
 $Comp
-L readout_slice-rescue:CITIROC1A-readout-readout_slice-rescue U?
+L readout:CITIROC1A U?
 U 3 1 60AFA4EB
 P 10100 900

Commit message: more progress on readout_slice
Other:
- moved on the sheet: U?C
Changed lines of the file:
@@
 	1700 6800 1450 6800
 Wire Wire Line
-	3700 1500 9450 1500
+	3700 1500 8450 1500
 Wire Wire Line
-	9450 1400 3600 1400
+	8450 1400 3600 1400
 Wire Wire Line
-	3500 1300 9450 1300
+	3500 1300 8450 1300
 Wire Wire Line
-	9450 1200 3400 1200
+	8450 1200 3400 1200
 Wire Wire Line
-	3300 1100 9450 1100
+	3300 1100 8450 1100
 Wire Wire Line
-	9450 1000 3200 1000
+	8450 1000 3200 1000
 Wire Wire Line
-	6600 4100 9450 4100
+	6600 4100 8450 4100
 Wire Wire Line
-	6500 4000 9450 4000
+	6500 4000 8450 4000
 Wire Wire Line
-	6400 3900 9450 3900
+	6400 3900 8450 3900
 Wire Wire Line
-	6300 3800 9450 3800
+	6300 3800 8450 3800
 Wire Wire Line
-	6200 3700 9450 3700
+	6200 3700 8450 3700
 Wire Wire Line
-	9450 3600 6100 3600
+	8450 3600 6100 3600
 Wire Wire Line
-	9450 3500 6000 3500
+	8450 3500 6000 3500
 Wire Wire Line
-	5900 3400 9450 3400
+	5900 3400 8450 3400
 Wire Wire Line
-	9450 3300 5700 3300
+	8450 3300 5700 3300
 Wire Wire Line
-	5600 3200 9450 3200
+	5600 3200 8450 3200
 Wire Wire Line
-	9450 3100 5500 3100
+	8450 3100 5500 3100
 Wire Wire Line
-	5400 3000 9450 3000
+	5400 3000 8450 3000
 Wire Wire Line
-	9450 2900 5300 2900
+	8450 2900 5300 2900
 Wire Wire Line
-	5200 2800 9450 2800
+	5200 2800 8450 2800
 Wire Wire Line
-	9450 2700 5100 2700
+	8450 2700 5100 2700
 Wire Wire Line
-	5000 2600 9450 2600
+	5000 2600 8450 2600
 Wire Wire Line
-	9450 2500 4800 2500
+	8450 2500 4800 2500
 Wire Wire Line
-	4700 2400 9450 2400
+	4700 2400 8450 2400
 Wire Wire Line
-	9450 2300 4600 2300
+	8450 2300 4600 2300
 Wire Wire Line
-	4500 2200 9450 2200
+	4500 2200 8450 2200
 Wire Wire Line
-	9450 2100 4400 2100
+	8450 2100 4400 2100
 Wire Wire Line
-	4300 2000 9450 2000
+	4300 2000 8450 2000
 Wire Wire Line
-	9450 1900 4200 1900
+	8450 1900 4200 1900
 Wire Wire Line
-	4100 1800 9450 1800
+	4100 1800 8450 1800
 Wire Wire Line
-	3900 1700 9450 1700
+	3900 1700 8450 1700
 Wire Wire Line
-	9450 1600 3800 1600
+	8450 1600 3800 1600
 $Comp
 L readout:CITIROC1A U?
 U 3 1 60AFA4EB
-P 10100 900
+P 9100 900
 AR Path="/60AFA4EB" Ref="U?"  Part="3"
 AR Path="/6076454A/60AFA4EB" Ref="U?"  Part="3"
-F 0 "U?" H 10100 -3623 50  0000 C CNN
-F 1 "CITIROC1A" H 10100 -3714 50  0000 C CNN
-F 2 "Package_QFP:LQFP-160_24x24mm_P0.5mm" H 9500 1050 50  0001 C CNN
-F 3 "http://gauss.bu.edu/svn/emphatic-doco/Docs/CITIROC1A%20-%20Datasheet%20V2.5.pdf" H 9500 1050 50  0001 C CNN
-	3    10100 900
+F 0 "U?" H 9100 -3623 50  0000 C CNN
+F 1 "CITIROC1A" H 9100 -3714 50  0000 C CNN
+F 2 "Package_QFP:LQFP-160_24x24mm_P0.5mm" H 8500 1050 50  0001 C CNN
+F 3 "http://gauss.bu.edu/svn/emphatic-doco/Docs/CITIROC1A%20-%20Datasheet%20V2.5.pdf" H 8500 1050 50  0001 C CNN
+	3    9100 900
 	1    0    0    -1
 $EndComp

Commit message: auto push run at Fri Apr  9 14:02:10 EDT 2021
Parts:
- removed RN? (x4): R_Network08_US, Resistor_THT:R_Array_SIP9, symbol Device:R_Network08_US
- added C? (x32): 100n, symbol Device:C_Small
- added C? (x2): 10u, symbol Device:C_Small
- added C? (x3): 1u, symbol Device:C_Small
- added J?: BNC, symbol Connector:Conn_Coaxial
- added J?: GPIO Header, symbol Connector_Generic:Conn_02x04_Odd_Even
- added R? (x32): 50, symbol Device:R
- added R?: 470k, symbol Device:R
- added R?: 1k, symbol Device:R
- added RV?: 10k, symbol Device:R_POT
- added U?: ADS7955, Package_SO:TSSOP-30_4.4x7.8mm_P0.5mm, symbol readout:ADS7955
- added U?: REF5025, Package_SO:SOIC-8_3.9x4.9mm_P1.27mm, symbol Reference_Voltage:REF5025ID
Connections:
- net GNDA: now also C?.2, C?.2, C?.2, C?.2, C?.2, C?.2, C?.2, C?.2, C?.2, C?.2, C?.2, C?.2, C?.2, C?.2, C?.2, C?.2, C?.2, C?.2, C?.2, C?.2, C?.2, C?.2, C?.2, C?.2, C?.2, C?.2, C?.2, C?.2, C?.2, C?.2, C?.2, C?.2, C?.2, C?.2, C?.2, C?.2, C?.2, J?.2 (Ext), R?.2, U?.10 (AGND), U?.22 (AGND), U?.3 (REFM), U?.4 (GND), U?.6 (AGND), U?.9 (AINM)
- net at J?.103, U?.32 (in25): now also R?.1
- net at J?.105, U?.33 (in26): now also R?.1
- net at J?.107, U?.34 (in27): now also R?.1
- net at J?.109, U?.35 (in28): now also R?.1
- net at J?.11, U?.6 (in2): now also R?.1
- net at J?.111, U?.36 (in29): now also R?.1
- net at J?.113, U?.37 (in30): now also R?.1
- net at J?.115, U?.38 (in31): now also R?.1
- net at J?.15, U?.7 (in3): now also R?.1
- net at J?.19, U?.8 (in4): now also R?.1
- net at J?.23, U?.9 (in5): now also R?.1
- net at J?.27, U?.10 (in6): now also R?.1
- net at J?.3, U?.4 (in0): now also R?.1
- net at J?.31, U?.11 (in7): now also R?.1
- net at J?.35, U?.13 (in8): now also R?.1
- net at J?.39, U?.14 (in9): now also R?.1
- net at J?.43, U?.15 (in10): now also R?.1
- net at J?.47, U?.16 (in11): now also R?.1
- net at J?.51, U?.17 (in12): now also R?.1
- net at J?.55, U?.18 (in13): now also R?.1
- net at J?.59, U?.19 (in14): now also R?.1
- net at J?.63, U?.20 (in15): now also R?.1
- net at J?.67, U?.22 (in16): now also R?.1
- net at J?.7, U?.5 (in1): now also R?.1
- net at J?.71, U?.23 (in17): now also R?.1
- net at J?.75, U?.24 (in18): now also R?.1
- net at J?.79, U?.25 (in19): now also R?.1
- net at J?.83, U?.26 (in20): now also R?.1
- net at J?.87, U?.27 (in21): now also R?.1
- net at J?.91, U?.28 (in22): now also R?.1
- net at J?.95, U?.29 (in23): now also R?.1
- net at J?.99, U?.31 (in24): now also R?.1
- net at U?.40 (out_temp): now also U?.13 (CH5)
- net at U?.42 (out_probe_dac_5V): now also U?.12 (CH6)
- net at U?.45 (v_bg): now also U?.20 (CH0)
- net at U?.48 (vth): now also U?.19 (CH1)
- net at U?.51 (vth_t): now also U?.18 (CH2)
- net at U?.61 (out_hg): now also U?.14 (CH4)
- net at U?.62 (out_lg): now also U?.17 (CH3)
- net at U?.63 (out_probe): now also J?.1 (In)
- new net: C?.1, R?.2 (x32)
- new net: J?.5 (Pin_5), U?.1 (GPI02)
- new net: J?.7 (Pin_7), U?.2 (GPIO3)
- new net: J?.1 (Pin_1), U?.29 (GPIO0)
- new net: J?.3 (Pin_3), U?.30 (GPI01)
- new net: C?.1, RV?.1, U?.4 (REFP), U?.6 (Vout)
- new net: U?.7 (MXO), U?.8 (AINP)
- new net: R?.2, U?.5 (Trim/NR)
- new net: R?.1, RV?.2
- new net: R?.1, RV?.3
- new net +3V3: C?.1, C?.1, C?.1, C?.1, U?.2 (Vin), U?.21 (+VA), U?.28 (+VBD), U?.5 (+VA)
- new net ADC_CS_1: U?.23 (~CS)
- new net ADC_SCLK_1: U?.24 (SCLK)
- new net ADC_SDI_1: U?.25 (SDI)
- new net ADC_SDO_1: U?.26 (SDO)
- new net GNDD: J?.2 (Pin_2), J?.4 (Pin_4), J?.6 (Pin_6), J?.8 (Pin_8), U?.27 (BDGND)
- no-connect marks 0 -> 2
Other:
- note added: "20Mhz max"
- note added: "BNC"
- note added: "Check\nPackage"
- note added: "May need RF circuit here\npage 48 of ADC datasheet"
- note added: "analog I/O supply"
- note added: "digital i/o supply"
- note added: "lots of details in datasheet"
- note added: "p46"
- note added: "should these\nbe different?"
- note added: "use 0402's"
- moved on the sheet: J?A, U?C

Commit message: auto push run at Fri Apr  9 16:59:37 EDT 2021
Other:
- note added: "as long as bank voltages match\nthis will work fine, just send to LVDS bank"
- note added: "could also be 2.5V,\nmust match bank voltage of FPGA"
Changed lines of the file:
@@
 Text HLabel 9950 2350 2    50   Input ~ 0
 ADC_SCLK_1
+Text Notes 9700 800  0    50   ~ 10
+could also be 2.5V,\nmust match bank voltage of FPGA
+Text Notes 11050 2700 0    157  ~ 31
+as long as bank voltages match\nthis will work fine, just send to LVDS bank
 $EndSCHEMATC

Commit message: auto push run at Wed Apr 14 09:17:01 EDT 2021
Connections:
- net +3V3: no longer C?.1, U?.28 (+VBD)
- new net +2V5: C?.1, U?.28 (+VBD)
Other:
- note added: "SPI to LVDS bank"
- note removed: "as long as bank voltages match\nthis will work fine, just send to LVDS bank"
- note removed: "could also be 2.5V,\nmust match bank voltage of FPGA"
- note removed: "should these\nbe different?"
Changed lines of the file:
@@
 $Descr A4 11693 8268
 encoding utf-8
-Sheet 4 15
+Sheet 4 14
 Title ""
 Date ""
@@
 Wire Wire Line
 	10800 1950 10800 2050
-Text Notes 8750 1300 0    50   ~ 0
-should these\nbe different?
 Wire Wire Line
 	8800 1450 8800 1350
@@
 	8700 1250 8700 1350
 Connection ~ 8700 1350
-Wire Wire Line
-	8800 1350 9100 1350
-Wire Wire Line
-	9100 1350 9100 1450
-Connection ~ 8800 1350
 Wire Wire Line
 	8250 2750 8200 2750
@@
 $EndComp
 $Comp
-L power:+3V3 #PWR?
-U 1 1 617357E4
-P 9500 800
-F 0 "#PWR?" H 9500 650 50  0001 C CNN
-F 1 "+3V3" H 9500 950 50  0000 C CNN
-F 2 "" H 9500 800 50  0001 C CNN
-F 3 "" H 9500 800 50  0001 C CNN
-	1    9500 800
-	1    0    0    -1
-$EndComp
-$Comp
 L Device:C_Small C?
 U 1 1 61751800
@@
 Text Notes 8750 2400 0    79   ~ 16
 Check\nPackage
-Text HLabel 10400 2650 2    50   Input ~ 0
-FPGA_CCLK_0
 Text HLabel 9950 2350 2    50   Input ~ 0
 ADC_SCLK_1
-Text Notes 9700 800  0    50   ~ 10
-could also be 2.5V,\nmust match bank voltage of FPGA
-Text Notes 11050 2700 0    157  ~ 31
-as long as bank voltages match\nthis will work fine, just send to LVDS bank
+$Comp
+L power:+2V5 #PWR?
+U 1 1 6083A712
+P 9100 1350
+F 0 "#PWR?" H 9100 1200 50  0001 C CNN
+F 1 "+2V5" H 9100 1500 50  0000 C CNB
+F 2 "" H 9100 1350 50  0001 C CNN
+F 3 "" H 9100 1350 50  0001 C CNN
+	1    9100 1350
+	1    0    0    -1
+$EndComp
+Wire Wire Line
+	9100 1350 9100 1450
+$Comp
+L power:+2V5 #PWR?
+U 1 1 6086BC85
+P 9500 800
+F 0 "#PWR?" H 9500 650 50  0001 C CNN
+F 1 "+2V5" H 9500 950 50  0000 C CNB
+F 2 "" H 9500 800 50  0001 C CNN
+F 3 "" H 9500 800 50  0001 C CNN
+	1    9500 800
+	1    0    0    -1
+$EndComp
+Text Notes 10500 2600 0    50   ~ 0
+SPI to LVDS bank
 $EndSCHEMATC

Commit message: auto push run at Tue Apr 20 18:13:16 EDT 2021
Other:
- note added: "May need RF circuit here\npage 48 of ADC datasheet\n- go ahead and do it, assume\nwe meet impedance\ndo resistor and cap"
- note added: "look for citiroc output \nbuffer\n"
- note added: "this is lg"
- note removed: "May need RF circuit here\npage 48 of ADC datasheet"
Changed lines of the file:
@@
 	7200 3250 7000 3250
 Text Notes 7150 1600 0    50   ~ 0
-May need RF circuit here\npage 48 of ADC datasheet
+May need RF circuit here\npage 48 of ADC datasheet\n- go ahead and do it, assume\nwe meet impedance\ndo resistor and cap
 $Comp
 L power:GNDA #PWR?
@@
 Text Notes 10500 2600 0    50   ~ 0
 SPI to LVDS bank
+Text Notes 7050 2100 0    50   ~ 0
+this is lg
+Text Notes 7100 2600 0    50   ~ 0
+look for citiroc output \nbuffer\n
 $EndSCHEMATC

Commit message: auto push run at Wed Apr 21 10:59:57 EDT 2021
Parts:
- added C? (x6): 150p, symbol Device:C_Small
- added C?: 100n, symbol Device:C_Small
- added J?: conn, symbol Connector_Generic:Conn_02x11_Counter_Clockwise
- added J?: conn, symbol Connector_Generic:Conn_02x03_Counter_Clockwise
Connections:
- net GNDA: now also C?.2, C?.2, C?.2, C?.2, C?.2, C?.2, C?.2, J?.12 (Pin_12), J?.13 (Pin_13), J?.14 (Pin_14), J?.15 (Pin_15), J?.16 (Pin_16), J?.17 (Pin_17), J?.18 (Pin_18), J?.19 (Pin_19), J?.20 (Pin_20), J?.21 (Pin_21), J?.22 (Pin_22), J?.4 (Pin_4), J?.5 (Pin_5), J?.6 (Pin_6)
- net at U?.144 (ib_sca): now also J?.5 (Pin_5)
- net at U?.146 (ib_1nA_peak): now also J?.6 (Pin_6)
- net at U?.147 (ibo_peak): now also J?.7 (Pin_7)
- net at U?.148 (ibi_peak): now also J?.8 (Pin_8)
- net at U?.149 (in_calib): now also J?.9 (Pin_9)
- net at U?.159 (ib_dac_5V): now also J?.10 (Pin_10)
- net at U?.160 (ibi_discri_t): now also J?.11 (Pin_11)
- net at U?.39 (ib_temp): now also J?.1 (Pin_1)
- net at U?.13 (CH5), U?.40 (out_temp): now also C?.1
- net at U?.12 (CH6), U?.42 (out_probe_dac_5V): now also C?.1
- net at U?.20 (CH0), U?.45 (v_bg): now also C?.1
- net at U?.19 (CH1), U?.48 (vth): now also C?.1
- net at U?.49 (iref_dac): now also J?.2 (Pin_2)
- net at U?.50 (vref_ssh_ig): now also J?.1 (Pin_1)
- net at U?.18 (CH2), U?.51 (vth_t): now also C?.1
- net at U?.52 (vref_ssh_hg): now also J?.2 (Pin_2)
- net at U?.53 (vref_fs): now also J?.3 (Pin_3)
- net at U?.14 (CH4), U?.61 (out_hg): now also C?.1
- net at U?.17 (CH3), U?.62 (out_lg): now also C?.1
- net at U?.64 (ib_otaq): now also J?.3 (Pin_3)
- net at U?.69 (ib_rec): now also J?.4 (Pin_4)
Other:
- note added: "page 34 of DS\n"
- note added: "page 48 of DS\n"
- note added: "page33 of DS"
- note removed: "BNC"
- note removed: "May need RF circuit here\npage 48 of ADC datasheet\n- go ahead and do it, assume\nwe meet impedance\ndo resistor and cap"
- note removed: "look for citiroc output \nbuffer\n"
- note removed: "lots of details in datasheet"
- note removed: "this is lg"
- moved on the sheet: C?
