File: hardware/readout_slice/Misc.sch (KiCad schematic (older format))
At the start: 1 part

Commit message: auto push run at Wed Apr 14 09:17:01 EDT 2021
Parts:
- added U? (x2): Mars_ZX2, Package_QFP:LQFP-160_24x24mm_P0.5mm, symbol readout:Mars_ZX2
Connections:
- new net SD_i0_CD#: U?.67 (IO_B34_L17_Y19_N)
Other:
- moved on the sheet: U?I
Changed lines of the file:
@@
 $Descr A4 11693 8268
 encoding utf-8
-Sheet 14 15
+Sheet 13 14
 Title ""
 Date ""
@@
 L readout:XC7A35T-1FGG484 U?
 U 9 1 608F9D82
-P 5150 2900
+P 6600 2450
 AR Path="/605605C8/608F9D82" Ref="U?"  Part="9"
 AR Path="/608F9D82" Ref="U?"  Part="9"
 AR Path="/608F6DFA/608F9D82" Ref="U?"  Part="9"
-F 0 "U?" H 5075 3075 50  0000 C CNN
-F 1 "XC7A35T-1FGG484" H 5075 2984 50  0000 C CNN
-F 2 "" H 4050 3050 50  0001 C CNN
-F 3 "" H 4050 3050 50  0001 C CNN
-	9    5150 2900
+F 0 "U?" H 6525 2625 50  0000 C CNN
+F 1 "XC7A35T-1FGG484" H 6525 2534 50  0000 C CNN
+F 2 "" H 5500 2600 50  0001 C CNN
+F 3 "" H 5500 2600 50  0001 C CNN
+	9    6600 2450
 	1    0    0    -1
 $EndComp
-NoConn ~ 4250 3550
-NoConn ~ 4250 3350
-NoConn ~ 4250 3250
-NoConn ~ 4250 3050
-NoConn ~ 4250 2950
-NoConn ~ 5900 2950
-NoConn ~ 5900 3050
-NoConn ~ 5900 3250
-NoConn ~ 5900 3350
-NoConn ~ 5900 3550
-NoConn ~ 5900 3650
-NoConn ~ 5900 3850
-NoConn ~ 5900 3950
-NoConn ~ 5900 4150
-NoConn ~ 5900 4250
-NoConn ~ 5900 4450
-NoConn ~ 5900 4550
-NoConn ~ 5900 4750
-NoConn ~ 5900 4850
-NoConn ~ 5900 5050
-NoConn ~ 5900 5150
+NoConn ~ 5700 3100
+NoConn ~ 5700 2900
+NoConn ~ 5700 2800
+NoConn ~ 5700 2600
+NoConn ~ 5700 2500
+NoConn ~ 7350 2500
+NoConn ~ 7350 2600
+NoConn ~ 7350 2800
+NoConn ~ 7350 2900
+NoConn ~ 7350 3100
+NoConn ~ 7350 3200
+NoConn ~ 7350 3400
+NoConn ~ 7350 3500
+NoConn ~ 7350 3700
+NoConn ~ 7350 3800
+NoConn ~ 7350 4000
+NoConn ~ 7350 4100
+NoConn ~ 7350 4300
+NoConn ~ 7350 4400
+NoConn ~ 7350 4600
+NoConn ~ 7350 4700
+$Comp
+L readout:Mars_ZX2 U?
+U 5 1 60768B75
+P 1950 1600
+AR Path="/60768B75" Ref="U?"  Part="5"
+AR Path="/605605C8/60768B75" Ref="U?"  Part="5"
+AR Path="/60767BB3/60768B75" Ref="U?"  Part="5"
+AR Path="/608F6DFA/60768B75" Ref="U?"  Part="5"
+F 0 "U?" H 1550 1750 50  0000 C CNN
+F 1 "Mars_ZX2" H 1600 1650 50  0000 C CNN
+F 2 "Package_QFP:LQFP-160_24x24mm_P0.5mm" H 2000 1950 50  0001 C CNN
+F 3 "http://gauss.bu.edu/svn/emphatic-doco/Docs/CITIROC1A%20-%20Datasheet%20V2.5.pdf" H 2000 1950 50  0001 C CNN
+	5    1950 1600
+	1    0    0    -1
+$EndComp
+Text HLabel 1350 6650 0    50   Input ~ 10
+SD_i0_CD#
+$Comp
+L readout:Mars_ZX2 U?
+U 4 1 6077706D
+P 3350 4700
+AR Path="/6077706D" Ref="U?"  Part="4"
+AR Path="/605605C8/6077706D" Ref="U?"  Part="4"
+AR Path="/60768143/6077706D" Ref="U?"  Part="4"
+F 0 "U?" H 3500 4900 50  0000 C CNN
+F 1 "Mars_ZX2" H 3550 4800 50  0000 C CNN
+F 2 "Package_QFP:LQFP-160_24x24mm_P0.5mm" H 3400 5050 50  0001 C CNN
+F 3 "http://gauss.bu.edu/svn/emphatic-doco/Docs/CITIROC1A%20-%20Datasheet%20V2.5.pdf" H 3400 5050 50  0001 C CNN
+	4    3350 4700
+	1    0    0    -1
+$EndComp
+Wire Wire Line
+	2150 6650 1350 6650
 $EndSCHEMATC

Commit message: auto push run at Wed Apr 21 11:14:23 EDT 2021
Parts:
- removed U?: XC7A35T-1FGG484, symbol readout:XC7A35T-1FGG484
Connections:
- no-connect marks 21 -> 0
Changed lines of the file:
@@
 $Descr A4 11693 8268
 encoding utf-8
-Sheet 13 14
+Sheet 9 14
 Title ""
 Date ""
@@
 $EndDescr
 $Comp
-L readout:XC7A35T-1FGG484 U?
-U 9 1 608F9D82
-P 6600 2450
-AR Path="/605605C8/608F9D82" Ref="U?"  Part="9"
-AR Path="/608F9D82" Ref="U?"  Part="9"
-AR Path="/608F6DFA/608F9D82" Ref="U?"  Part="9"
-F 0 "U?" H 6525 2625 50  0000 C CNN
-F 1 "XC7A35T-1FGG484" H 6525 2534 50  0000 C CNN
-F 2 "" H 5500 2600 50  0001 C CNN
-F 3 "" H 5500 2600 50  0001 C CNN
-	9    6600 2450
-	1    0    0    -1
-$EndComp
-NoConn ~ 5700 3100
-NoConn ~ 5700 2900
-NoConn ~ 5700 2800
-NoConn ~ 5700 2600
-NoConn ~ 5700 2500
-NoConn ~ 7350 2500
-NoConn ~ 7350 2600
-NoConn ~ 7350 2800
-NoConn ~ 7350 2900
-NoConn ~ 7350 3100
-NoConn ~ 7350 3200
-NoConn ~ 7350 3400
-NoConn ~ 7350 3500
-NoConn ~ 7350 3700
-NoConn ~ 7350 3800
-NoConn ~ 7350 4000
-NoConn ~ 7350 4100
-NoConn ~ 7350 4300
-NoConn ~ 7350 4400
-NoConn ~ 7350 4600
-NoConn ~ 7350 4700
-$Comp
 L readout:Mars_ZX2 U?
