File: hardware/readout_slice/FPGA-3V3-Bank.sch (KiCad schematic (older format))
At the start: 8 parts

Commit message: auto push run at Fri Apr  9 14:02:10 EDT 2021
Connections:
- net labels added: NOR32T_oc_1, NOR32_oc_1, OR32_1
- wire segments 71 -> 74
Other:
- note added: "note colors have different Vf"
- note added: "regular LEDS in a few colors - red, green. orange"
- note added: "think 1mA"
- note added: "use less than half LED specified current\n"
Changed lines of the file:
@@
 $Descr A4 11693 8268
 encoding utf-8
-Sheet 16 16
+Sheet 13 15
 Title ""
 Date ""
@@
 	1    0    0    -1
 $EndComp
-Text HLabel 9350 3750 2    50   Input ~ 0
+Text HLabel 8850 3950 2    50   Input ~ 0
 FPGA_tx
-Text HLabel 9350 3850 2    50   Input ~ 0
+Text HLabel 8850 4050 2    50   Input ~ 0
 FPGA_rx
 Wire Wire Line
-	9350 3750 9250 3750
-Wire Wire Line
-	9250 3850 9350 3850
-Text Notes 9200 3650 0    50   ~ 0
+	8850 3950 8750 3950
+Wire Wire Line
+	8750 4050 8850 4050
+Text Notes 8700 3850 0    50   ~ 0
 to sparkfun
-Text HLabel 2650 2800 0    50   Input ~ 0
+Text HLabel 3550 2650 0    50   Input ~ 0
 resetb_pa
-Text HLabel 2650 2900 0    50   Input ~ 0
+Text HLabel 3550 2750 0    50   Input ~ 0
 rstb_PSC
-Text HLabel 2650 3000 0    50   Input ~ 0
+Text HLabel 3550 2850 0    50   Input ~ 0
 pwr_on
 Wire Wire Line
-	2800 3000 2650 3000
-Wire Wire Line
-	2800 2900 2650 2900
-Wire Wire Line
-	2800 2800 2650 2800
-Text HLabel 2650 3100 0    50   Input ~ 0
+	3700 2850 3550 2850
+Wire Wire Line
+	3700 2750 3550 2750
+Wire Wire Line
+	3700 2650 3550 2650
+Text HLabel 3550 2950 0    50   Input ~ 0
 PS_global_trig
-Text HLabel 2650 3200 0    50   Input ~ 0
+Text HLabel 3550 3050 0    50   Input ~ 0
 PS_modeb_ext
-Text HLabel 2650 3800 0    50   Input ~ 0
+Text HLabel 3550 3650 0    50   Input ~ 0
 load_sc_1
-Text HLabel 2650 3700 0    50   Input ~ 0
+Text HLabel 3550 3550 0    50   Input ~ 0
 select_1
-Text HLabel 2650 3300 0    50   Input ~ 0
+Text HLabel 3550 3150 0    50   Input ~ 0
 hold_lg
-Text HLabel 2650 3400 0    50   Input ~ 0
+Text HLabel 3550 3250 0    50   Input ~ 0
 hold_hg
-Text HLabel 2650 3900 0    50   Input ~ 0
+Text HLabel 3550 3750 0    50   Input ~ 0
 srin_read_1
-Text HLabel 2650 4000 0    50   Input ~ 0
+Text HLabel 3550 3850 0    50   Input ~ 0
 clk_read_1
-Text HLabel 2650 4100 0    50   Input ~ 0
+Text HLabel 3550 3950 0    50   Input ~ 0
 resetb_read_1
-Text HLabel 2650 4200 0    50   Input ~ 0
+Text HLabel 3550 4050 0    50   Input ~ 0
 srin_sc_1
-Text HLabel 2650 4300 0    50   Input ~ 0
+Text HLabel 3550 4150 0    50   Input ~ 0
 clk_sr_1
-Text HLabel 2650 4400 0    50   Input ~ 0
+Text HLabel 3550 4250 0    50   Input ~ 0
 rstb_sr_1
 Wire Wire Line
-	2800 3900 2650 3900
-Wire Wire Line
-	2800 4000 2650 4000
-Wire Wire Line
-	2650 4100 2800 4100
-Wire Wire Line
-	2800 4200 2650 4200
-Wire Wire Line
-	2650 4300 2800 4300
-Wire Wire Line
-	2800 4400 2650 4400
-Wire Wire Line
-	2650 3100 2800 3100
-Wire Wire Line
-	2800 3200 2650 3200
-Wire Wire Line
-	2650 3300 2800 3300
-Wire Wire Line
-	2800 3400 2650 3400
-Wire Wire Line
-	2800 3800 2650 3800
-Wire Wire Line
-	2650 3700 2800 3700
-Text Notes 2000 2700 0    50   ~ 0
+	3700 3750 3550 3750
+Wire Wire Line
+	3700 3850 3550 3850
+Wire Wire Line
+	3550 3950 3700 3950
+Wire Wire Line
+	3700 4050 3550 4050
+Wire Wire Line
+	3550 4150 3700 4150
+Wire Wire Line
+	3700 4250 3550 4250
+Wire Wire Line
+	3550 2950 3700 2950
+Wire Wire Line
+	3700 3050 3550 3050
+Wire Wire Line
+	3550 3150 3700 3150
+Wire Wire Line
+	3700 3250 3550 3250
+Wire Wire Line
+	3700 3650 3550 3650
+Wire Wire Line
+	3550 3550 3700 3550
+Text Notes 2900 2550 0    50   ~ 0
 Shared Citiroc Controls
-Text Notes 2200 3600 0    50   ~ 0
+Text Notes 3100 3450 0    50   ~ 0
 Citiroc 1 Controls
-Text HLabel 2650 5100 0    50   Input ~ 0
+Text HLabel 3550 5250 0    50   Input ~ 0
 load_sc_2
-Text HLabel 2650 5000 0    50   Input ~ 0
+Text HLabel 3550 5150 0    50   Input ~ 0
 select_2
-Text HLabel 2650 5200 0    50   Input ~ 0
+Text HLabel 3550 5350 0    50   Input ~ 0
 srin_read_2
-Text HLabel 2650 5300 0    50   Input ~ 0
+Text HLabel 3550 5450 0    50   Input ~ 0
 clk_read_2
-Text HLabel 2650 5400 0    50   Input ~ 0
+Text HLabel 3550 5550 0    50   Input ~ 0
 resetb_read_2
-Text HLabel 2650 5500 0    50   Input ~ 0
+Text HLabel 3550 5650 0    50   Input ~ 0
 srin_sc_2
-Text HLabel 2650 5600 0    50   Input ~ 0
+Text HLabel 3550 5750 0    50   Input ~ 0
 clk_sr_2
-Text HLabel 2650 5700 0    50   Input ~ 0
+Text HLabel 3550 5850 0    50   Input ~ 0
 rstb_sr_2
 Wire Wire Line
-	2800 5200 2650 5200
-Wire Wire Line
-	2800 5300 2650 5300
-Wire Wire Line
-	2650 5400 2800 5400
-Wire Wire Line
-	2800 5500 2650 5500
-Wire Wire Line
-	2650 5600 2800 5600
-Wire Wire Line
-	2800 5700 2650 5700
-Wire Wire Line
-	2800 5100 2650 5100
-Wire Wire Line
-	2650 5000 2800 5000
-Text Notes 2200 4900 0    50   ~ 0
+	3700 5350 3550 5350
+Wire Wire Line
+	3700 5450 3550 5450
+Wire Wire Line
+	3550 5550 3700 5550
+Wire Wire Line
+	3700 5650 3550 5650
+Wire Wire Line
+	3550 5750 3700 5750
+Wire Wire Line
+	3700 5850 3550 5850
+Wire Wire Line
+	3700 5250 3550 5250
+Wire Wire Line
+	3550 5150 3700 5150
+Text Notes 3100 5050 0    50   ~ 0
 Citiroc 2 Controls
-Text HLabel 2650 4500 0    50   Input ~ 0
+Text HLabel 3550 4350 0    50   Input ~ 0
 srout_read_1
-Text HLabel 2650 4600 0    50   Input ~ 0
+Text HLabel 3550 4450 0    50   Input ~ 0
 srout_sc_1
 Wire Wire Line
-	2650 4500 2800 4500
-Wire Wire Line
-	2650 4600 2800 4600
-Text HLabel 2650 4700 0    50   Input ~ 0
+	3550 4350 3700 4350
+Wire Wire Line
+	3550 4450 3700 4450
+Text HLabel 3550 4550 0    50   Input ~ 0
 dig_out_1
 Wire Wire Line
-	2650 4700 2800 4700
-Text HLabel 2650 5800 0    50   Input ~ 0
+	3550 4550 3700 4550
+Text HLabel 3550 5950 0    50   Input ~ 0
 srout_read_2
-Text HLabel 2650 5900 0    50   Input ~ 0
+Text HLabel 3550 6050 0    50   Input ~ 0
 srout_sc_2
 Wire Wire Line
-	2650 5800 2800 5800
-Wire Wire Line
-	2650 5900 2800 5900
-Text HLabel 2650 6000 0    50   Input ~ 0
+	3550 5950 3700 5950
+Wire Wire Line
+	3550 6050 3700 6050
+Text HLabel 3550 6150 0    50   Input ~ 0
 dig_out_2
 Wire Wire Line
-	2650 6000 2800 6000
+	3550 6150 3700 6150
+Text Notes 5000 1150 0    157  ~ 31
+regular LEDS in a few colors - red, green. orange
+Text Notes 5950 1500 0    157  ~ 31
+use less than half LED specified current\n
+Text Notes 8150 1850 0    157  ~ 31
+think 1mA
+Text Notes 7900 2150 0    79   ~ 16
+note colors have different Vf
+Wire Wire Line
+	3700 4850 3550 4850
+Wire Wire Line
+	3700 4750 3550 4750
+Wire Wire Line
+	3700 4650 3550 4650
+Text HLabel 3550 4850 0    50   Input ~ 0
+NOR32T_oc_1
+Text HLabel 3550 4750 0    50   Input ~ 0
+NOR32_oc_1
+Text HLabel 3550 4650 0    50   Input ~ 0
+OR32_1
 $EndSCHEMATC

Commit message: auto push run at Fri Apr  9 14:13:27 EDT 2021
Connections:
- net labels added: NOR32T_oc_2, NOR32_oc_2, OR32_2
- wire segments 74 -> 77
Changed lines of the file:
@@
 $Descr A4 11693 8268
 encoding utf-8
-Sheet 13 15
+Sheet 15 15
 Title ""
 Date ""
@@
 Text HLabel 3550 4650 0    50   Input ~ 0
 OR32_1
+Wire Wire Line
+	3700 6450 3550 6450
+Wire Wire Line
+	3700 6350 3550 6350
+Wire Wire Line
+	3700 6250 3550 6250
+Text HLabel 3550 6450 0    50   Input ~ 0
+NOR32T_oc_2
+Text HLabel 3550 6350 0    50   Input ~ 0
+NOR32_oc_2
+Text HLabel 3550 6250 0    50   Input ~ 0
+OR32_2
 $EndSCHEMATC

Commit message: auto push run at Wed Apr 14 11:08:32 EDT 2021
Connections:
- net labels added: 3v3_GPIO1, 3v3_GPIO2, 3v3_GPIO3, 3v3_GPIO4
- wire segments 77 -> 81
Other:
- note added: "to GPIO"
Changed lines of the file:
@@
 $Descr A4 11693 8268
 encoding utf-8
-Sheet 15 14
+Sheet 14 14
 Title ""
 Date ""
@@
 Text HLabel 3550 6250 0    50   Input ~ 0
 OR32_2
+Text HLabel 8900 4350 2    50   Input ~ 0
+3v3_GPIO1
+Text HLabel 8900 4450 2    50   Input ~ 0
+3v3_GPIO2
+Text HLabel 8900 4550 2    50   Input ~ 0
+3v3_GPIO3
+Text HLabel 8900 4650 2    50   Input ~ 0
+3v3_GPIO4
+Wire Wire Line
+	8900 4350 8750 4350
+Wire Wire Line
+	8900 4450 8750 4450
+Wire Wire Line
+	8900 4550 8750 4550
+Wire Wire Line
+	8900 4650 8750 4650
+Text Notes 8700 4300 0    50   ~ 0
+to GPIO
 $EndSCHEMATC

Commit message: auto push run at Wed Apr 21 10:59:57 EDT 2021
Connections:
- net labels removed: dig_out_1, dig_out_2
- wire segments 81 -> 79
Changed lines of the file:
@@
 $Descr A4 11693 8268
 encoding utf-8
-Sheet 14 14
+Sheet 13 14
 Title ""
 Date ""
@@
 	1    0    0    -1
 $EndComp
-Text HLabel 8850 3950 2    50   Input ~ 0
+Text HLabel 7150 2600 2    50   Input ~ 0
 FPGA_tx
-Text HLabel 8850 4050 2    50   Input ~ 0
+Text HLabel 7150 2700 2    50   Input ~ 0
 FPGA_rx
 Wire Wire Line
-	8850 3950 8750 3950
-Wire Wire Line
-	8750 4050 8850 4050
-Text Notes 8700 3850 0    50   ~ 0
+	7150 2600 7050 2600
+Wire Wire Line
+	7050 2700 7150 2700
+Text Notes 7000 2500 0    50   ~ 0
 to sparkfun
-Text HLabel 3550 2650 0    50   Input ~ 0
+Text HLabel 4250 2400 0    50   Input ~ 0
 resetb_pa
-Text HLabel 3550 2750 0    50   Input ~ 0
+Text HLabel 4250 2500 0    50   Input ~ 0
 rstb_PSC
-Text HLabel 3550 2850 0    50   Input ~ 0
+Text HLabel 4250 2700 0    50   Input ~ 0
 pwr_on
 Wire Wire Line
-	3700 2850 3550 2850
-Wire Wire Line
-	3700 2750 3550 2750
-Wire Wire Line
-	3700 2650 3550 2650
-Text HLabel 3550 2950 0    50   Input ~ 0
+	4400 2700 4250 2700
+Wire Wire Line
+	4400 2500 4250 2500
+Wire Wire Line
+	4400 2400 4250 2400
+Text HLabel 4250 2800 0    50   Input ~ 0
 PS_global_trig
-Text HLabel 3550 3050 0    50   Input ~ 0
+Text HLabel 4250 3000 0    50   Input ~ 0
 PS_modeb_ext
-Text HLabel 3550 3650 0    50   Input ~ 0
+Text HLabel 4250 3600 0    50   Input ~ 0
 load_sc_1
-Text HLabel 3550 3550 0    50   Input ~ 0
+Text HLabel 4250 3400 0    50   Input ~ 0
 select_1
-Text HLabel 3550 3150 0    50   Input ~ 0
+Text HLabel 4250 3100 0    50   Input ~ 0
 hold_lg
-Text HLabel 3550 3250 0    50   Input ~ 0
+Text HLabel 4250 3300 0    50   Input ~ 0
 hold_hg
-Text HLabel 3550 3750 0    50   Input ~ 0
+Text HLabel 4250 3700 0    50   Input ~ 0
 srin_read_1
-Text HLabel 3550 3850 0    50   Input ~ 0
+Text HLabel 4250 3900 0    50   Input ~ 0
 clk_read_1
-Text HLabel 3550 3950 0    50   Input ~ 0
+Text HLabel 4250 4000 0    50   Input ~ 0
 resetb_read_1
-Text HLabel 3550 4050 0    50   Input ~ 0
+Text HLabel 4250 4200 0    50   Input ~ 0
 srin_sc_1
-Text HLabel 3550 4150 0    50   Input ~ 0
+Text HLabel 4250 4300 0    50   Input ~ 0
 clk_sr_1
-Text HLabel 3550 4250 0    50   Input ~ 0
+Text HLabel 4250 4500 0    50   Input ~ 0
 rstb_sr_1
 Wire Wire Line
-	3700 3750 3550 3750
-Wire Wire Line
-	3700 3850 3550 3850
-Wire Wire Line
-	3550 3950 3700 3950
-Wire Wire Line
-	3700 4050 3550 4050
-Wire Wire Line
-	3550 4150 3700 4150
-Wire Wire Line
-	3700 4250 3550 4250
-Wire Wire Line
-	3550 2950 3700 2950
-Wire Wire Line
-	3700 3050 3550 3050
-Wire Wire Line
-	3550 3150 3700 3150
-Wire Wire Line
-	3700 3250 3550 3250
-Wire Wire Line
-	3700 3650 3550 3650
-Wire Wire Line
-	3550 3550 3700 3550
-Text Notes 2900 2550 0    50   ~ 0
+	4400 3700 4250 3700
+Wire Wire Line
+	4400 3900 4250 3900
+Wire Wire Line
+	4250 4000 4400 4000
+Wire Wire Line
+	4400 4200 4250 4200
+Wire Wire Line
+	4250 4300 4400 4300
+Wire Wire Line
+	4400 4500 4250 4500
+Wire Wire Line
+	4250 2800 4400 2800
+Wire Wire Line
+	4400 3000 4250 3000
+Wire Wire Line
+	4250 3100 4400 3100
+Wire Wire Line
+	4400 3300 4250 3300
+Wire Wire Line
+	4400 3600 4250 3600
+Wire Wire Line
+	4250 3400 4400 3400
+Text Notes 3600 2300 0    50   ~ 0
 Shared Citiroc Controls
-Text Notes 3100 3450 0    50   ~ 0
+Text Notes 3250 3400 0    50   ~ 0
 Citiroc 1 Controls
-Text HLabel 3550 5250 0    50   Input ~ 0
+Text HLabel 4250 5500 0    50   Input ~ 0
 load_sc_2
-Text HLabel 3550 5150 0    50   Input ~ 0
+Text HLabel 4250 5400 0    50   Input ~ 0
 select_2
-Text HLabel 3550 5350 0    50   Input ~ 0
+Text HLabel 4250 5700 0    50   Input ~ 0
 srin_read_2
-Text HLabel 3550 5450 0    50   Input ~ 0
+Text HLabel 4250 5800 0    50   Input ~ 0
 clk_read_2
-Text HLabel 3550 5550 0    50   Input ~ 0
+Text HLabel 7200 6000 2    50   Input ~ 0
 resetb_read_2
-Text HLabel 3550 5650 0    50   Input ~ 0
+Text HLabel 7200 5700 2    50   Input ~ 0
 srin_sc_2
-Text HLabel 3550 5750 0    50   Input ~ 0
+Text HLabel 7200 5900 2    50   Input ~ 0
 clk_sr_2
-Text HLabel 3550 5850 0    50   Input ~ 0
+Text HLabel 7200 5600 2    50   Input ~ 0
 rstb_sr_2
 Wire Wire Line
-	3700 5350 3550 5350
-Wire Wire Line
-	3700 5450 3550 5450
-Wire Wire Line
-	3550 5550 3700 5550
-Wire Wire Line
-	3700 5650 3550 5650
-Wire Wire Line
-	3550 5750 3700 5750
-Wire Wire Line
-	3700 5850 3550 5850
-Wire Wire Line
-	3700 5250 3550 5250
-Wire Wire Line
-	3550 5150 3700 5150
-Text Notes 3100 5050 0    50   ~ 0
+	4400 5700 4250 5700
+Wire Wire Line
+	4400 5800 4250 5800
+Wire Wire Line
+	7200 6000 7050 6000
+Wire Wire Line
+	7050 5700 7200 5700
+Wire Wire Line
+	7200 5900 7050 5900
+Wire Wire Line
+	7050 5600 7200 5600
+Wire Wire Line
+	4400 5500 4250 5500
+Wire Wire Line
+	4250 5400 4400 5400
+Text Notes 3450 5350 0    50   ~ 0
 Citiroc 2 Controls
-Text HLabel 3550 4350 0    50   Input ~ 0
+Text HLabel 4250 4600 0    50   Input ~ 0
 srout_read_1
-Text HLabel 3550 4450 0    50   Input ~ 0
+Text HLabel 4250 4800 0    50   Input ~ 0
 srout_sc_1
 Wire Wire Line
-	3550 4350 3700 4350
-Wire Wire Line
-	3550 4450 3700 4450
-Text HLabel 3550 4550 0    50   Input ~ 0
-dig_out_1
-Wire Wire Line
-	3550 4550 3700 4550
-Text HLabel 3550 5950 0    50   Input ~ 0
+	4250 4600 4400 4600
+Wire Wire Line
+	4250 4800 4400 4800
+Text HLabel 7200 5300 2    50   Input ~ 0
 srout_read_2
-Text HLabel 3550 6050 0    50   Input ~ 0
+Text HLabel 7200 5400 2    50   Input ~ 0
 srout_sc_2
 Wire Wire Line
-	3550 5950 3700 5950
-Wire Wire Line
-	3550 6050 3700 6050
-Text HLabel 3550 6150 0    50   Input ~ 0
-dig_out_2
-Wire Wire Line
-	3550 6150 3700 6150
+	7200 5300 7050 5300
+Wire Wire Line
+	7200 5400 7050 5400
 Text Notes 5000 1150 0    157  ~ 31
 regular LEDS in a few colors - red, green. orange
@@
 note colors have different Vf
 Wire Wire Line
-	3700 4850 3550 4850
-Wire Wire Line
-	3700 4750 3550 4750
-Wire Wire Line
-	3700 4650 3550 4650
-Text HLabel 3550 4850 0    50   Input ~ 0
+	4400 5200 4250 5200
+Wire Wire Line
+	4400 5100 4250 5100
+Wire Wire Line
+	4400 4900 4250 4900
+Text HLabel 4250 5200 0    50   Input ~ 0
 NOR32T_oc_1
-Text HLabel 3550 4750 0    50   Input ~ 0
+Text HLabel 4250 5100 0    50   Input ~ 0
 NOR32_oc_1
-Text HLabel 3550 4650 0    50   Input ~ 0
+Text HLabel 4250 4900 0    50   Input ~ 0
 OR32_1
 Wire Wire Line
-	3700 6450 3550 6450
-Wire Wire Line
-	3700 6350 3550 6350
-Wire Wire Line
-	3700 6250 3550 6250
-Text HLabel 3550 6450 0    50   Input ~ 0
+	7050 5000 7200 5000
+Wire Wire Line
+	7050 4800 7200 4800
+Wire Wire Line
+	7050 5100 7200 5100
+Text HLabel 7200 5000 2    50   Input ~ 0
 NOR32T_oc_2
-Text HLabel 3550 6350 0    50   Input ~ 0
+Text HLabel 7200 4800 2    50   Input ~ 0
 NOR32_oc_2
-Text HLabel 3550 6250 0    50   Input ~ 0
+Text HLabel 7200 5100 2    50   Input ~ 0
 OR32_2
-Text HLabel 8900 4350 2    50   Input ~ 0
+Text HLabel 7200 2850 2    50   Input ~ 0
 3v3_GPIO1
-Text HLabel 8900 4450 2    50   Input ~ 0
+Text HLabel 7200 2950 2    50   Input ~ 0
 3v3_GPIO2
-Text HLabel 8900 4550 2    50   Input ~ 0
+Text HLabel 7200 3200 2    50   Input ~ 0
 3v3_GPIO3
-Text HLabel 8900 4650 2    50   Input ~ 0
+Text HLabel 7200 3300 2    50   Input ~ 0
 3v3_GPIO4
 Wire Wire Line
-	8900 4350 8750 4350
-Wire Wire Line
-	8900 4450 8750 4450
-Wire Wire Line
-	8900 4550 8750 4550
-Wire Wire Line
-	8900 4650 8750 4650
-Text Notes 8700 4300 0    50   ~ 0
+	7200 2850 7050 2850
+Wire Wire Line
+	7200 2950 7050 2950
+Wire Wire Line
+	7200 3200 7050 3200
+Wire Wire Line
+	7200 3300 7050 3300
+Text Notes 7000 2800 0    50   ~ 0
 to GPIO
 $EndSCHEMATC

Commit message: auto push run at Wed Apr 21 11:14:23 EDT 2021
Changed lines of the file:
@@
 $Descr A4 11693 8268
 encoding utf-8
-Sheet 13 14
+Sheet 10 14
 Title ""
 Date ""
@@
 	1    0    0    -1
 $EndComp
-Text HLabel 7150 2600 2    50   Input ~ 0
+Text HLabel 6950 2600 2    50   Input ~ 0
 FPGA_tx
-Text HLabel 7150 2700 2    50   Input ~ 0
+Text HLabel 6950 2700 2    50   Input ~ 0
 FPGA_rx
 Wire Wire Line
-	7150 2600 7050 2600
-Wire Wire Line
-	7050 2700 7150 2700
-Text Notes 7000 2500 0    50   ~ 0
+	6950 2600 6850 2600
+Wire Wire Line
+	6850 2700 6950 2700
+Text Notes 6800 2500 0    50   ~ 0
 to sparkfun
-Text HLabel 4250 2400 0    50   Input ~ 0
+Text HLabel 4450 2400 0    50   Input ~ 0
 resetb_pa
-Text HLabel 4250 2500 0    50   Input ~ 0
+Text HLabel 4450 2500 0    50   Input ~ 0
 rstb_PSC
-Text HLabel 4250 2700 0    50   Input ~ 0
+Text HLabel 4450 2700 0    50   Input ~ 0
 pwr_on
 Wire Wire Line
-	4400 2700 4250 2700
-Wire Wire Line
-	4400 2500 4250 2500
-Wire Wire Line
-	4400 2400 4250 2400
-Text HLabel 4250 2800 0    50   Input ~ 0
+	4600 2700 4450 2700
+Wire Wire Line
+	4600 2500 4450 2500
+Wire Wire Line
+	4600 2400 4450 2400
+Text HLabel 4450 2800 0    50   Input ~ 0
 PS_global_trig
-Text HLabel 4250 3000 0    50   Input ~ 0
+Text HLabel 4450 3000 0    50   Input ~ 0
 PS_modeb_ext
-Text HLabel 4250 3600 0    50   Input ~ 0
+Text HLabel 4450 3600 0    50   Input ~ 0
 load_sc_1
-Text HLabel 4250 3400 0    50   Input ~ 0
+Text HLabel 4450 3400 0    50   Input ~ 0
 select_1
-Text HLabel 4250 3100 0    50   Input ~ 0
+Text HLabel 4450 3100 0    50   Input ~ 0
 hold_lg
-Text HLabel 4250 3300 0    50   Input ~ 0
+Text HLabel 4450 3300 0    50   Input ~ 0
 hold_hg
-Text HLabel 4250 3700 0    50   Input ~ 0
+Text HLabel 4450 3700 0    50   Input ~ 0
 srin_read_1
-Text HLabel 4250 3900 0    50   Input ~ 0
+Text HLabel 4450 3900 0    50   Input ~ 0
 clk_read_1
-Text HLabel 4250 4000 0    50   Input ~ 0
+Text HLabel 4450 4000 0    50   Input ~ 0
 resetb_read_1
-Text HLabel 4250 4200 0    50   Input ~ 0
+Text HLabel 4450 4200 0    50   Input ~ 0
 srin_sc_1
-Text HLabel 4250 4300 0    50   Input ~ 0
+Text HLabel 4450 4300 0    50   Input ~ 0
 clk_sr_1
-Text HLabel 4250 4500 0    50   Input ~ 0
+Text HLabel 4450 4500 0    50   Input ~ 0
 rstb_sr_1
 Wire Wire Line
-	4400 3700 4250 3700
-Wire Wire Line
-	4400 3900 4250 3900
-Wire Wire Line
-	4250 4000 4400 4000
-Wire Wire Line
-	4400 4200 4250 4200
-Wire Wire Line
-	4250 4300 4400 4300
-Wire Wire Line
-	4400 4500 4250 4500
-Wire Wire Line
-	4250 2800 4400 2800
-Wire Wire Line
-	4400 3000 4250 3000
-Wire Wire Line
-	4250 3100 4400 3100
-Wire Wire Line
-	4400 3300 4250 3300
-Wire Wire Line
-	4400 3600 4250 3600
-Wire Wire Line
-	4250 3400 4400 3400
-Text Notes 3600 2300 0    50   ~ 0
+	4600 3700 4450 3700
+Wire Wire Line
+	4600 3900 4450 3900
+Wire Wire Line
+	4450 4000 4600 4000
+Wire Wire Line
+	4600 4200 4450 4200
+Wire Wire Line
+	4450 4300 4600 4300
+Wire Wire Line
+	4600 4500 4450 4500
+Wire Wire Line
+	4450 2800 4600 2800
+Wire Wire Line
+	4600 3000 4450 3000
+Wire Wire Line
+	4450 3100 4600 3100
+Wire Wire Line
+	4600 3300 4450 3300
+Wire Wire Line
+	4600 3600 4450 3600
+Wire Wire Line
+	4450 3400 4600 3400
+Text Notes 3800 2300 0    50   ~ 0
 Shared Citiroc Controls
-Text Notes 3250 3400 0    50   ~ 0
+Text Notes 3450 3400 0    50   ~ 0
 Citiroc 1 Controls
-Text HLabel 4250 5500 0    50   Input ~ 0
+Text HLabel 4450 5500 0    50   Input ~ 0
 load_sc_2
-Text HLabel 4250 5400 0    50   Input ~ 0
+Text HLabel 4450 5400 0    50   Input ~ 0
 select_2
-Text HLabel 4250 5700 0    50   Input ~ 0
+Text HLabel 4450 5700 0    50   Input ~ 0
 srin_read_2
-Text HLabel 4250 5800 0    50   Input ~ 0
+Text HLabel 4450 5800 0    50   Input ~ 0
 clk_read_2
-Text HLabel 7200 6000 2    50   Input ~ 0
+Text HLabel 7000 6000 2    50   Input ~ 0
 resetb_read_2
-Text HLabel 7200 5700 2    50   Input ~ 0
+Text HLabel 7000 5700 2    50   Input ~ 0
 srin_sc_2
-Text HLabel 7200 5900 2    50   Input ~ 0
+Text HLabel 7000 5900 2    50   Input ~ 0
 clk_sr_2
-Text HLabel 7200 5600 2    50   Input ~ 0
+Text HLabel 7000 5600 2    50   Input ~ 0
 rstb_sr_2
 Wire Wire Line
-	4400 5700 4250 5700
-Wire Wire Line
-	4400 5800 4250 5800
-Wire Wire Line
-	7200 6000 7050 6000
-Wire Wire Line
-	7050 5700 7200 5700
-Wire Wire Line
-	7200 5900 7050 5900
-Wire Wire Line
-	7050 5600 7200 5600
-Wire Wire Line
-	4400 5500 4250 5500
-Wire Wire Line
-	4250 5400 4400 5400
-Text Notes 3450 5350 0    50   ~ 0
+	4600 5700 4450 5700
+Wire Wire Line
+	4600 5800 4450 5800
+Wire Wire Line
+	7000 6000 6850 6000
+Wire Wire Line
+	6850 5700 7000 5700
+Wire Wire Line
+	7000 5900 6850 5900
+Wire Wire Line
+	6850 5600 7000 5600
+Wire Wire Line
+	4600 5500 4450 5500
+Wire Wire Line
+	4450 5400 4600 5400
+Text Notes 3650 5350 0    50   ~ 0
 Citiroc 2 Controls
-Text HLabel 4250 4600 0    50   Input ~ 0
+Text HLabel 4450 4600 0    50   Input ~ 0
 srout_read_1
-Text HLabel 4250 4800 0    50   Input ~ 0
+Text HLabel 4450 4800 0    50   Input ~ 0
 srout_sc_1
 Wire Wire Line
-	4250 4600 4400 4600
-Wire Wire Line
-	4250 4800 4400 4800
-Text HLabel 7200 5300 2    50   Input ~ 0
+	4450 4600 4600 4600
+Wire Wire Line
+	4450 4800 4600 4800
+Text HLabel 7000 5300 2    50   Input ~ 0
 srout_read_2
-Text HLabel 7200 5400 2    50   Input ~ 0
+Text HLabel 7000 5400 2    50   Input ~ 0
 srout_sc_2
 Wire Wire Line
-	7200 5300 7050 5300
-Wire Wire Line
-	7200 5400 7050 5400
+	7000 5300 6850 5300
+Wire Wire Line
+	7000 5400 6850 5400
 Text Notes 5000 1150 0    157  ~ 31
 regular LEDS in a few colors - red, green. orange
@@
 note colors have different Vf
 Wire Wire Line
-	4400 5200 4250 5200
-Wire Wire Line
-	4400 5100 4250 5100
-Wire Wire Line
-	4400 4900 4250 4900
-Text HLabel 4250 5200 0    50   Input ~ 0
+	4600 5200 4450 5200
+Wire Wire Line
+	4600 5100 4450 5100
+Wire Wire Line
+	4600 4900 4450 4900
+Text HLabel 4450 5200 0    50   Input ~ 0
 NOR32T_oc_1
-Text HLabel 4250 5100 0    50   Input ~ 0
+Text HLabel 4450 5100 0    50   Input ~ 0
 NOR32_oc_1
-Text HLabel 4250 4900 0    50   Input ~ 0
+Text HLabel 4450 4900 0    50   Input ~ 0
 OR32_1
 Wire Wire Line
-	7050 5000 7200 5000
-Wire Wire Line
-	7050 4800 7200 4800
-Wire Wire Line
-	7050 5100 7200 5100
-Text HLabel 7200 5000 2    50   Input ~ 0
+	6850 5000 7000 5000
+Wire Wire Line
+	6850 4800 7000 4800
+Wire Wire Line
+	6850 5100 7000 5100
+Text HLabel 7000 5000 2    50   Input ~ 0
 NOR32T_oc_2
-Text HLabel 7200 4800 2    50   Input ~ 0
+Text HLabel 7000 4800 2    50   Input ~ 0
 NOR32_oc_2
-Text HLabel 7200 5100 2    50   Input ~ 0
+Text HLabel 7000 5100 2    50   Input ~ 0
 OR32_2
-Text HLabel 7200 2850 2    50   Input ~ 0
+Text HLabel 7000 2900 2    50   Input ~ 0
 3v3_GPIO1
-Text HLabel 7200 2950 2    50   Input ~ 0
+Text HLabel 7000 3000 2    50   Input ~ 0
 3v3_GPIO2
-Text HLabel 7200 3200 2    50   Input ~ 0
+Text HLabel 7000 3200 2    50   Input ~ 0
 3v3_GPIO3
-Text HLabel 7200 3300 2    50   Input ~ 0
+Text HLabel 7000 3300 2    50   Input ~ 0
 3v3_GPIO4
 Wire Wire Line
-	7200 2850 7050 2850
-Wire Wire Line
-	7200 2950 7050 2950
-Wire Wire Line
-	7200 3200 7050 3200
-Wire Wire Line
-	7200 3300 7050 3300
-Text Notes 7000 2800 0    50   ~ 0
+	7000 2900 6850 2900
+Wire Wire Line
+	7000 3000 6850 3000
+Wire Wire Line
+	7000 3200 6850 3200
+Wire Wire Line
+	7000 3300 6850 3300
+Text Notes 6800 2850 0    50   ~ 0
 to GPIO
 $EndSCHEMATC
