File: hardware/readout_slice/FPGA_SERDES.sch (KiCad schematic (older format))
At the start: 21 parts

Commit message: auto push run at Wed Apr 28 10:51:45 EDT 2021
Parts:
- added U?: Vcc0, symbol readout:Vcc0
- added U?: VccSFP, symbol readout:VccSFP
Connections:
- net VCC: now reaches R?.1, R?.1, R?.1, R?.1, R?.1
- net VCC: now also C?.2, C?.2, L?.2, L?.2, U?.1 (VCC), U?.1 (VCC)
- no-connect marks 9 -> 10
Other:
- note removed: "VCCSFP"
- note removed: "VCC_0"
Changed lines of the file:
@@
 $Descr A4 11693 8268
 encoding utf-8
-Sheet 11 11
+Sheet 9 11
 Title ""
 Date ""
@@
 	7450 2900 7450 2600
 Connection ~ 7450 2900
-Text Notes 7600 2600 2    118  ~ 0
-VCC_0
 $Comp
 L Device:L L?
@@
 Wire Wire Line
 	8250 2450 8450 2450
-Text Notes 7900 2350 0    118  ~ 0
-VCCSFP
 Wire Wire Line
 	8150 2450 8150 2350
@@
 	7950 3250 7750 3250
 Connection ~ 7950 3250
-Text Notes 9050 3850 0    118  ~ 24
+Text Notes 9000 3950 0    118  ~ 24
 NEED to do cage
 Wire Wire Line
@@
 Text Notes 6550 4950 0    50   ~ 10
 to vcco bank
+$Comp
+L readout:Vcc0 U?
+U 1 1 62C7AC21
+P 7450 2500
+F 0 "U?" H 7450 2500 79  0001 C CNN
+F 1 "Vcc0" H 7350 2550 47  0000 L CNB
+F 2 "" H 7450 2500 79  0001 C CNN
+F 3 "" H 7450 2500 79  0001 C CNN
+	1    7450 2500
+	1    0    0    -1
+$EndComp
+$Comp
+L readout:VccSFP U?
+U 1 1 62C7E003
+P 8150 2250
+F 0 "U?" H 8150 2250 79  0001 C CNN
+F 1 "VccSFP" H 8050 2300 47  0000 L CNB
+F 2 "" H 8150 2250 79  0001 C CNN
+F 3 "" H 8150 2250 79  0001 C CNN
+	1    8150 2250
+	1    0    0    -1
+$EndComp
+NoConn ~ 6000 2450
 $EndSCHEMATC

Commit message: working on power
Parts:
- added U?: SFP+cage, symbol readout:SFP+cage
Connections:
- net GNDD: now also U?.CAGE, U?.1, U?.10, U?.11, U?.12, U?.13, U?.14, U?.15, U?.16, U?.17, U?.18, U?.19, U?.2, U?.20, U?.3, U?.4, U?.5, U?.6, U?.7, U?.8, U?.9
Other:
- note added: "get part num\nfrom BoM"
- note added: "have to confirm frequency b4 ordering"
- note removed: "NEED to do cage"
Changed lines of the file:
@@
 	7950 3250 7750 3250
 Connection ~ 7950 3250
-Text Notes 9000 3950 0    118  ~ 24
-NEED to do cage
+Text Notes 10200 3800 0    118  ~ 24
+get part num\nfrom BoM
 Wire Wire Line
 	3650 2650 3650 2500
@@
 Wire Wire Line
 	2900 2900 3350 2900
-Text Notes 1850 3900 0    118  ~ 24
+Text Notes 1700 4100 0    118  ~ 24
 IM GUESSING DAN’S \ndesign here
 Text Notes 2300 3200 0    50   ~ 10
@@
 $EndComp
 NoConn ~ 6000 2450
+Text Notes 1000 2650 0    79   ~ 16
+have to confirm frequency b4 ordering
+$Comp
+L readout:SFP+cage U?
+U 1 1 60AA3CBE
+P 9800 3200
+F 0 "U?" H 10028 2251 50  0000 L CNN
+F 1 "SFP+cage" H 10028 2160 50  0000 L CNN
+F 2 "" H 9850 3300 50  0001 C CNN
+F 3 "" H 9850 3300 50  0001 C CNN
+	1    9800 3200
+	1    0    0    -1
+$EndComp
+Wire Wire Line
+	8850 4150 9600 4150
+Wire Wire Line
+	9600 3250 9700 3250
+Connection ~ 9600 4150
+Wire Wire Line
+	9600 4150 9700 4150
+Wire Wire Line
+	9700 3350 9600 3350
+Wire Wire Line
+	9600 3250 9600 3350
+Connection ~ 9600 3350
+Wire Wire Line
+	9600 3350 9600 3450
+Wire Wire Line
+	9600 3450 9700 3450
+Connection ~ 9600 3450
+Wire Wire Line
+	9600 3450 9600 3550
+Wire Wire Line
+	9700 3550 9600 3550
+Connection ~ 9600 3550
+Wire Wire Line
+	9600 3550 9600 3650
+Wire Wire Line
+	9700 3650 9600 3650
+Connection ~ 9600 3650
+Wire Wire Line
+	9600 3650 9600 3750
+Wire Wire Line
+	9700 3750 9600 3750
+Connection ~ 9600 3750
+Wire Wire Line
+	9600 3750 9600 3850
+Wire Wire Line
+	9700 3850 9600 3850
+Connection ~ 9600 3850
+Wire Wire Line
+	9600 3850 9600 3950
+Wire Wire Line
+	9700 3950 9600 3950
+Connection ~ 9600 3950
+Wire Wire Line
+	9600 3950 9600 4050
+Wire Wire Line
+	9700 4050 9600 4050
+Connection ~ 9600 4050
+Wire Wire Line
+	9600 4050 9600 4150
+Wire Wire Line
+	9700 4250 9600 4250
+Wire Wire Line
+	9600 5150 9700 5150
+Wire Wire Line
+	9600 4150 9600 4250
+Connection ~ 9600 4250
+Wire Wire Line
+	9600 4250 9600 4350
+Wire Wire Line
+	9700 5050 9600 5050
+Connection ~ 9600 5050
+Wire Wire Line
+	9600 5050 9600 5150
+Wire Wire Line
+	9600 4950 9700 4950
+Connection ~ 9600 4950
+Wire Wire Line
+	9600 4950 9600 5050
+Wire Wire Line
+	9700 4850 9600 4850
+Connection ~ 9600 4850
+Wire Wire Line
+	9600 4850 9600 4950
+Wire Wire Line
+	9600 4750 9700 4750
+Connection ~ 9600 4750
+Wire Wire Line
+	9600 4750 9600 4850
+Wire Wire Line
+	9700 4650 9600 4650
+Connection ~ 9600 4650
+Wire Wire Line
+	9600 4650 9600 4750
+Wire Wire Line
+	9600 4550 9700 4550
+Connection ~ 9600 4550
+Wire Wire Line
+	9600 4550 9600 4650
+Wire Wire Line
+	9700 4450 9600 4450
+Connection ~ 9600 4450
+Wire Wire Line
+	9600 4450 9600 4550
+Wire Wire Line
+	9600 4350 9700 4350
+Connection ~ 9600 4350
+Wire Wire Line
+	9600 4350 9600 4450
+$Comp
+L power:GNDD #PWR?
+U 1 1 60B02076
+P 9600 5300
+F 0 "#PWR?" H 9600 5050 50  0001 C CNN
+F 1 "GNDD" H 9604 5145 50  0000 C CNN
+F 2 "" H 9600 5300 50  0001 C CNN
+F 3 "" H 9600 5300 50  0001 C CNN
+	1    9600 5300
+	1    0    0    -1
+$EndComp
+Wire Wire Line
+	9600 5300 9600 5150
+Connection ~ 9600 5150
 $EndSCHEMATC

Commit message: working on power
Parts:
- removed U?: Vcc0, symbol readout:Vcc0
- removed U?: VccSFP, symbol readout:VccSFP
- added U? (x2): Vcc0_3v3, symbol readout:Vcc0
- added U?: Vcc0_2v5, symbol readout:VccSFP
Connections:
- net +3V3 is gone; now on net VCC: C?.1, J?.1 (Pin_1), U?.6 (VDD)
- net VCC: now also U?.1 (VCC), U?.1 (VCC), U?.1 (VCC)
Other:
- note added: "for dan vcc0 is 2v5\nand vvcsfp is 3v3"
Changed lines of the file:
@@
 Connection ~ 1550 2800
-$Comp
-L power:+3V3 #PWR?
-U 1 1 60C8459E
-P 1550 2250
-AR Path="/60768143/60C8459E" Ref="#PWR?"  Part="1"
-AR Path="/608CAA95/60C8459E" Ref="#PWR?"  Part="1"
-F 0 "#PWR?" H 1550 2100 50  0001 C CNN
-F 1 "+3V3" H 1565 2423 50  0000 C CNN
-F 2 "" H 1550 2250 50  0001 C CNN
-F 3 "" H 1550 2250 50  0001 C CNN
-	1    1550 2250
-	1    0    0    -1
-$EndComp
 $Comp
 L Device:R_Small R?
@@
 $Comp
 L readout:Vcc0 U?
-U 1 1 62C7AC21
+U 1 1 609FAAE7
+P 8150 2250
+AR Path="/6076C700/609FAAE7" Ref="U?"  Part="1"
+AR Path="/62251D77/609FAAE7" Ref="U?"  Part="1"
+AR Path="/608CAA95/609FAAE7" Ref="U?"  Part="1"
+F 0 "U?" H 8150 2250 79  0001 C CNN
+F 1 "Vcc0_3v3" H 8000 2300 47  0000 L CNB
+F 2 "" H 8150 2250 79  0001 C CNN
+F 3 "" H 8150 2250 79  0001 C CNN
+	1    8150 2250
+	1    0    0    -1
+$EndComp
+$Comp
+L readout:VccSFP U?
+U 1 1 609FAAED
 P 7450 2500
+AR Path="/62251D77/609FAAED" Ref="U?"  Part="1"
+AR Path="/608CAA95/609FAAED" Ref="U?"  Part="1"
 F 0 "U?" H 7450 2500 79  0001 C CNN
-F 1 "Vcc0" H 7350 2550 47  0000 L CNB
+F 1 "Vcc0_2v5" H 7300 2550 47  0000 L CNB
 F 2 "" H 7450 2500 79  0001 C CNN
 F 3 "" H 7450 2500 79  0001 C CNN
@@
 	1    0    0    -1
 $EndComp
-$Comp
-L readout:VccSFP U?
-U 1 1 62C7E003
-P 8150 2250
-F 0 "U?" H 8150 2250 79  0001 C CNN
-F 1 "VccSFP" H 8050 2300 47  0000 L CNB
-F 2 "" H 8150 2250 79  0001 C CNN
-F 3 "" H 8150 2250 79  0001 C CNN
-	1    8150 2250
-	1    0    0    -1
-$EndComp
+Text Notes 8150 1900 0    50   ~ 0
+for dan vcc0 is 2v5\nand vvcsfp is 3v3
+$Comp
+L readout:Vcc0 U?
+U 1 1 60B6AA60
+P 1550 2150
+AR Path="/6076C700/60B6AA60" Ref="U?"  Part="1"
+AR Path="/62251D77/60B6AA60" Ref="U?"  Part="1"
+AR Path="/608CAA95/60B6AA60" Ref="U?"  Part="1"
+F 0 "U?" H 1550 2150 79  0001 C CNN
+F 1 "Vcc0_3v3" H 1400 2200 47  0000 L CNB
+F 2 "" H 1550 2150 79  0001 C CNN
+F 3 "" H 1550 2150 79  0001 C CNN
+	1    1550 2150
+	1    0    0    -1
+$EndComp
