File: hardware/backplane-prototype/backplane-prototype.kicad_pcb (KiCad board)
At the start: 2 copper layers, 60 x 60 mm, 3 parts, among them J1 Conn_02x34_Odd_Even, J2 ERF8-060-05.0-L-DV, J3 Conn_02x34_Odd_Even

Commit message: Add files via upload
Parts:
- moved J1 95.0 mm to (87.5, 108.0)
- moved J2 95.0 mm to (100.0, 108.0), turned to 90 degrees
- moved J3 95.0 mm to (112.5, 108.0)
Connections:
- J2 pad 10: /BCH3 -> /CH3
- J2 pad 11: /CH4 -> /BCH4
- J2 pad 12: /BCH4 -> /CH4
- J2 pad 13: /CH5 -> /BCH5
- J2 pad 14: /BCH5 -> /CH5
- J2 pad 15: /CH6 -> /BCH6
- J2 pad 16: /BCH6 -> /CH6
- J2 pad 17: /CH7 -> /BCH7
- J2 pad 18: /BCH7 -> /CH7
- J2 pad 21: /CH8 -> /BCH8
- J2 pad 22: /BCH8 -> /CH8
- J2 pad 23: /CH9 -> /BCH9
- J2 pad 24: /BCH9 -> /CH9
- J2 pad 25: /CH10 -> /BCH10
- J2 pad 26: /BCH10 -> /CH10
- J2 pad 27: /CH11 -> /BCH11
- J2 pad 28: /BCH11 -> /CH11
- J2 pad 29: /CH12 -> /BCH12
- J2 pad 3: /CH0 -> /BCH0
- J2 pad 30: /BCH12 -> /CH12
- J2 pad 31: /CH13 -> /BCH13
- J2 pad 32: /BCH13 -> /CH13
- J2 pad 33: /CH14 -> /BCH14
- J2 pad 34: /BCH14 -> /CH14
- J2 pad 35: /CH15 -> /BCH15
- J2 pad 36: /BCH15 -> /CH15
- J2 pad 39: /CH16 -> /BCH16
- J2 pad 4: /BCH0 -> /CH0
- J2 pad 40: /BCH16 -> /CH16
- J2 pad 41: /CH17 -> /BCH17
- J2 pad 42: /BCH17 -> /CH17
- J2 pad 43: /CH18 -> /BCH18
- J2 pad 44: /BCH18 -> /CH18
- J2 pad 45: /CH19 -> /BCH19
- J2 pad 46: /BCH19 -> /CH19
- J2 pad 47: /CH20 -> /BCH20
- J2 pad 48: /BCH20 -> /CH20
- J2 pad 49: /CH21 -> /BCH21
- J2 pad 5: /CH1 -> /BCH1
- J2 pad 50: /BCH21 -> /CH21
- J2 pad 51: /CH22 -> /BCH22
- J2 pad 52: /BCH22 -> /CH22
- J2 pad 53: /CH23 -> /BCH23
- J2 pad 54: /BCH23 -> /CH23
- J2 pad 57: /CH24 -> /BCH24
- J2 pad 58: /BCH24 -> /CH24
- J2 pad 59: /CH25 -> /BCH25
- J2 pad 6: /BCH1 -> /CH1
- J2 pad 60: /BCH25 -> /CH25
- J2 pad 61: /CH26 -> /BCH26
- J2 pad 62: /BCH26 -> /CH26
- J2 pad 63: /CH27 -> /BCH27
- J2 pad 64: /BCH27 -> /CH27
- J2 pad 65: /CH28 -> /BCH28
- J2 pad 66: /BCH28 -> /CH28
- J2 pad 67: /CH29 -> /BCH29
- J2 pad 68: /BCH29 -> /CH29
- J2 pad 69: /CH30 -> /BCH30
- J2 pad 7: /CH2 -> /BCH2
- J2 pad 70: /BCH30 -> /CH30
- J2 pad 71: /CH31 -> /BCH31
- J2 pad 72: /BCH31 -> /CH31
- J2 pad 75: /BIAS1 -> /BIAS3
- J2 pad 76: /BIAS3 -> /BIAS1
- J2 pad 77: /VDD -> /OUT
- J2 pad 78: /OUT -> /VDD
- J2 pad 79: /BIAS2 -> /BIAS4
- J2 pad 8: /BCH2 -> /CH2
- J2 pad 80: /BIAS4 -> /BIAS2
- J2 pad 9: /CH3 -> /BCH3
Routing:
- net GND: track 192.5 -> 137.6 mm, vias 2 -> 32
- net /CH1: track 46.1 -> 14.7 mm
- net /CH0: track 47.7 -> 16.9 mm
- net /CH2: track 44.2 -> 15.3 mm
- net /CH31: track 0.00 -> 16.5 mm, vias 0 -> 1
- net /CH29: track 0.00 -> 16.2 mm, vias 0 -> 1
- net /CH27: track 0.00 -> 16.2 mm, vias 0 -> 1
- net /CH28: track 0.00 -> 16.2 mm, vias 0 -> 1
- net /CH30: track 0.00 -> 16.0 mm, vias 0 -> 1
- net /CH26: track 0.00 -> 15.9 mm, vias 0 -> 1
- net /CH25: track 0.00 -> 15.4 mm, vias 0 -> 1
- net /CH4: track 0.00 -> 15.3 mm, vias 0 -> 1
- net /CH5: track 0.00 -> 15.2 mm, vias 0 -> 1
- net /CH6: track 0.00 -> 15.2 mm, vias 0 -> 1
- net /CH3: track 0.00 -> 15.2 mm, vias 0 -> 1
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- added copper zone on B.Cu, net GND

Commit message: Signal tracing on Backplane Prototype
Parts:
- removed J3: Conn_02x34_Odd_Even, Backplane-prototype:SAMTEC_CLM-134-02-F-D
- added J: Conn_02x34_Odd_Even, Backplane-prototype:SAMTEC_CLM-134-02-F-D, F.Cu at (202.8, 107.6)
- moved J1 90.3 mm to (177.8, 107.6)
- moved J2 90.3 mm to (190.3, 107.6)
Routing:
- net GND: track 137.6 -> 11.9 mm, vias 32 -> 0
- net /BCH11: track 1.45 -> 30.9 mm, vias 0 -> 1
- net /BCH10: track 1.45 -> 30.4 mm, vias 0 -> 1
- net /BCH12: track 1.45 -> 30.3 mm, vias 0 -> 1
- net /BCH9: track 1.45 -> 29.7 mm, vias 0 -> 1
- net /BCH13: track 1.45 -> 29.6 mm, vias 0 -> 1
- net /BCH7: track 1.45 -> 29.3 mm, vias 0 -> 1
- net /BCH8: track 1.45 -> 29.2 mm, vias 0 -> 1
- net /BCH14: track 1.45 -> 29.0 mm, vias 0 -> 1
- net /BCH6: track 1.45 -> 28.6 mm, vias 0 -> 1
- net /BCH5: track 1.45 -> 28.3 mm, vias 0 -> 1
- net /BCH15: track 1.45 -> 28.3 mm, vias 0 -> 1
- net /BCH4: track 1.45 -> 27.8 mm, vias 0 -> 1
- net /BCH16: track 1.45 -> 27.5 mm, vias 0 -> 1
- net /BCH3: track 1.45 -> 27.4 mm, vias 0 -> 1
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- added copper zone on F.Cu, net GND
- removed copper zone on B.Cu, net GND

Commit message: Prelinary Layout Made
Routing:
- net GND: track 11.9 -> 114.1 mm, vias 0 -> 23
- net /BIAS1: track 0.00 -> 47.2 mm, vias 0 -> 1
- net /BIAS3: track 0.00 -> 30.5 mm, vias 0 -> 1
- net /OUT: track 1.35 -> 22.4 mm, vias 0 -> 1
- net /VDD: track 1.35 -> 19.5 mm, vias 0 -> 1
- net /BIAS4: track 3.20 -> 20.1 mm, vias 0 -> 1
- net /BIAS2: track 0.00 -> 16.4 mm, vias 0 -> 1

Commit message: PCB Layout Edited
Parts:
- moved J 40.8 mm to (162.0, 106.0)
- moved J1 40.8 mm to (137.0, 106.0)
- moved J2 40.8 mm to (149.5, 106.0)
Routing:
- net GND: track 114.1 -> 226.0 mm, vias 23 -> 55
- net /BCH9: track 29.7 -> 34.0 mm, vias 1 -> 2
- net /BCH24: track 17.7 -> 20.8 mm
- net /BCH11: track 30.9 -> 33.8 mm, vias 1 -> 2
- net /BCH30: track 20.7 -> 17.8 mm
- net /BCH8: track 29.2 -> 32.1 mm
- net /BCH13: track 29.6 -> 32.1 mm, vias 1 -> 2
- net /BCH14: track 29.0 -> 30.2 mm
- net /BCH31: track 20.9 -> 19.7 mm, vias 1 -> 2
- net /BCH23: track 23.6 -> 22.5 mm
- net /BCH22: track 24.3 -> 25.4 mm
- net /BCH17: track 27.0 -> 28.0 mm, vias 1 -> 2
- net /BCH18: track 26.4 -> 27.2 mm
- net /BCH27: track 19.0 -> 19.5 mm, vias 1 -> 2
- net /BCH20: track 25.4 -> 24.9 mm, vias 1 -> 2
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- added copper zone on Ground, net GND
- removed copper zone on F.Cu, net GND
Other:
- copper layers 2 -> 4

Commit message: PCB Layout Edited
Routing:
- net /BCH21: track 24.8 -> 38.0 mm
- net /BCH19: track 25.9 -> 37.4 mm
- net /BCH17: track 28.0 -> 37.1 mm
- net /BCH15: track 28.3 -> 35.3 mm
- net /BCH1: track 26.6 -> 33.4 mm
- net /BCH3: track 27.4 -> 33.6 mm
- net /BCH9: track 34.0 -> 40.0 mm
- net /BCH5: track 28.3 -> 33.7 mm
- net /BCH13: track 32.1 -> 37.3 mm
- net /BCH7: track 29.3 -> 33.9 mm
- net /BCH11: track 33.8 -> 36.8 mm

Commit message: PCB Layout Edited
Routing:
- net /BCH9: track 40.0 -> 36.7 mm
- net /BCH7: track 33.9 -> 36.5 mm, vias 1 -> 2
- net /BCH5: vias 1 -> 2
- net /BCH3: vias 1 -> 2
- net /BCH1: vias 1 -> 2
Changed lines of the file:
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@@
     (thickness 1.6)
     (drawings 4)
-    (tracks 848)
+    (tracks 852)
     (zones 0)
     (modules 3)
@@
   )
   (setup
-    (last_trace_width 0.25)
+    (last_trace_width 0.381)
     (user_trace_width 0.2794)
     (user_trace_width 0.3302)
@@
   (segment (start 151.75 83.2) (end 162.9 83.2) (width 0.381) (layer B.Cu) (net 38))
   (segment (start 163.55 89.5) (end 169.4 89.5) (width 0.381) (layer F.Cu) (net 38))
-  (segment (start 169.6 90.5) (end 169.6 90.5) (width 0.381) (layer B.Cu) (net 39))
   (segment (start 164.616 90.5) (end 163.55 90.5) (width 0.381) (layer F.Cu) (net 39))
-  (segment (start 162.837969 84) (end 151.75 84) (width 0.381) (layer B.Cu) (net 39))
-  (segment (start 169.337969 90.5) (end 162.837969 84) (width 0.381) (layer B.Cu) (net 39))
   (via (at 173 90.5) (size 0.5588) (drill 0.3048) (layers F.Cu B.Cu) (net 39))
-  (segment (start 173 90.5) (end 169.337969 90.5) (width 0.381) (layer B.Cu) (net 39))
   (segment (start 173 90.5) (end 164.616 90.5) (width 0.381) (layer F.Cu) (net 39))
+  (segment (start 151.75 84) (end 153.4 84) (width 0.381) (layer B.Cu) (net 39))
+  (segment (start 153.4 84) (end 153.4 84) (width 0.381) (layer B.Cu) (net 39))
+  (segment (start 169.408546 90.5) (end 173 90.5) (width 0.381) (layer In1.Cu) (net 39))
+  (segment (start 162.908546 84) (end 169.408546 90.5) (width 0.381) (layer In1.Cu) (net 39))
+  (segment (start 153.4 84) (end 153.4 84) (width 0.381) (layer In1.Cu) (net 39))
+  (segment (start 153.4 84) (end 162.908546 84) (width 0.381) (layer In1.Cu) (net 39))
+  (via (at 153.4 84) (size 0.5588) (drill 0.3048) (layers F.Cu B.Cu) (net 39))
   (segment (start 151.75 84.8) (end 162.816297 84.8) (width 0.381) (layer B.Cu) (net 40))
   (segment (start 162.816297 84.8) (end 169.516297 91.5) (width 0.381) (layer B.Cu) (net 40))
@@
   (via (at 169.7 91.5) (size 0.5588) (drill 0.3048) (layers F.Cu B.Cu) (net 40))
   (segment (start 163.55 91.5) (end 169.7 91.5) (width 0.381) (layer F.Cu) (net 40))
-  (segment (start 169.9 92.5) (end 169.9 92.5) (width 0.381) (layer B.Cu) (net 41))
   (segment (start 163.55 92.5) (end 173 92.5) (width 0.381) (layer F.Cu) (net 41))
-  (segment (start 162.794625 85.6) (end 151.75 85.6) (width 0.381) (layer B.Cu) (net 41))
-  (segment (start 169.694625 92.5) (end 162.794625 85.6) (width 0.381) (layer B.Cu) (net 41))
-  (segment (start 173 92.5) (end 169.694625 92.5) (width 0.381) (layer B.Cu) (net 41))
   (via (at 173 92.5) (size 0.5588) (drill 0.3048) (layers F.Cu B.Cu) (net 41))
+  (segment (start 151.75 85.6) (end 153.4 85.6) (width 0.381) (layer B.Cu) (net 41))
+  (segment (start 153.4 85.6) (end 153.4 85.6) (width 0.381) (layer B.Cu) (net 41))
+  (segment (start 169.708546 92.5) (end 173 92.5) (width 0.381) (layer In1.Cu) (net 41))
+  (segment (start 162.808546 85.6) (end 169.708546 92.5) (width 0.381) (layer In1.Cu) (net 41))
+  (segment (start 153.4 85.6) (end 153.4 85.6) (width 0.381) (layer In1.Cu) (net 41))
+  (segment (start 153.4 85.6) (end 162.808546 85.6) (width 0.381) (layer In1.Cu) (net 41))
+  (via (at 153.4 85.6) (size 0.5588) (drill 0.3048) (layers F.Cu B.Cu) (net 41))
   (segment (start 151.75 86.4) (end 162.772953 86.4) (width 0.381) (layer B.Cu) (net 42))
   (segment (start 162.772953 86.4) (end 169.872953 93.5) (width 0.381) (layer B.Cu) (net 42))
@@
   (via (at 170.1 93.5) (size 0.5588) (drill 0.3048) (layers F.Cu B.Cu) (net 42))
   (segment (start 163.55 93.5) (end 170.1 93.5) (width 0.381) (layer F.Cu) (net 42))
-  (segment (start 170.3 94.5) (end 170.3 94.5) (width 0.381) (layer B.Cu) (net 43))
-  (segment (start 170.051281 94.5) (end 162.751281 87.2) (width 0.381) (layer B.Cu) (net 43))
   (segment (start 163.55 94.5) (end 173 94.5) (width 0.381) (layer F.Cu) (net 43))
-  (segment (start 162.751281 87.2) (end 151.75 87.2) (width 0.381) (layer B.Cu) (net 43))
-  (segment (start 173 94.5) (end 170.051281 94.5) (width 0.381) (layer B.Cu) (net 43))
   (via (at 173 94.5) (size 0.5588) (drill 0.3048) (layers F.Cu B.Cu) (net 43))
-  (segment (start 151.75 88) (end 162.729609 88) (width 0.381) (layer B.Cu) (net 44))
-  (segment (start 162.729609 88) (end 170.229609 95.5) (width 0.381) (layer B.Cu) (net 44))
-  (segment (start 170.229609 95.5) (end 170.4 95.5) (width 0.381) (layer B.Cu) (net 44))
+  (segment (start 151.75 87.2) (end 153.4 87.2) (width 0.381) (layer B.Cu) (net 43))
+  (segment (start 170.108546 94.5) (end 173 94.5) (width 0.381) (layer In1.Cu) (net 43))
+  (segment (start 162.808546 87.2) (end 170.108546 94.5) (width 0.381) (layer In1.Cu) (net 43))
+  (segment (start 153.4 87.2) (end 153.4 87.2) (width 0.381) (layer In1.Cu) (net 43))
+  (segment (start 153.4 87.2) (end 162.808546 87.2) (width 0.381) (layer In1.Cu) (net 43))
+  (via (at 153.4 87.2) (size 0.5588) (drill 0.3048) (layers F.Cu B.Cu) (net 43))
   (segment (start 170.4 95.5) (end 170.4 95.5) (width 0.381) (layer B.Cu) (net 44))
   (via (at 170.4 95.5) (size 0.5588) (drill 0.3048) (layers F.Cu B.Cu) (net 44))
   (segment (start 164.616 95.5) (end 170.4 95.5) (width 0.381) (layer F.Cu) (net 44))
   (segment (start 163.55 95.5) (end 164.616 95.5) (width 0.381) (layer F.Cu) (net 44))
+  (segment (start 170.229609 95.5) (end 170.4 95.5) (width 0.381) (layer B.Cu) (net 44))
+  (segment (start 162.729609 88) (end 170.229609 95.5) (width 0.381) (layer B.Cu) (net 44))
+  (segment (start 151.75 88) (end 162.729609 88) (width 0.381) (layer B.Cu) (net 44))
   (segment (start 170.7 96.5) (end 170.7 96.5) (width 0.381) (layer B.Cu) (net 45))
   (segment (start 163.55 96.5) (end 173 96.5) (width 0.381) (layer F.Cu) (net 45))
-  (segment (start 162.846557 88.93862) (end 162.83862 88.93862) (width 0.381) (layer B.Cu) (net 45))
-  (segment (start 162.7 88.8) (end 153.7 88.8) (width 0.381) (layer B.Cu) (net 45))
-  (segment (start 170.407937 96.5) (end 162.846557 88.93862) (width 0.381) (layer B.Cu) (net 45))
-  (segment (start 153.7 88.8) (end 151.75 88.8) (width 0.381) (layer B.Cu) (net 45))
-  (segment (start 162.83862 88.93862) (end 162.7 88.8) (width 0.381) (layer B.Cu) (net 45))
   (segment (start 173 96.5) (end 170.407937 96.5) (width 0.381) (layer B.Cu) (net 45))
   (via (at 173 96.5) (size 0.5588) (drill 0.3048) (layers F.Cu B.Cu) (net 45))
+  (segment (start 162.708546 88.8) (end 170.408546 96.5) (width 0.381) (layer In1.Cu) (net 45))
+  (segment (start 151.75 88.8) (end 153.4 88.8) (width 0.381) (layer B.Cu) (net 45))
+  (segment (start 170.408546 96.5) (end 173 96.5) (width 0.381) (layer In1.Cu) (net 45))
+  (segment (start 153.4 88.8) (end 153.4 88.8) (width 0.381) (layer In1.Cu) (net 45))
+  (segment (start 153.4 88.8) (end 162.708546 88.8) (width 0.381) (layer In1.Cu) (net 45))
+  (via (at 153.4 88.8) (size 0.5588) (drill 0.3048) (layers F.Cu B.Cu) (net 45))
   (segment (start 170.8 97.5) (end 170.586265 97.5) (width 0.381) (layer B.Cu) (net 46))
   (segment (start 163.55 97.5) (end 170.8 97.5) (width 0.381) (layer F.Cu) (net 46))
   (via (at 170.8 97.5) (size 0.5588) (drill 0.3048) (layers F.Cu B.Cu) (net 46))
-  (segment (start 153.561371 89.519629) (end 162.605893 89.519629) (width 0.381) (layer B.Cu) (net 46))
-  (segment (start 152.681 90.4) (end 153.561371 89.519629) (width 0.381) (layer B.Cu) (net 46))
   (segment (start 162.605893 89.519629) (end 164.993132 91.906868) (width 0.381) (layer B.Cu) (net 46))
-  (segment (start 151.75 90.4) (end 152.681 90.4) (width 0.381) (layer B.Cu) (net 46))
   (segment (start 164.993132 91.906868) (end 163.486265 90.4) (width 0.381) (layer B.Cu) (net 46))
   (segment (start 170.586265 97.5) (end 164.993132 91.906868) (width 0.381) (layer B.Cu) (net 46))
-  (segment (start 163.464593 91.2) (end 164.121566 91.856973) (width 0.381) (layer B.Cu) (net 47))
-  (segment (start 171 98.5) (end 171 98.5) (width 0.381) (layer B.Cu) (net 47))
+  (segment (start 158.330058 90.4) (end 159.210429 89.519629) (width 0.381) (layer B.Cu) (net 46))
+  (segment (start 159.210429 89.519629) (end 162.605893 89.519629) (width 0.381) (layer B.Cu) (net 46))
+  (segment (start 151.75 90.4) (end 158.330058 90.4) (width 0.381) (layer B.Cu) (net 46))
   (segment (start 151.75 91.2) (end 150.7 91.2) (width 0.381) (layer B.Cu) (net 47))
   (segment (start 150.7 91.2) (end 150.7 91.2) (width 0.381) (layer B.Cu) (net 47))
@@
   (segment (start 173 98.5) (end 170.808546 98.5) (width 0.381) (layer In1.Cu) (net 47))
   (segment (start 163.55 98.5) (end 173 98.5) (width 0.381) (layer F.Cu) (net 47))
-  (segment (start 173 98.5) (end 170.764593 98.5) (width 0.381) (layer B.Cu) (net 47))
-  (segment (start 170.764593 98.5) (end 170.682296 98.417703) (width 0.381) (layer B.Cu) (net 47))
   (via (at 173 98.5) (size 0.5588) (drill 0.3048) (layers F.Cu B.Cu) (net 47))
   (segment (start 151.75 92) (end 163.442921 92) (width 0.381) (layer B.Cu) (net 48))
@@
   (segment (start 171.242922 99.5) (end 171.271461 99.528539) (width 0.381) (layer F.Cu) (net 48))
   (segment (start 163.55 99.5) (end 171.242922 99.5) (width 0.381) (layer F.Cu) (net 48))
-  (segment (start 171.489375 100.489375) (end 171.489375 100.489375) (width 0.381) (layer B.Cu) (net 49))
   (segment (start 151.75 92.8) (end 150.7 92.8) (width 0.381) (layer B.Cu) (net 49))
   (segment (start 150.7 92.8) (end 150.7 92.8) (width 0.381) (layer B.Cu) (net 49))

Commit message: Backplane Prototype Layour Made
Parts:
- renumbered J to J3
Routing:
- net /BIAS1: track 47.2 -> 51.4 mm
- net /BCH25: track 17.2 -> 21.1 mm, vias 1 -> 2
- net /BIAS2: track 16.4 -> 20.1 mm
- net /CH1: track 14.7 -> 11.4 mm
- net /CH4: track 15.3 -> 12.0 mm
- net /BCH29: track 20.2 -> 17.4 mm
- net /BCH7: track 36.5 -> 33.9 mm
- net /CH7: track 15.1 -> 12.7 mm
- net /CH10: track 14.5 -> 12.4 mm
- net /CH31: track 16.5 -> 18.4 mm
- net /CH30: track 16.0 -> 17.6 mm
- net /CH16: track 14.4 -> 12.8 mm
- net /CH29: track 16.2 -> 17.8 mm, vias 1 -> 2
- net /CH2: track 15.3 -> 13.8 mm, vias 1 -> 2
- net /CH28: track 16.2 -> 17.7 mm
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
Commit message: Backplane Prototype (Rev A) Completed
Routing:
- net /BCH24: track 20.8 -> 19.9 mm
- net GND: track 226.3 -> 225.6 mm, vias 56 -> 55
Other:
- board text added: "EMPHATIC Backplane Prototype REV A"
- board text added: "S/N:"
- board text added: "T.Agarwal - 2021 - 04"
- board text added: "http://edf.bu.edu"
