File: hardware/backplane/backplane.kicad_pcb (KiCad board)
At the start: 4 copper layers, 50 x 455 mm, 24 parts, among them J1 ERF8-060-05.0-L-DV, J101 Conn_02x34_Odd_Even, J102 ERF8-060-05.0-L-DV, J103 Conn_02x34_Odd_Even, J2 ERF8-060-05.0-L-DV, J201 Conn_02x34_Odd_Even-Connector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, J203 Conn_02x34_Odd_Even-Connector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, J301 Conn_02x34_Odd_Even-Connector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, J302 ERF8-060-05.0-L-DV, J303 Conn_02x34_Odd_Even-Connector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, J401 Conn_02x34_Odd_Even, J402 ERF8-060-05.0-L-DV, J403 Conn_02x34_Odd_Even, J501 Conn_02x34_Odd_Even-Connector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, J503 Conn_02x34_Odd_Even-Connector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, J601 Conn_02x34_Odd_Even-Connector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, J602 ERF8-060-05.0-L-DV, J603 Conn_02x34_Odd_Even-Connector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, J701 Conn_02x34_Odd_Even, J703 Conn_02x34_Odd_Even, J801 Conn_02x34_Odd_Even-Connector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, J803 Conn_02x34_Odd_Even-Connector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, J901 Conn_02x34_Odd_Even-Connector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, J903 Conn_02x34_Odd_Even-Connector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

Commit message: 9 SiPM Array Backplane Completed
Routing:
- net GND: track 1029.8 -> 1076.5 mm, vias 343 -> 378
- net /SiPM_Connector(4-6)/OUT: track 24.5 -> 55.6 mm, vias 2 -> 3
- net /SiPM_Connector(4-6)/VDD: track 32.0 -> 56.6 mm
- net /SiPM_Connector(4-6)/BCH50: track 0.00 -> 20.1 mm, vias 0 -> 1
- net /SiPM_Connector(4-6)/BIAS22: track 3.42 -> 23.1 mm
- net /SiPM_Connector(4-6)/BIAS24: track 3.42 -> 23.1 mm
- net /SiPM_Connector(4-6)/BCH57: track 0.00 -> 19.1 mm, vias 0 -> 1
- net /SiPM_Connector(4-6)/BCH54: track 0.00 -> 18.9 mm, vias 0 -> 1
- net /SiPM_Connector(4-6)/BCH49: track 0.00 -> 18.9 mm, vias 0 -> 2
- net /SiPM_Connector(4-6)/BCH60: track 0.00 -> 18.5 mm, vias 0 -> 1
- net /SiPM_Connector(4-6)/BCH62: track 0.00 -> 18.5 mm, vias 0 -> 1
- net /SiPM_Connector(4-6)/BCH52: track 0.00 -> 18.5 mm, vias 0 -> 2
- net /SiPM_Connector(4-6)/BCH51: track 0.00 -> 18.1 mm, vias 0 -> 1
- net /SiPM_Connector(4-6)/BCH53: track 0.00 -> 17.9 mm, vias 0 -> 1
- net /SiPM_Connector(4-6)/BCH58: track 0.00 -> 17.9 mm, vias 0 -> 2
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Other:
- outline, holes or cut-outs redrawn
