File: hardware/backplane/SiPM_Connector(4-6).sch (KiCad schematic (older format))
At the start: 8 parts, among them J101 Conn_02x34_Odd_Even, J103 Conn_02x34_Odd_Even, J201 Conn_02x34_Odd_Even-Connector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, J203 Conn_02x34_Odd_Even-Connector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, J301 Conn_02x34_Odd_Even-Connector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, J303 Conn_02x34_Odd_Even-Connector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, J402 ERF8-060-05.0-L-DV, J602 ERF8-060-05.0-L-DV

Commit message: Edited Backplane
Connections:
- removed net BIAS1: J101.2 (Pin_2), J201.2 (Pin_2), J301.2 (Pin_2), J402.76, J602.116, J602.36
- removed net BIAS2: J101.68 (Pin_68), J201.68 (Pin_68), J301.68 (Pin_68), J402.80, J602.120, J602.40
- removed net BIAS3: J103.1 (Pin_1), J203.1 (Pin_1), J303.1 (Pin_1), J402.75, J602.115, J602.35
- removed net BIAS4: J103.67 (Pin_67), J203.67 (Pin_67), J303.67 (Pin_67), J402.79, J602.119, J602.39
- new net BIAS13: J101.2 (Pin_2), J402.76
- new net BIAS14: J101.68 (Pin_68), J402.80
- new net BIAS15: J103.1 (Pin_1), J402.75
- new net BIAS16: J103.67 (Pin_67), J402.79
- new net BIAS17: J201.2 (Pin_2), J602.36
- new net BIAS18: J201.68 (Pin_68), J602.40
- new net BIAS19: J203.1 (Pin_1), J602.35
- new net BIAS20: J203.67 (Pin_67), J602.39
- new net BIAS21: J301.2 (Pin_2), J602.116
- new net BIAS22: J301.68 (Pin_68), J602.120
- new net BIAS23: J303.1 (Pin_1), J602.115
- new net BIAS24: J303.67 (Pin_67), J602.119
Changed lines of the file:
@@
 	2150 2300 1950 2300
 Text Label 1950 2300 2    50   ~ 0
-BIAS1
+BIAS13
 Text Label 2750 2300 0    50   ~ 0
 CH0
@@
 OUT
 Text Label 9050 5600 0    50   ~ 0
-BIAS4
+BIAS16
 Text Label 8250 5400 2    50   ~ 0
 BCH31
@@
 Connection ~ 8950 5500
 Text Label 9050 2300 0    50   ~ 0
-BIAS3
+BIAS15
 Wire Wire Line
 	5000 6050 4800 6050
@@
 	6000 6250 6200 6250
 Text Label 4800 6050 2    50   ~ 0
-BIAS1
+BIAS13
 Text Label 4800 6150 2    50   ~ 0
 VDD
 Text Label 4800 6250 2    50   ~ 0
-BIAS2
+BIAS14
 Text Label 6200 6050 0    50   ~ 0
-BIAS3
+BIAS15
 Text Label 6200 6150 0    50   ~ 0
 OUT
@@
 $EndComp
 Text Label 6200 6250 0    50   ~ 0
-BIAS4
+BIAS16
 Text Label 2750 10050 0    50   ~ 0
 VDD
@@
 	6000 10650 6200 10650
 Text Label 6200 10450 0    50   ~ 0
-BIAS3
+BIAS19
 Text Label 6200 10550 0    50   ~ 0
 OUT
 Text Label 6200 10650 0    50   ~ 0
-BIAS4
+BIAS20
 Wire Wire Line
 	6000 14450 6200 14450
@@
 	6000 14650 6200 14650
 Text Label 6200 14450 0    50   ~ 0
-BIAS3
+BIAS23
 Text Label 6200 14550 0    50   ~ 0
 OUT
 Text Label 6200 14650 0    50   ~ 0
-BIAS4
+BIAS24
 Wire Wire Line
 	5000 10450 4800 10450
@@
 	5000 10650 4800 10650
 Text Label 4800 10450 2    50   ~ 0
-BIAS1
+BIAS17
 Text Label 4800 10550 2    50   ~ 0
 VDD
 Text Label 4800 10650 2    50   ~ 0
-BIAS2
+BIAS18
 Wire Wire Line
 	5000 14450 4800 14450
@@
 	5000 14650 4800 14650
 Text Label 4800 14450 2    50   ~ 0
-BIAS1
+BIAS21
 Text Label 4800 14550 2    50   ~ 0
 VDD
 Text Label 4800 14650 2    50   ~ 0
-BIAS2
+BIAS22
 Wire Wire Line
 	4750 8250 5000 8250
@@
 Connection ~ 8950 10050
 Text Label 9050 6850 0    50   ~ 0
-BIAS3
+BIAS19
 Wire Wire Line
 	8850 6850 9050 6850
@@
 Connection ~ 8950 14500
 Text Label 9050 11300 0    50   ~ 0
-BIAS3
+BIAS23
 Wire Wire Line
 	8850 11300 9050 11300
 Text Label 9050 10150 0    50   ~ 0
-BIAS4
+BIAS20
 NoConn ~ 8350 10050
 NoConn ~ 8350 14500
@@
 	2150 14600 1950 14600
 Text Label 1950 14600 2    50   ~ 0
-BIAS2
+BIAS22
 Connection ~ 2050 14500
 Wire Wire Line
 	2150 11300 1950 11300
 Text Label 1950 11300 2    50   ~ 0
-BIAS1
+BIAS21
 Connection ~ 2050 10050
 Wire Wire Line
 	2150 10150 1950 10150
 Text Label 1950 10150 2    50   ~ 0
-BIAS2
+BIAS18
 Text Label 1950 5600 2    50   ~ 0
-BIAS2
+BIAS14
 Connection ~ 2050 5500
 Wire Wire Line
 	2150 6850 1950 6850
 Text Label 1950 6850 2    50   ~ 0
-BIAS1
+BIAS17
 Text Label 2750 14500 0    50   ~ 0
 VDD
@@
 	9050 14600 8850 14600
 Text Label 9050 14600 0    50   ~ 0
-BIAS4
+BIAS24
 NoConn ~ 8350 14600
 Wire Wire Line

Commit message: -
Parts:
- J101, J103, J201, J203, J301, J303: symbol backplane-rescue:Conn_02x34_Odd_Even-Connector_Generic-backplane-prototype-rescue -> Connector_Generic:Conn_02x34_Odd_Even
- J402, J602: symbol backplane-rescue:ERF8-060-XX.X-X-DV-ERF8-060-05.0-L-DV-backplane-prototype-rescue -> ERF8-060-05.0-L-DV:ERF8-060-05.0-L-DV
Changed lines of the file:
@@
 	4300 3350 5000 3350
 $Comp
-L backplane-rescue:ERF8-060-XX.X-X-DV-ERF8-060-05.0-L-DV-backplane-prototype-rescue J402
+L ERF8-060-05.0-L-DV:ERF8-060-05.0-L-DV J402
 U 1 1 682C5401
 P 6000 2350
+AR Path="/682C5401" Ref="J402"  Part="1"
+AR Path="/60A16277/682C5401" Ref="J402"  Part="1"
 F 0 "J402" H 6500 2617 50  0000 C CNN
 F 1 "ERF8-060-05.0-L-DV" H 6500 2526 50  0000 C CNN
@@
 	8850 2300 9050 2300
 $Comp
-L backplane-rescue:Conn_02x34_Odd_Even-Connector_Generic-backplane-prototype-rescue J103
+L Connector_Generic:Conn_02x34_Odd_Even J103
 U 1 1 682C5400
 P 8650 3900
@@
 $EndComp
 $Comp
-L backplane-rescue:Conn_02x34_Odd_Even-Connector_Generic-backplane-prototype-rescue J101
+L Connector_Generic:Conn_02x34_Odd_Even J101
 U 1 1 682C53FF
 P 2450 3900
@@
 Connection ~ 6100 5950
 $Comp
-L backplane-rescue:GND-power-backplane-prototype-rescue #PWR0101
+L power:GND #PWR0101
 U 1 1 682C5402
 P 5500 14950
@@
 	6100 8150 6100 9450
 $Comp
-L backplane-rescue:ERF8-060-XX.X-X-DV-ERF8-060-05.0-L-DV-backplane-prototype-rescue J602
+L ERF8-060-05.0-L-DV:ERF8-060-05.0-L-DV J602
 U 1 1 682C53FE
 P 6000 8750
+AR Path="/682C53FE" Ref="J602"  Part="1"
+AR Path="/60A16277/682C53FE" Ref="J602"  Part="1"
 F 0 "J602" H 6500 9017 50  0000 C CNN
 F 1 "ERF8-060-05.0-L-DV" H 6500 8926 50  0000 C CNN
@@
 $EndComp
 $Comp
-L backplane-rescue:Conn_02x34_Odd_Even-Connector_Generic-backplane-prototype-rescue J301
+L Connector_Generic:Conn_02x34_Odd_Even J301
 U 1 1 682C5403
 P 2450 12900
@@
 $EndComp
 $Comp
-L backplane-rescue:Conn_02x34_Odd_Even-Connector_Generic-backplane-prototype-rescue J303
+L Connector_Generic:Conn_02x34_Odd_Even J303
 U 1 1 682C53FD
 P 8650 12900
@@
 $EndComp
 $Comp
-L backplane-rescue:Conn_02x34_Odd_Even-Connector_Generic-backplane-prototype-rescue J201
+L Connector_Generic:Conn_02x34_Odd_Even J201
 U 1 1 682C53FB
 P 2450 8450
@@
 	8350 8250 6350 8250
 $Comp
-L backplane-rescue:Conn_02x34_Odd_Even-Connector_Generic-backplane-prototype-rescue J203
+L Connector_Generic:Conn_02x34_Odd_Even J203
 U 1 1 682C53FC
 P 8650 8450
