File: hardware/readout_trenz/Citiroc-in-2.sch (KiCad schematic (older format))
At the start: 104 parts

Commit message: Readout Trenz Modified
Parts:
- removed C? (x37): 100n, symbol readout_trenz-rescue:C_Small-Device
- removed C? (x2): 10u, symbol readout_trenz-rescue:C_Small-Device
- removed C? (x3): 1u, symbol readout_trenz-rescue:C_Small-Device
- removed C? (x6): 150p, symbol readout_trenz-rescue:C_Small-Device
- removed J?: ERF8-060-XX.X-X-DV, ERF8-060-XX.X-X-DV, symbol erf:ERF8-060-XX.X-X-DV
- removed J?: BNC, symbol readout_trenz-rescue:Conn_Coaxial-Connector
- removed J?: GPIO Header, symbol readout_trenz-rescue:Conn_02x04_Odd_Even-Connector_Generic
- removed J?: conn, symbol readout_trenz-rescue:Conn_02x11_Counter_Clockwise-Connector_Generic
- removed R? (x32): 50, symbol readout_trenz-rescue:R-Device
- removed R?: 470k, symbol readout_trenz-rescue:R-Device
- removed R?: 1k, symbol readout_trenz-rescue:R-Device
- removed R? (x7): 0, symbol readout_trenz-rescue:R_Small-Device
- removed RV?: 10k, symbol readout_trenz-rescue:R_POT-Device
- removed U? (x2): Vcc0_2v5, symbol readout:VccSFP
- removed U? (x5): Vcc0_3v3, symbol readout:Vcc0
- removed U?: CITIROC1A, Package_QFP:LQFP-160_24x24mm_P0.5mm, symbol readout:CITIROC1A
- removed U?: ADS7955, Package_SO:TSSOP-30_4.4x7.8mm_P0.5mm, symbol readout:ADS7955
- removed U?: REF5025, Package_SO:SOIC-8_3.9x4.9mm_P1.27mm, symbol readout_trenz-rescue:REF5025ID-Reference_Voltage
- added C? (x37): 100n, symbol readout_trenz-rescue:C_Small-Device
- added C? (x3): 1u, symbol readout_trenz-rescue:C_Small-Device
- added C? (x6): 150p, symbol readout_trenz-rescue:C_Small-Device
- added C? (x2): 10u, symbol readout_trenz-rescue:C_Small-Device
- added J?: conn, symbol readout_trenz-rescue:Conn_02x11_Counter_Clockwise-Connector_Generic
- added J?: BNC, symbol readout_trenz-rescue:Conn_Coaxial-Connector
- added J?: GPIO Header, symbol readout_trenz-rescue:Conn_02x04_Odd_Even-Connector_Generic
- added R? (x32): 50, symbol readout_trenz-rescue:R-Device
- added R?: 470k, symbol readout_trenz-rescue:R-Device
- added R?: 1k, symbol readout_trenz-rescue:R-Device
- added R? (x7): 0, symbol readout_trenz-rescue:R_Small-Device
- added RV?: 10k, symbol readout_trenz-rescue:R_POT-Device
- added U?: CITIROC1A, Package_QFP:LQFP-160_24x24mm_P0.5mm, symbol readout:CITIROC1A
- added U? (x2): Vcc0_2v5, symbol readout:VccSFP
- added U? (x5): Vcc0_3v3, symbol readout:Vcc0
- added U?: REF5025, Package_SO:SOIC-8_3.9x4.9mm_P1.27mm, symbol readout_trenz-rescue:REF5025ID-Reference_Voltage
- added U?: ADS7955, Package_SO:TSSOP-30_4.4x7.8mm_P0.5mm, symbol readout:ADS7955
Connections:
- net GNDA: now also C?.1, C?.1, C?.1, C?.1, C?.2, C?.2, C?.2, C?.2, C?.2, C?.2, C?.2, C?.2, C?.2, C?.2, C?.2, C?.2, C?.2, C?.2, C?.2, C?.2, C?.2, C?.2, C?.2, C?.2, C?.2, C?.2, C?.2, C?.2, C?.2, C?.2, C?.2, C?.2, C?.2, C?.2, C?.2, C?.2, C?.2, C?.2, C?.2, C?.2, C?.2, C?.2, C?.2, C?.2, C?.2, C?.2, C?.2, C?.2, J?.12 (Pin_12), J?.13 (Pin_13), J?.14 (Pin_14), J?.15 (Pin_15), J?.16 (Pin_16), J?.17 (Pin_17), J?.18 (Pin_18), J?.19 (Pin_19), J?.2 (Ext), J?.20 (Pin_20), J?.21 (Pin_21), J?.22 (Pin_22), R?.2, U?.10 (AGND), U?.22 (AGND), U?.3 (REFM), U?.4 (GND), U?.6 (AGND), U?.9 (AINM)
- net GNDD: now also J?.2 (Pin_2), J?.4 (Pin_4), J?.6 (Pin_6), J?.8 (Pin_8), U?.27 (BDGND)
- net VCC: now also C?.1, C?.1, C?.1, C?.1, U?.1 (VCC), U?.1 (VCC), U?.1 (VCC), U?.1 (VCC), U?.1 (VCC), U?.1 (VCC), U?.1 (VCC), U?.2 (Vin), U?.21 (+VA), U?.28 (+VBD), U?.5 (+VA)
- new net: C?.1, R?.2 (x32)
- new net: R?.1, U?.18 (in13)
- new net: R?.1, U?.10 (in6)
- new net: R?.1, RV?.2
- new net: R?.2, U?.5 (Trim/NR)
- new net: R?.1, RV?.3
- new net: C?.1, RV?.1, U?.4 (REFP), U?.6 (Vout)
- new net: C?.1, R?.2, U?.45 (v_bg)
- new net: R?.1, U?.20 (in15)
- new net: R?.1, U?.11 (in7)
- new net: R?.1, U?.13 (in8)
- new net: R?.1, U?.14 (in9)
- new net: J?.5 (Pin_5), U?.144 (ib_sca)
- new net: J?.6 (Pin_6), U?.146 (ib_1nA_peak)
- new net: J?.7 (Pin_7), U?.147 (ibo_peak)
- new net: J?.8 (Pin_8), U?.148 (ibi_peak)
- new net: J?.9 (Pin_9), U?.149 (in_calib)
- new net: R?.1, U?.15 (in10)
- new net: J?.10 (Pin_10), U?.159 (ib_dac_5V)
- new net: R?.1, U?.16 (in11)
- new net: J?.11 (Pin_11), U?.160 (ibi_discri_t)
- new net: R?.1, U?.17 (in12)
- new net: R?.1, U?.19 (in14)
- new net: R?.1, U?.22 (in16)
- new net: R?.1, U?.23 (in17)
- new net: R?.1, U?.24 (in18)
- new net: R?.1, U?.25 (in19)
- new net: R?.1, U?.26 (in20)
- new net: R?.1, U?.27 (in21)
- new net: R?.1, U?.28 (in22)
- new net: R?.1, U?.29 (in23)
- new net: R?.1, U?.31 (in24)
- new net: R?.1, U?.32 (in25)
- new net: R?.1, U?.33 (in26)
- new net: R?.1, U?.34 (in27)
- new net: R?.1, U?.35 (in28)
- new net: R?.1, U?.36 (in29)
- new net: R?.1, U?.37 (in30)
- new net: R?.1, U?.38 (in31)
- new net: J?.1 (Pin_1), U?.39 (ib_temp)
- new net: R?.1, U?.4 (in0)
- new net: R?.2, U?.40 (out_temp)
- new net: R?.2, U?.42 (out_probe_dac_5V)
- new net: R?.2, U?.48 (vth)
- new net: C?.2, J?.2 (Pin_2), U?.49 (iref_dac)
- new net: R?.1, U?.5 (in1)
- new net: C?.2, U?.50 (vref_ssh_ig)
- new net: R?.2, U?.51 (vth_t)
- new net: C?.2, U?.52 (vref_ssh_hg)
- new net: C?.2, U?.53 (vref_fs)
- new net: R?.1, U?.6 (in2)
- new net: R?.2, U?.61 (out_hg)
- new net: R?.2, U?.62 (out_lg)
- new net: J?.1 (In), U?.63 (out_probe)
- new net: J?.3 (Pin_3), U?.64 (ib_otaq)
- new net: J?.4 (Pin_4), U?.69 (ib_rec)
- new net: R?.1, U?.7 (in3)
- new net: R?.1, U?.8 (in4)
- new net: R?.1, U?.9 (in5)
- new net: C?.1, R?.1, U?.13 (CH5)
- new net: C?.1, R?.1, U?.19 (CH1)
- new net: C?.1, R?.1, U?.14 (CH4)
- new net: C?.1, R?.1, U?.12 (CH6)
- new net: R?.1, U?.20 (CH0)
- new net: J?.5 (Pin_5), U?.1 (GPI02)
- new net: C?.1, R?.1, U?.17 (CH3)
- new net: C?.1, R?.1, U?.18 (CH2)
- new net: J?.7 (Pin_7), U?.2 (GPIO3)
- new net: J?.1 (Pin_1), U?.29 (GPIO0)
- new net: J?.3 (Pin_3), U?.30 (GPI01)
- new net: U?.7 (MXO), U?.8 (AINP)
- new net ADC_CS_1: U?.23 (~CS)
- new net ADC_SCLK_1: U?.24 (SCLK)
- new net ADC_SDI_1: U?.25 (SDI)
- new net ADC_SDO_1: U?.26 (SDO)
- no-connect marks 22 -> 2
