File: hardware/readout_trenz/FPGA-LVDS.sch (KiCad schematic (older format))
At the start: 15 parts

Commit message: Trenz Module Work in Progress
Other:
- note added: "Replace FPGA symbol with Trenz\n"
Changed lines of the file:
@@
 $Descr A4 11693 8268
 encoding utf-8
-Sheet 3 12
+Sheet 3 13
 Title ""
 Date ""
@@
 	1    0    0    -1
 $EndComp
+Text Notes 5300 1550 0    50   ~ 0
+Replace FPGA symbol with Trenz\n
 $EndSCHEMATC
