File: hardware/readout_trenz/Citiroc-in-1.sch (KiCad schematic (older format))
At the start: 104 parts

Commit message: Readout Trenz Modified
Parts:
- removed C? (x32): 100n, symbol readout_trenz-rescue:C_Small-Device
- removed C? (x6): 150p, symbol readout_trenz-rescue:C_Small-Device
- removed C? (x2): 10u, symbol readout_trenz-rescue:C_Small-Device
- removed C? (x2): 1u, symbol readout_trenz-rescue:C_Small-Device
- removed J?: conn, symbol readout_trenz-rescue:Conn_02x11_Counter_Clockwise-Connector_Generic
- removed J?: ERF8-060-XX.X-X-DV, ERF8-060-XX.X-X-DV, symbol erf:ERF8-060-XX.X-X-DV
- removed J?: BNC, symbol readout_trenz-rescue:Conn_Coaxial-Connector
- removed J?: GPIO Header, symbol readout_trenz-rescue:Conn_02x04_Odd_Even-Connector_Generic
- removed R? (x31): 50, symbol readout_trenz-rescue:R-Device
- removed R?: 470k, symbol readout_trenz-rescue:R-Device
- removed R?: 1k, symbol readout_trenz-rescue:R-Device
- removed R? (x7): 0, symbol readout_trenz-rescue:R_Small-Device
- removed RV?: 10k, symbol readout_trenz-rescue:R_POT-Device
- removed U? (x2): Vcc0_2v5, symbol readout:VccSFP
- removed U?: CITIROC1A, Package_QFP:LQFP-160_24x24mm_P0.5mm, symbol readout:CITIROC1A
- removed U? (x4): Vcc0_3v3, symbol readout:Vcc0
- removed U?: ADS7955, Package_SO:TSSOP-30_4.4x7.8mm_P0.5mm, symbol readout:ADS7955
- removed U?: REF5025, Package_SO:SOIC-8_3.9x4.9mm_P1.27mm, symbol readout_trenz-rescue:REF5025ID-Reference_Voltage
- added C? (x32): 100n, symbol readout_trenz-rescue:C_Small-Device
- added C? (x2): 10u, symbol readout_trenz-rescue:C_Small-Device
- added C? (x2): 1u, symbol readout_trenz-rescue:C_Small-Device
- added C? (x6): 150p, symbol readout_trenz-rescue:C_Small-Device
- added J?: conn, symbol readout_trenz-rescue:Conn_02x11_Counter_Clockwise-Connector_Generic
- added J?: GPIO Header, symbol readout_trenz-rescue:Conn_02x04_Odd_Even-Connector_Generic
- added J?: BNC, symbol readout_trenz-rescue:Conn_Coaxial-Connector
- added R? (x31): 50, symbol readout_trenz-rescue:R-Device
- added R? (x7): 0, symbol readout_trenz-rescue:R_Small-Device
- added R?: 470k, symbol readout_trenz-rescue:R-Device
- added R?: 1k, symbol readout_trenz-rescue:R-Device
- added RV?: 10k, symbol readout_trenz-rescue:R_POT-Device
- added U? (x2): Vcc0_2v5, symbol readout:VccSFP
- added U?: CITIROC1A, Package_QFP:LQFP-160_24x24mm_P0.5mm, symbol readout:CITIROC1A
- added U? (x4): Vcc0_3v3, symbol readout:Vcc0
- added U?: ADS7955, Package_SO:TSSOP-30_4.4x7.8mm_P0.5mm, symbol readout:ADS7955
- added U?: REF5025, Package_SO:SOIC-8_3.9x4.9mm_P1.27mm, symbol readout_trenz-rescue:REF5025ID-Reference_Voltage
Connections:
- net labels added: CITIROC_B2[0,31]
- net labels removed: Bias_3, Bias_4, out
- wire segments 363 -> 350
- no-connect marks 22 -> 2
