File: hardware/readout_trenz/FPGA-Connectivity.sch (KiCad schematic (older format))
At the start: 34 parts

Commit message: Trenz Module Work in Progress
Other:
- note added: "Only keep JTAG and FT23RL\n(Going to Trenz)"
Changed lines of the file:
@@
 $Descr A4 11693 8268
 encoding utf-8
-Sheet 7 12
+Sheet 7 13
 Title ""
 Date ""
@@
 	1    0    0    -1
 $EndComp
+Text Notes 1350 4800 0    197  ~ 39
+Only keep JTAG and FT23RL\n(Going to Trenz)
 $EndSCHEMATC
