File: hardware/readout_trenz/JTAG.sch (KiCad schematic (older format))
At the start: 0 parts

Commit message: Readout Trenz in Progress
Parts:
- added J?: Digilent JTAG header, readout_slice:87832-1420, symbol readout_trenz-rescue:Conn_02x07_Odd_Even-Connector_Generic
- added U?: Vcc0_3v3, symbol readout:Vcc0
Connections:
- new net GNDD: J?.1 (Pin_1), J?.11 (Pin_11), J?.13 (Pin_13), J?.3 (Pin_3), J?.5 (Pin_5), J?.7 (Pin_7), J?.9 (Pin_9)
- new net TCK: J?.6 (Pin_6)
- new net TDI: J?.10 (Pin_10)
- new net TDO: J?.8 (Pin_8)
- new net TMS: J?.4 (Pin_4)
- new net VCC: J?.2 (Pin_2), U?.1 (VCC)
- no-connect marks 0 -> 2
Changed lines of the file:
@@
 Comment4 ""
 $EndDescr
+$Comp
+L readout_trenz-rescue:Conn_02x07_Odd_Even-Connector_Generic J?
+U 1 1 60E990B0
+P 5800 3300
+AR Path="/60E990B0" Ref="J?"  Part="1"
+AR Path="/608B2FC0/60E990B0" Ref="J?"  Part="1"
+AR Path="/6099D1B7/60E990B0" Ref="J?"  Part="1"
+AR Path="/60AD0200/60AFD3C0/60E990B0" Ref="J?"  Part="1"
+AR Path="/606EBC4D/60E990B0" Ref="J?"  Part="1"
+AR Path="/60BC24EA/60E990B0" Ref="J?"  Part="1"
+F 0 "J?" H 5650 3800 50  0000 C CNN
+F 1 "Digilent JTAG header" H 5650 3700 50  0000 C CNN
+F 2 "readout_slice:87832-1420" H 5800 3300 50  0001 C CNN
+F 3 "~" H 5800 3300 50  0001 C CNN
+	1    5800 3300
+	1    0    0    -1
+$EndComp
+Wire Wire Line
+	5600 3000 5550 3000
+Wire Wire Line
+	5550 3000 5550 3100
+$Comp
+L readout_trenz-rescue:GNDD-power #PWR?
+U 1 1 60E990B8
+P 5550 3700
+AR Path="/60E990B8" Ref="#PWR?"  Part="1"
+AR Path="/608B2FC0/60E990B8" Ref="#PWR?"  Part="1"
+AR Path="/6099D1B7/60E990B8" Ref="#PWR?"  Part="1"
+AR Path="/60AD0200/60AFD3C0/60E990B8" Ref="#PWR?"  Part="1"
+AR Path="/606EBC4D/60E990B8" Ref="#PWR?"  Part="1"
+AR Path="/60BC24EA/60E990B8" Ref="#PWR?"  Part="1"
+F 0 "#PWR?" H 5550 3450 50  0001 C CNN
+F 1 "GNDD" H 5554 3545 50  0000 C CNN
+F 2 "" H 5550 3700 50  0001 C CNN
+F 3 "" H 5550 3700 50  0001 C CNN
+	1    5550 3700
+	-1   0    0    -1
+$EndComp
+Wire Wire Line
+	5600 3600 5550 3600
+Connection ~ 5550 3600
+Wire Wire Line
+	5550 3600 5550 3700
+Wire Wire Line
+	5550 3500 5600 3500
+Connection ~ 5550 3500
+Wire Wire Line
+	5550 3500 5550 3600
+Wire Wire Line
+	5600 3400 5550 3400
+Connection ~ 5550 3400
+Wire Wire Line
+	5550 3400 5550 3500
+Wire Wire Line
+	5550 3300 5600 3300
+Connection ~ 5550 3300
+Wire Wire Line
+	5550 3300 5550 3400
+Wire Wire Line
+	5600 3200 5550 3200
+Connection ~ 5550 3200
+Wire Wire Line
+	5550 3200 5550 3300
+Wire Wire Line
+	5550 3100 5600 3100
+Connection ~ 5550 3100
+Wire Wire Line
+	5550 3100 5550 3200
+NoConn ~ 6100 3600
+NoConn ~ 6100 3500
+Wire Wire Line
+	6200 2900 6200 3000
+Wire Wire Line
+	6200 3000 6100 3000
+Wire Wire Line
+	6100 3400 6200 3400
+Wire Wire Line
+	6100 3300 6200 3300
+Wire Wire Line
+	6100 3200 6200 3200
+Wire Wire Line
+	6100 3100 6200 3100
+$Comp
+L readout:Vcc0 U?
+U 1 1 60E990D8
+P 6200 2800
+AR Path="/6076C700/60E990D8" Ref="U?"  Part="1"
+AR Path="/62251D77/60E990D8" Ref="U?"  Part="1"
+AR Path="/608CAA95/60E990D8" Ref="U?"  Part="1"
+AR Path="/606EBC4D/60E990D8" Ref="U?"  Part="1"
+AR Path="/60BC24EA/60E990D8" Ref="U?"  Part="1"
+F 0 "U?" H 6200 2800 79  0001 C CNN
+F 1 "Vcc0_3v3" H 6050 2850 47  0000 L CNB
+F 2 "" H 6200 2800 79  0001 C CNN
+F 3 "" H 6200 2800 79  0001 C CNN
+	1    6200 2800
+	1    0    0    -1
+$EndComp
+Text HLabel 6200 3100 2    50   BiDi ~ 0
+TMS
+Text HLabel 6200 3200 2    50   BiDi ~ 0
+TCK
+Text HLabel 6200 3300 2    50   BiDi ~ 0
+TDO
+Text HLabel 6200 3400 2    50   BiDi ~ 0
+TDI
 $EndSCHEMATC
