File: hardware/readout_trenz/Trenz_Module.sch (KiCad schematic (older format))
At the start: 15 parts

Commit message: -
Connections:
- net +3V3: now also J?.6 (Pin_6)
- net at J?.1 (Pin_1): now also J?.3 (Pin_3), J?.5 (Pin_5), J?.61 (VCCIO34)
- net +1V8: now reaches J?.2 (Pin_2)
- net +2V5: now reaches J?.4 (Pin_4)
Other:
- moved on the sheet: J?
Changed lines of the file:
@@
 L readout_trenz-rescue:Conn_02x03_Odd_Even-Connector_Generic J?
 U 1 1 60B0C983
-P 2850 3550
+P 5000 4000
 AR Path="/60B0C983" Ref="J?"  Part="1"
 AR Path="/60D04563/60B0C983" Ref="J?"  Part="1"
-F 0 "J?" H 2900 3867 50  0000 C CNN
-F 1 "SMD -254-9132-14-6" H 2900 3776 50  0000 C CNN
-F 2 "" H 2850 3550 50  0001 C CNN
-F 3 "~" H 2850 3550 50  0001 C CNN
-	1    2850 3550
-	1    0    0    -1
+F 0 "J?" H 5050 4317 50  0000 C CNN
+F 1 "SMD -254-9132-14-6" H 5050 4226 50  0000 C CNN
+F 2 "" H 5000 4000 50  0001 C CNN
+F 3 "~" H 5000 4000 50  0001 C CNN
+	1    5000 4000
+	-1   0    0    -1
 $EndComp
 $Comp
@@
 T1_23
 Wire Wire Line
-	3150 3450 3250 3450
-Wire Wire Line
-	3150 3550 3250 3550
-Wire Wire Line
-	3150 3650 3250 3650
+	4700 3900 4600 3900
+$Comp
+L power:+1V8 #PWR?
+U 1 1 60C0EFC5
+P 4600 3900
+F 0 "#PWR?" H 4600 3750 50  0001 C CNN
+F 1 "+1V8" H 4615 4073 50  0000 C CNN
+F 2 "" H 4600 3900 50  0001 C CNN
+F 3 "" H 4600 3900 50  0001 C CNN
+	1    4600 3900
+	-1   0    0    -1
+$EndComp
+Wire Wire Line
+	4700 4000 4500 4000
+$Comp
+L power:+2V5 #PWR?
+U 1 1 60C185FA
+P 4500 4000
+F 0 "#PWR?" H 4500 3850 50  0001 C CNN
+F 1 "+2V5" H 4515 4173 50  0000 C CNN
+F 2 "" H 4500 4000 50  0001 C CNN
+F 3 "" H 4500 4000 50  0001 C CNN
+	1    4500 4000
+	-1   0    0    -1
+$EndComp
+Wire Wire Line
+	4700 4100 4400 4100
+$Comp
+L power:+3.3V #PWR?
+U 1 1 60C21C91
+P 4400 4100
+F 0 "#PWR?" H 4400 3950 50  0001 C CNN
+F 1 "+3.3V" H 4415 4273 50  0000 C CNN
+F 2 "" H 4400 4100 50  0001 C CNN
+F 3 "" H 4400 4100 50  0001 C CNN
+	1    4400 4100
+	-1   0    0    -1
+$EndComp
+Wire Wire Line
+	5200 3900 5300 3900
+Wire Wire Line
+	5300 3900 5300 4000
+Wire Wire Line
+	5300 4100 5200 4100
+Wire Wire Line
+	5200 4000 5300 4000
+Connection ~ 5300 4000
+Wire Wire Line
+	5300 4000 5300 4100
+Wire Wire Line
+	5300 3900 5550 3900
+Connection ~ 5300 3900
 Wire Bus Line
 	8500 800  8500 1500

Commit message: -
Parts:
- added C?: 10n, symbol readout_trenz-rescue:C_Small-Device
- added C?: 4.7u, symbol readout_trenz-rescue:C_Small-Device
Connections:
- net +2V5: now also U?.5 (OUT), C?.1
- net +3V3: now also U?.1 (IN), U?.3 (EN)
- net GNDD: now also J?.100 (GND), J?.98 (GND), U?.2 (GND), C?.2, C?.2; no longer J?.83 (3.3V_OUT), J?.97, J?.99
- net TCK: now also J?.90 (TCK); no longer J?.89 (B14_L23_N)
- net TDI: now also J?.86 (TDI); no longer J?.85 (B14_L24_N)
- net TDO: now also J?.88 (TDO); no longer J?.87 (B14_L24_P)
- net TMS: now also J?.92 (TMS); no longer J?.91 (B14_L23_P)
- net at U?.4 (NR): now also C?.1
Changed lines of the file:
@@
 	0    1    1    0
 $EndComp
-$Comp
-L readout_trenz-rescue:GNDD-power #PWR?
-U 1 1 60D90161
-P 5550 5000
-F 0 "#PWR?" H 5550 4750 50  0001 C CNN
-F 1 "GNDD-power" V 5554 4891 50  0000 R CNN
-F 2 "" H 5550 5000 50  0001 C CNN
-F 3 "" H 5550 5000 50  0001 C CNN
-	1    5550 5000
-	0    1    1    0
-$EndComp
-Wire Wire Line
-	5550 5700 5450 5700
-Wire Wire Line
-	5450 5700 5450 5800
 Wire Wire Line
 	5550 5900 5450 5900
-Connection ~ 5450 5900
 Wire Wire Line
 	5450 5900 5450 6000
-Wire Wire Line
-	5550 5800 5450 5800
-Connection ~ 5450 5800
-Wire Wire Line
-	5450 5800 5450 5900
-Text HLabel 5450 5100 0    50   BiDi ~ 0
+Text HLabel 6850 5100 2    50   BiDi ~ 0
 TDI
-Text HLabel 5450 5200 0    50   BiDi ~ 0
+Text HLabel 6850 5200 2    50   BiDi ~ 0
 TDO
-Text HLabel 5450 5300 0    50   BiDi ~ 0
+Text HLabel 6850 5300 2    50   BiDi ~ 0
 TCK
-Text HLabel 5450 5400 0    50   BiDi ~ 0
+Text HLabel 6850 5400 2    50   BiDi ~ 0
 TMS
 Wire Wire Line
-	5450 5100 5550 5100
-Wire Wire Line
-	5450 5200 5550 5200
-Wire Wire Line
-	5450 5300 5550 5300
-Wire Wire Line
-	5450 5400 5550 5400
-Text Notes 5400 5500 2    50   ~ 0
+	6850 5100 6750 5100
+Wire Wire Line
+	6850 5200 6750 5200
+Wire Wire Line
+	6850 5300 6750 5300
+Wire Wire Line
+	6850 5400 6750 5400
+Text Notes 6900 5500 0    50   ~ 0
 PROG_B\n
-Text Notes 5400 5600 2    50   ~ 0
+Text Notes 6900 5600 0    50   ~ 0
 DONE\n
 Wire Wire Line
@@
 	4700 3900 4600 3900
 $Comp
-L power:+1V8 #PWR?
+L readout_trenz-rescue:+1V8-power #PWR?
 U 1 1 60C0EFC5
 P 4600 3900
+AR Path="/60C0EFC5" Ref="#PWR?"  Part="1"
+AR Path="/60D04563/60C0EFC5" Ref="#PWR?"  Part="1"
 F 0 "#PWR?" H 4600 3750 50  0001 C CNN
 F 1 "+1V8" H 4615 4073 50  0000 C CNN
@@
 	4700 4000 4500 4000
 $Comp
-L power:+2V5 #PWR?
+L readout_trenz-rescue:+2V5-power #PWR?
 U 1 1 60C185FA
 P 4500 4000
@@
 	4700 4100 4400 4100
 $Comp
-L power:+3.3V #PWR?
+L readout_trenz-rescue:+3.3V-power #PWR?
 U 1 1 60C21C91
 P 4400 4100
@@
 	5300 3900 5550 3900
 Connection ~ 5300 3900
+Wire Wire Line
+	6750 5800 6850 5800
+Wire Wire Line
+	6850 5800 6850 5900
+Connection ~ 6850 5900
+Wire Wire Line
+	6750 5700 6850 5700
+Wire Wire Line
+	6850 5700 6850 5800
+Connection ~ 6850 5800
+$Comp
+L readout_trenz-rescue:+2V5-power #PWR?
+U 1 1 60C4B55D
+P 2400 2900
+F 0 "#PWR?" H 2400 2750 50  0001 C CNN
+F 1 "+2V5-power" H 2415 3073 50  0000 C CNN
+F 2 "" H 2400 2900 50  0001 C CNN
+F 3 "" H 2400 2900 50  0001 C CNN
+	1    2400 2900
+	1    0    0    -1
+$EndComp
+$Comp
+L readout_trenz-rescue:GNDD-power #PWR?
+U 1 1 60C4D776
+P 1600 3400
+F 0 "#PWR?" H 1600 3150 50  0001 C CNN
+F 1 "GNDD-power" H 1604 3245 50  0000 C CNN
+F 2 "" H 1600 3400 50  0001 C CNN
+F 3 "" H 1600 3400 50  0001 C CNN
+	1    1600 3400
+	1    0    0    -1
+$EndComp
+$Comp
+L readout_trenz-rescue:C_Small-Device C?
+U 1 1 60C51052
+P 2000 3200
+AR Path="/60767640/60C51052" Ref="C?"  Part="1"
+AR Path="/60D04563/60C51052" Ref="C?"  Part="1"
+F 0 "C?" H 1908 3246 50  0000 R CNN
+F 1 "10n" H 1908 3155 50  0000 R CNB
+F 2 "" H 2000 3200 50  0001 C CNN
+F 3 "~" H 2000 3200 50  0001 C CNN
+	1    2000 3200
+	-1   0    0    -1
+$EndComp
+$Comp
+L readout_trenz-rescue:C_Small-Device C?
+U 1 1 60C6173D
+P 2300 3200
+AR Path="/60767640/60C6173D" Ref="C?"  Part="1"
+AR Path="/60D04563/60C6173D" Ref="C?"  Part="1"
+F 0 "C?" H 2208 3246 50  0000 R CNN
+F 1 "4.7u" H 2208 3155 50  0000 R CNB
+F 2 "" H 2300 3200 50  0001 C CNN
+F 3 "~" H 2300 3200 50  0001 C CNN
+	1    2300 3200
+	-1   0    0    -1
+$EndComp
+$Comp
+L readout_trenz-rescue:GNDD-power #PWR?
+U 1 1 60C700F5
+P 2000 3400
+F 0 "#PWR?" H 2000 3150 50  0001 C CNN
+F 1 "GNDD-power" H 2004 3245 50  0000 C CNN
+F 2 "" H 2000 3400 50  0001 C CNN
+F 3 "" H 2000 3400 50  0001 C CNN
+	1    2000 3400
+	1    0    0    -1
+$EndComp
+$Comp
+L readout_trenz-rescue:GNDD-power #PWR?
+U 1 1 60C80B5B
+P 2300 3400
+F 0 "#PWR?" H 2300 3150 50  0001 C CNN
+F 1 "GNDD-power" H 2304 3245 50  0000 C CNN
+F 2 "" H 2300 3400 50  0001 C CNN
+F 3 "" H 2300 3400 50  0001 C CNN
+	1    2300 3400
+	1    0    0    -1
+$EndComp
+Wire Wire Line
+	1900 2900 2300 2900
+Wire Wire Line
+	2300 2900 2300 3100
+Connection ~ 2300 2900
+Wire Wire Line
+	2300 2900 2400 2900
+Wire Wire Line
+	2300 3300 2300 3400
+Wire Wire Line
+	1900 3100 2000 3100
+Wire Wire Line
+	2000 3300 2000 3400
+Wire Wire Line
+	1600 3250 1600 3400
+$Comp
+L readout_trenz-rescue:+3.3V-power #PWR?
+U 1 1 60CC7C9F
+P 1200 2900
+F 0 "#PWR?" H 1200 2750 50  0001 C CNN
+F 1 "+3.3V-power" H 1215 3073 50  0000 C CNN
+F 2 "" H 1200 2900 50  0001 C CNN
+F 3 "" H 1200 2900 50  0001 C CNN
+	1    1200 2900
+	1    0    0    -1
+$EndComp
+Wire Wire Line
+	1300 2900 1200 2900
+Wire Wire Line
+	1200 2900 1200 3100
+Wire Wire Line
+	1200 3100 1300 3100
 Wire Bus Line
 	8500 800  8500 1500
@@
 Wire Bus Line
 	10100 800  10100 3300
+Connection ~ 1200 2900
 $EndSCHEMATC

Commit message: Readout Trenz in progress
Parts:
- added C?: 47u, symbol readout_trenz-rescue:C_Small-Device
- added J?: Digilent JTAG header, readout_slice:87832-1420, symbol readout_trenz-rescue:Conn_02x07_Odd_Even-Connector_Generic
- added J?: Serial USB, symbol readout_trenz-rescue:Conn_01x04-Connector_Generic
- added J? (x2): Mounting, symbol readout_trenz-rescue:Conn_01x09-Connector_Generic
- added PS? (x6): 3.3V_OUT, symbol readout:3.3V_OUT
- added U? (x2): Vcc0_3v3, symbol readout:Vcc0
Connections:
- net +1V8: now also J?.18 (1.8V)
- net +3V3: now also J?.97, J?.99, C?.1; no longer J?.6 (Pin_6), R?.1, R?.1, U?.3 (EN)
- net GNDD: now also J?.17 (GND), J?.72 (GND), J?.83 (GND), J?.90 (GND), C?.2, J?.1 (Pin_1), J?.11 (Pin_11), J?.13 (Pin_13), J?.3 (Pin_3), J?.4 (Pin_4), J?.5 (Pin_5), J?.7 (Pin_7), J?.9 (Pin_9); no longer J?.18 (1.8V), J?.65 (B34_L17_P), J?.71 (SPI-DQ1), J?.84 (B14_L12_N), J?.89 (B14_L17_N)
- net MGT_RX2_N: now also J?.9 (MGT_RX2_N)
- net MGT_RX2_P: now also J?.7 (MGT_RX2_P)
- net MGT_TX2_N: now also J?.16 (MGT_TX2_N)
- net MGT_TX2_P: now also J?.14 (MGT_TX2_P)
- net SFP0_LOS: now also J?.34 (SFP0_LOS)
- net SFP0_M-DEF0: now also J?.40 (SFP0_M-DEF0)
- net SFP0_RS0: now also J?.38 (SFP0_RS0)
- net SFP0_RS1: now also J?.32 (SFP0_RSI)
- net SFP0_SCL: now also J?.48 (SFP0_SCL)
- net SFP0_SDA: now also J?.46 (SFP0_SDA)
- net SFP0_TX_DIS: now also J?.44 (SFP0_TX_DIS)
- net SFP0_TX_FAULT: now also J?.42 (SFP0_TX_FAULT)
- net T2_0: now also J?.1 (B15_L7_N); no longer J?.2 (B15_L3_P)
- net T2_1: now also J?.3 (B15_L7_P); no longer J?.4 (B15_L3_N)
- net T2_10: now also J?.23 (B15_L16_N); no longer J?.24 (RLED)
- net T2_11: now also J?.25 (B15_L16_P); no longer J?.26 (GLED)
- net T2_12: now also J?.27 (B15_L18_N); no longer J?.28 (B15_L11_P)
- net T2_13: now also J?.29 (B15_L18_P); no longer J?.30 (B15_L11_N)
- net T2_14: now also J?.31 (B15_L17_N); no longer J?.32 (SFP0_RSI)
- net T2_15: now also J?.33 (B15_L17_P); no longer J?.34 (SFP0_LOS)
- net T2_16: now also J?.37 (B15_L24_N); no longer J?.38 (SFP0_RS0)
- net T2_17: now also J?.39 (B15_L24_P); no longer J?.40 (SFP0_M-DEF0)
- net T2_18: now also J?.41 (B15_L19_N); no longer J?.42 (SFP0_TX_FAULT)
- net T2_19: now also J?.43 (B15_L19_P); no longer J?.44 (SFP0_TX_DIS)
- net T2_2: now also J?.5 (B15_L8_P); no longer J?.6 (B15_L5_P)
- net T2_20: now also J?.45 (B15_L21_N); no longer J?.46 (SFP0_SDA)
- net T2_21: now also J?.47 (B15_L21_P); no longer J?.48 (SFP0_SCL)
- net T2_22: now also J?.49 (B15_L23_P); no longer J?.50 (B15_L20_N)
- net T2_23: now also J?.51 (B15_L23_N); no longer J?.52 (B15_L20_P)
- net T2_24: now also J?.2 (B15_L3_P); no longer J?.1 (B15_L7_N)
- net T2_25: now also J?.4 (B15_L3_N); no longer J?.3 (B15_L7_P)
- net T2_26: now also J?.6 (B15_L5_P); no longer J?.5 (B15_L8_P)
- net T2_27: now also J?.8 (B15_L5_N); no longer J?.7 (B15_L8_N)
- net T2_28: now also J?.10 (B15_L4_N); no longer J?.9 (B15_L10_P)
- net T2_29: now also J?.12 (B15_L4_P); no longer J?.11 (B15_L10_N)
- net T2_3: now also J?.7 (B15_L8_N); no longer J?.8 (B15_L5_N)
- net T2_30: now also J?.14 (B15_L1_N); no longer J?.13 (B15_L9_P)
- net T2_31: now also J?.16 (B15_L1_P); no longer J?.15 (B15_L9_N)
- net T2_4: now also J?.9 (B15_L10_P); no longer J?.10 (B15_L4_N)
- net T2_5: now also J?.11 (B15_L10_N); no longer J?.12 (B15_L4_P)
- net T2_6: now also J?.13 (B15_L9_P); no longer J?.14 (B15_L1_N)
- net T2_7: now also J?.15 (B15_L9_N); no longer J?.16 (B15_L1_P)
- net T2_8: now also J?.19 (B15_L15_N); no longer J?.20 (B15_L2_N)
- net T2_9: now also J?.21 (B15_L15_P); no longer J?.22 (B15_L2_P)
- net TCK: now also J?.6 (Pin_6)
- net TDI: now also J?.10 (Pin_10)
- net TDO: now also J?.8 (Pin_8)
- net TMS: now also J?.4 (Pin_4)
- net ADC_CS_1: now reaches J?.53 (B34_L11_N)
- net ADC_SCLK_1: now reaches J?.55 (B34_L11_P)
- net ADC_SDI_1: now reaches J?.57 (B34_L12_N)
- net ADC_SDO_1: now reaches J?.59 (B34_L12_P)
- net ADC_CS_2: now reaches J?.75 (B34_L22_N)
- net ADC_SCLK_2: now reaches J?.77 (B34_L22_P)
- net ADC_SDI_2: now reaches J?.79 (B34_L23_N)
- net ADC_SDO_2: now reaches J?.81 (B34_L23_P)
- net VCC: now reaches J?.83 (3.3V_OUT)
- net VCC: now also J?.54 (3.3V_OUT), J?.6 (Pin_6), R?.1, R?.1, U?.3 (EN), J?.1 (Pin_1), J?.2 (Pin_2), PS?.1 (VCC), PS?.1 (VCC), PS?.1 (VCC), PS?.1 (VCC), PS?.1 (VCC), PS?.1 (VCC), U?.1 (VCC), U?.1 (VCC)
- new net FPGA_rx: J?.3 (Pin_3)
- new net FPGA_tx: J?.2 (Pin_2)
- no-connect marks 0 -> 20
Other:
- note added: "Ask Eric: Is this necessary?\n"
- note added: "Make a new symbol : 3v3_OUT\n"
- note added: "To sparkfun FT232RL"

Commit message: Readout Trenz in progress
Connections:
- net ADC_CS_1: now also J?.49 (B34_L10_P); no longer J?.53 (B34_L11_N)
- net ADC_CS_2: now also J?.93 (B14_L20_P); no longer J?.75 (B34_L22_N)
- net ADC_SCLK_1: now also J?.51 (B34_L10_N); no longer J?.55 (B34_L11_P)
- net ADC_SCLK_2: now also J?.95 (B14_L20_N); no longer J?.77 (B34_L22_P)
- net ADC_SDI_1: now also J?.53 (B34_L11_N); no longer J?.57 (B34_L12_N)
- net ADC_SDI_2: now also J?.97 (B14_L25); no longer J?.79 (B34_L23_N)
- net ADC_SDO_1: now also J?.55 (B34_L11_P); no longer J?.59 (B34_L12_P)
- net ADC_SDO_2: now also J?.99 (B14_L0); no longer J?.81 (B34_L23_P)
- net at J?.1 (Pin_1), J?.3 (Pin_3), J?.5 (Pin_5): no longer J?.61 (VCCIO34)
- net Val_Ext_n1: now reaches J?.63 (B34_L17_N)
- net Val_Ext_n1: now also J?.60 (B14_L8_P)
- net Val_Ext_p1: now reaches J?.65 (B34_L17_P)
- net Val_Ext_p1: now also J?.62 (B14_L8_N)
- net select_1: now reaches J?.67 (B34_L21_P)
- net select_1: now also J?.64 (B14_L9_P)
- net load_sc_1: now reaches J?.69 (B34_L21_N)
- net load_sc_1: now also J?.66 (B14_L9_N)
- net srin_read_1: now reaches J?.71 (B34_L19_N)
- net srin_read_1: now also J?.74 (B14_L11_N)
- net clk_read_1: now reaches J?.73 (B34_L19_P)
- net clk_read_1: now also J?.76 (B14_L11_P)
- net srout_read_1: now reaches J?.85 (B14_L24_N)
- net srout_read_1: now also J?.86 (B14_L13_N)
- net srout_sc_1: now reaches J?.87 (B14_L24_P)
- net srout_sc_1: now also J?.88 (B14_L13_P)
- net NOR32T_oc_1: now reaches J?.89 (B14_L23_N)
- net NOR32T_oc_1: now also J?.92 (B14_L19_P)
- net NOR32_oc_1: now reaches J?.91 (B14_L23_P)
- net NOR32_oc_1: now also J?.94 (B14_L19_N)
- net OR32_1: now reaches J?.93 (B14_L21_P)
- net OR32_1: now also J?.96 (B14_L22_N)
- net dig_out_1: now reaches J?.95 (B14_L21_N)
- net dig_out_1: now also J?.98 (B14_L22_P)
- net Raz_Chn_n1: now reaches J?.56 (B14_L5_P)
- net Raz_Chn_n1: now also J?.57 (B34_L12_N)
- net Raz_Chn_p1: now reaches J?.58 (B14_L5_N)
- net Raz_Chn_p1: now also J?.59 (B34_L12_P)
- net resetb_pa: now reaches J?.77 (B14_L10_N)
- net resetb_read_1: now reaches J?.78 (B14_L14_N)
- net resetb_read_1: now also J?.75 (B34_L22_N)
- net rstb_PSC: now reaches J?.79 (B14_L16_P)
- net srin_sc_1: now reaches J?.80 (B14_L14_P)
- net srin_sc_1: now also J?.77 (B34_L22_P)
- net pwr_on: now reaches J?.81 (B14_L16_N)
- net clk_sr_1: now reaches J?.82 (B14_L12_P)
- net clk_sr_1: now also J?.79 (B34_L23_N)
- net rstb_sr_1: now reaches J?.84 (B14_L12_N)
- net rstb_sr_1: now also J?.81 (B34_L23_P)
- net PS_global_trig: now reaches J?.85 (B14_L18_N)
- net PS_modeb_ext: now reaches J?.87 (B14_L18_P)
- net hold_lg: now reaches J?.89 (B14_L17_N)
- net hold_hg: now reaches J?.91 (B14_L17_P)
Other:
- note removed: "Make a new symbol : 3v3_OUT\n"
- moved on the sheet: J?, PS?

Commit message: Readout Trenz in progress
Connections:
- wire segments 265 -> 281
Changed lines of the file:
@@
 Text HLabel 3600 5600 2    50   Output ~ 0
 MGT_RX2_P
-Text HLabel 3600 5400 2    50   Input ~ 0
-MGT_TX2_N
-Text HLabel 3600 5300 2    50   Input ~ 0
-MGT_TX2_P
 $Comp
 L readout_trenz-rescue:C_Small-Device C?
@@
 Text HLabel 11200 3500 2    50   Output ~ 0
 CITIROC_IN_2
+Text HLabel 3600 5400 2    50   Input ~ 0
+MGT_TX2_N
+Text HLabel 3600 5300 2    50   Input ~ 0
+MGT_TX2_P
+Text Label -500 5850 2    50   ~ 0
+SFP0_TX_FAULT
+Wire Wire Line
+	-1000 5850 -500 5850
+Text Label -500 5950 2    50   ~ 0
+SFP0_TX_DIS
+Wire Wire Line
+	-1000 5950 -500 5950
+Text Label -500 6050 2    50   ~ 0
+SFP0_SDA
+Wire Wire Line
+	-1000 6050 -500 6050
+Text Label -500 6150 2    50   ~ 0
+SFP0_SCL
+Wire Wire Line
+	-1000 6150 -500 6150
+Text Label -500 6250 2    50   ~ 0
+SFP0_M-DEF0
+Wire Wire Line
+	-1000 6250 -500 6250
+Text Label -500 6350 2    50   ~ 0
+SFP0_RS0
+Wire Wire Line
+	-1000 6350 -500 6350
+Text Label -500 6450 2    50   ~ 0
+SFP0_LOS
+Wire Wire Line
+	-1000 6450 -500 6450
+Text Label -500 6550 2    50   ~ 0
+SFP0_RS1
+Wire Wire Line
+	-1000 6550 -500 6550
+Wire Wire Line
+	-1000 7000 -500 7000
+Wire Wire Line
+	-1000 7100 -500 7100
+Wire Wire Line
+	-1000 7200 -500 7200
+Wire Wire Line
+	-1000 7300 -500 7300
+Text Label -500 7000 2    50   ~ 0
+TMS
+Text Label -500 7100 2    50   ~ 0
+TCK
+Text Label -500 7200 2    50   ~ 0
+TDO
+Text Label -500 7300 2    50   ~ 0
+TDI
+Wire Wire Line
+	-1000 5650 -500 5650
+Text Label -500 5650 2    50   ~ 0
+MGT_RX2_N
+Wire Wire Line
+	-1000 5550 -500 5550
+Text Label -500 5550 2    50   ~ 0
+MGT_RX2_P
+Wire Wire Line
+	-1000 5350 -500 5350
+Text Label -500 5350 2    50   ~ 0
+MGT_TX2_N
+Wire Wire Line
+	-1000 5250 -500 5250
+Text Label -500 5250 2    50   ~ 0
+MGT_TX2_P
 Wire Bus Line
 	5350 3200 5350 3500

Commit message: Readout Trenz in progress
Parts:
- added R? (x2): 100, symbol readout_trenz-rescue:R-Device
- added R? (x2): 1k, symbol readout_trenz-rescue:R-Device
- added TP?: probe, symbol readout_trenz-rescue:TestPoint_2Pole-Connector
- added U?: CITIROC1A, Package_QFP:LQFP-160_24x24mm_P0.5mm, symbol readout:CITIROC1A
- added U?: Vcc0_1v8, symbol readout:VccAux
Connections:
- net labels added: NOR32T_oc_2, NOR32_oc_2, OR32_2, PS_global_trig_1, PS_modeb_ext_1, T1_[0,17], T1_[18,31], T2_[0..23], T2_[0..31], T2_[24..31], dig_out_2, hold_hg_1, hold_lg_1, pwr_on_1, resetb_pa_1, rstb_PSC_1
- net labels removed: T1_[0.23], T1_[24,31], T2_[0,23], T2_[0,31], T2_[24,31]
- wire segments 281 -> 381
Other:
- note added: "All other control signals go to B34\n"
- note added: "Go to the same bank as T\n"
- note added: "from bank?"
- moved on the sheet: C?, J?, PS?

Commit message: Readout Trenz in progress
Connections:
- net labels added: PS_global_trig_2, PS_modeb_ext_2, Raz_Chn_n2, Raz_Chn_p2, Val_Ext_n2, Val_Ext_p2, clk_read_2, clk_sr_2, hold_hg_2, hold_lg_2, load_sc_2, pwr_on_2, resetb_pa_2, resetb_read_2, rstb_PSC_2, rstb_sr_2, select_2, srin_read_2, srin_sc_2, srout_read_2, srout_sc_2
- wire segments 381 -> 390
Other:
- moved on the sheet: PS?

Commit message: -
Parts:
- removed R? (x2): 100, symbol readout_trenz-rescue:R-Device
- removed R? (x2): 1k, symbol readout_trenz-rescue:R-Device
- removed TP?: probe, symbol readout_trenz-rescue:TestPoint_2Pole-Connector
- removed U?: CITIROC1A, Package_QFP:LQFP-160_24x24mm_P0.5mm, symbol readout:CITIROC1A
- removed U?: Vcc0_1v8, symbol readout:VccAux
Connections:
- net labels added: UART_FROM_MOD, UART_TO_MOD
- net labels removed: PS_global_trig, PS_modeb_ext, hold_hg, hold_lg, pwr_on, resetb_pa, rstb_PSC
- wire segments 390 -> 303
Other:
- note removed: "All other control signals go to B34\n"
- note removed: "Go to the same bank as T\n"
- note removed: "from bank?"
- moved on the sheet: J?
