File: hardware/readout_trenz/POWER.sch (KiCad schematic (older format))
At the start: 36 parts

Commit message: Readout Trenz in progress
Parts:
- added J? (x2): Conn_02x10_Odd_Even, symbol Connector_Generic:Conn_02x10_Odd_Even
- added J?: Conn_Coaxial_Power, symbol Connector:Conn_Coaxial_Power
- added JP? (x2): Jumper, symbol Device:Jumper
Connections:
- net labels removed: +12V
- wire segments 137 -> 175
Other:
- note added: "+12V"
- moved on the sheet: R?
Changed lines of the file:
@@
 Wire Wire Line
 	3550 2300 3450 2300
-Wire Wire Line
-	900  2300 900  2150
 $Comp
 L Device:C_Small C?
@@
 L Device:R R?
 U 1 1 60F71B32
-P 6200 5300
-F 0 "R?" V 6270 5346 50  0000 L CNN
-F 1 "4.7k" V 6200 5200 50  0000 L CNN
-F 2 "Resistor_SMD:R_0603_1608Metric_Pad1.05x0.95mm_HandSolder" V 6130 5300 50  0001 C CNN
-F 3 "~" H 6200 5300 50  0001 C CNN
-	1    6200 5300
-	0    -1   -1   0
+P 6350 5450
+F 0 "R?" V 6420 5496 50  0000 L CNN
+F 1 "4.7k" V 6350 5350 50  0000 L CNN
+F 2 "Resistor_SMD:R_0603_1608Metric_Pad1.05x0.95mm_HandSolder" V 6280 5450 50  0001 C CNN
+F 3 "~" H 6350 5450 50  0001 C CNN
+	1    6350 5450
+	-1   0    0    1
 $EndComp
 $Comp
 L power:GNDA #PWR?
 U 1 1 60F7AF0B
-P 6050 5400
+P 6350 5700
 AR Path="/6076C700/60F7AF0B" Ref="#PWR?"  Part="1"
 AR Path="/62251D77/60F7AF0B" Ref="#PWR?"  Part="1"
-F 0 "#PWR?" H 6050 5150 50  0001 C CNN
-F 1 "GNDA" H 6050 5250 50  0000 C CNN
-F 2 "" H 6050 5400 50  0001 C CNN
-F 3 "" H 6050 5400 50  0001 C CNN
-	1    6050 5400
-	1    0    0    -1
-$EndComp
-Wire Wire Line
-	6050 5300 6050 5400
+F 0 "#PWR?" H 6350 5450 50  0001 C CNN
+F 1 "GNDA" H 6350 5550 50  0000 C CNN
+F 2 "" H 6350 5700 50  0001 C CNN
+F 3 "" H 6350 5700 50  0001 C CNN
+	1    6350 5700
+	1    0    0    -1
+$EndComp
+Wire Wire Line
+	6350 5600 6350 5700
 Wire Wire Line
 	6350 2100 6350 1500
@@
 Text HLabel 6350 1500 0    50   Input ~ 0
 ENABLE
-$Comp
-L power:+12V #PWR?
-U 1 1 60FEABA1
-P 900 2150
-F 0 "#PWR?" H 900 2000 50  0001 C CNN
-F 1 "+12V" H 915 2323 50  0000 C CNN
-F 2 "" H 900 2150 50  0001 C CNN
-F 3 "" H 900 2150 50  0001 C CNN
-	1    900  2150
-	1    0    0    -1
-$EndComp
-Wire Wire Line
-	900  2300 1200 2300
 $Comp
 L Device:LED_Small D?
@@
 Text HLabel 3500 5600 1    50   Input ~ 0
 ENABLE
+$Comp
+L Connector_Generic:Conn_02x10_Odd_Even J?
+U 1 1 60DE5052
+P 8150 -1050
+F 0 "J?" H 8200 -433 50  0000 C CNN
+F 1 "Conn_02x10_Odd_Even" H 8200 -524 50  0000 C CNN
+F 2 "" H 8150 -1050 50  0001 C CNN
+F 3 "~" H 8150 -1050 50  0001 C CNN
+	1    8150 -1050
+	1    0    0    -1
+$EndComp
+$Comp
+L Connector_Generic:Conn_02x10_Odd_Even J?
+U 1 1 60DE60C3
+P 9100 -1050
+F 0 "J?" H 9150 -433 50  0000 C CNN
+F 1 "Conn_02x10_Odd_Even" H 9150 -524 50  0000 C CNN
+F 2 "" H 9100 -1050 50  0001 C CNN
+F 3 "~" H 9100 -1050 50  0001 C CNN
+	1    9100 -1050
+	1    0    0    -1
+$EndComp
+Wire Wire Line
+	1000 2300 1000 2400
+$Comp
+L power:GNDA #PWR?
+U 1 1 60DF7A2C
+P 1000 2400
+AR Path="/6076C700/60DF7A2C" Ref="#PWR?"  Part="1"
+AR Path="/62251D77/60DF7A2C" Ref="#PWR?"  Part="1"
+F 0 "#PWR?" H 1000 2150 50  0001 C CNN
+F 1 "GNDA" H 1000 2250 50  0000 C CNN
+F 2 "" H 1000 2400 50  0001 C CNN
+F 3 "" H 1000 2400 50  0001 C CNN
+	1    1000 2400
+	-1   0    0    -1
+$EndComp
+Wire Wire Line
+	1000 2300 1200 2300
+Text Notes 1100 1950 0    100  ~ 0
++12V
+$Comp
+L Connector:Conn_Coaxial_Power J?
+U 1 1 60E19C4C
+P 7300 -1450
+F 0 "J?" V 7525 -1500 50  0000 C CNN
+F 1 "Conn_Coaxial_Power" V 7434 -1500 50  0000 C CNN
+F 2 "" H 7300 -1500 50  0001 C CNN
+F 3 "~" H 7300 -1500 50  0001 C CNN
+	1    7300 -1450
+	0    -1   -1   0
+$EndComp
+Wire Wire Line
+	7000 -1450 7000 -1350
+$Comp
+L power:GNDA #PWR?
+U 1 1 60E19C58
+P 7000 -1350
+AR Path="/6076C700/60E19C58" Ref="#PWR?"  Part="1"
+AR Path="/62251D77/60E19C58" Ref="#PWR?"  Part="1"
+F 0 "#PWR?" H 7000 -1600 50  0001 C CNN
+F 1 "GNDA" H 7000 -1500 50  0000 C CNN
+F 2 "" H 7000 -1350 50  0001 C CNN
+F 3 "" H 7000 -1350 50  0001 C CNN
+	1    7000 -1350
+	-1   0    0    -1
+$EndComp
+Wire Wire Line
+	7000 -1450 7200 -1450
+Text Notes 7100 -1800 0    100  ~ 0
++12V
+Wire Wire Line
+	7500 -1450 7850 -1450
+Wire Wire Line
+	7850 -1450 7850 -1350
+Wire Wire Line
+	7850 -1150 7950 -1150
+Connection ~ 7850 -1450
+Wire Wire Line
+	7850 -1450 7950 -1450
+Wire Wire Line
+	7850 -1250 7950 -1250
+Connection ~ 7850 -1250
+Wire Wire Line
+	7850 -1250 7850 -1150
+Wire Wire Line
+	7850 -1350 7950 -1350
+Connection ~ 7850 -1350
+Wire Wire Line
+	7850 -1350 7850 -1250
+Wire Wire Line
+	7950 -850 7850 -850
+Wire Wire Line
+	7850 -850 7850 -750
+Wire Wire Line
+	7850 -550 7950 -550
+Connection ~ 7850 -550
+Wire Wire Line
+	7850 -550 7850 -500
+Wire Wire Line
+	7850 -650 7950 -650
+Connection ~ 7850 -650
+Wire Wire Line
+	7850 -650 7850 -550
+Wire Wire Line
+	7850 -750 7950 -750
+Connection ~ 7850 -750
+Wire Wire Line
+	7850 -750 7850 -650
+$Comp
+L power:GNDA #PWR?
+U 1 1 60E78581
+P 7850 -500
+AR Path="/6076C700/60E78581" Ref="#PWR?"  Part="1"
+AR Path="/62251D77/60E78581" Ref="#PWR?"  Part="1"
+F 0 "#PWR?" H 7850 -750 50  0001 C CNN
+F 1 "GNDA" H 7850 -650 50  0000 C CNN
+F 2 "" H 7850 -500 50  0001 C CNN
+F 3 "" H 7850 -500 50  0001 C CNN
+	1    7850 -500
+	-1   0    0    -1
+$EndComp
+Wire Wire Line
+	9400 -850 9500 -850
+Wire Wire Line
+	9500 -850 9500 -750
+Wire Wire Line
+	9500 -550 9400 -550
+Connection ~ 9500 -550
+Wire Wire Line
+	9500 -550 9500 -500
+Wire Wire Line
+	9500 -650 9400 -650
+Connection ~ 9500 -650
+Wire Wire Line
+	9500 -650 9500 -550
+Wire Wire Line
+	9500 -750 9400 -750
+Connection ~ 9500 -750
+Wire Wire Line
+	9500 -750 9500 -650
+$Comp
+L power:GNDA #PWR?
+U 1 1 60E823D3
+P 9500 -500
+AR Path="/6076C700/60E823D3" Ref="#PWR?"  Part="1"
+AR Path="/62251D77/60E823D3" Ref="#PWR?"  Part="1"
+F 0 "#PWR?" H 9500 -750 50  0001 C CNN
+F 1 "GNDA" H 9500 -650 50  0000 C CNN
+F 2 "" H 9500 -500 50  0001 C CNN
+F 3 "" H 9500 -500 50  0001 C CNN
+	1    9500 -500
+	1    0    0    -1
+$EndComp
+Wire Wire Line
+	9400 -1450 9500 -1450
+Wire Wire Line
+	9500 -1450 9500 -1350
+Wire Wire Line
+	9500 -1350 9400 -1350
+Wire Wire Line
+	9500 -1450 9900 -1450
+Connection ~ 9500 -1450
+$Comp
+L Device:Jumper JP?
+U 1 1 60E9F02D
+P 10200 -1450
+F 0 "JP?" H 10200 -1186 50  0000 C CNN
+F 1 "Jumper" H 10200 -1277 50  0000 C CNN
+F 2 "" H 10200 -1450 50  0001 C CNN
+F 3 "~" H 10200 -1450 50  0001 C CNN
+	1    10200 -1450
+	1    0    0    -1
+$EndComp
+Wire Wire Line
+	9400 -1250 9500 -1250
+Wire Wire Line
+	9500 -1250 9500 -1150
+Wire Wire Line
+	9500 -1150 9400 -1150
+Wire Wire Line
+	9500 -1250 9900 -1250
+Connection ~ 9500 -1250
+$Comp
+L Device:Jumper JP?
+U 1 1 60EA0402
+P 10200 -1250
+F 0 "JP?" H 10200 -986 50  0000 C CNN
+F 1 "Jumper" H 10200 -1077 50  0000 C CNN
+F 2 "" H 10200 -1250 50  0001 C CNN
+F 3 "~" H 10200 -1250 50  0001 C CNN
+	1    10200 -1250
+	1    0    0    -1
+$EndComp
+Wire Wire Line
+	10500 -1450 10600 -1450
+Wire Wire Line
+	10500 -1250 10600 -1250
+Wire Wire Line
+	10600 -1250 10600 -1450
+Connection ~ 10600 -1450
+Wire Wire Line
+	10600 -1450 11000 -1450
 $EndSCHEMATC

Commit message: File Clean pu done
Parts:
- removed C?: 330u, Capacitor_SMD:C_0603_1608Metric_Pad1.05x0.95mm_HandSolder, symbol Device:C_Small
- removed C?: 10u, Capacitor_SMD:C_0603_1608Metric_Pad1.05x0.95mm_HandSolder, symbol Device:C_Small
- removed C? (x2): .1u, Capacitor_SMD:C_0603_1608Metric_Pad1.05x0.95mm_HandSolder, symbol Device:C_Small
- removed C? (x2): 47u, Capacitor_SMD:C_0603_1608Metric_Pad1.05x0.95mm_HandSolder, symbol Device:C_Small
- removed D? (x3): LED_Small, symbol Device:LED_Small
- removed J?: Conn_Coaxial_Power, symbol Connector:Conn_Coaxial_Power
- removed R? (x3): R_Small, symbol Device:R_Small
- removed R?: 250k, Resistor_SMD:R_0603_1608Metric_Pad1.05x0.95mm_HandSolder, symbol Device:R
- removed R?: 22k, Resistor_SMD:R_0603_1608Metric_Pad1.05x0.95mm_HandSolder, symbol Device:R
- removed R?: 12k, Resistor_SMD:R_0603_1608Metric_Pad1.05x0.95mm_HandSolder, symbol Device:R
- removed R?: 10k, Resistor_SMD:R_0603_1608Metric_Pad1.05x0.95mm_HandSolder, symbol Device:R
- removed U?: LTM4622, symbol readout:LTM4622
- added D? (x2): LED_Small, symbol Device:LED_Small
- added R? (x2): R_Small, symbol Device:R_Small
Connections:
- net GNDA: now also D?.1 (K), D?.1 (K)
- net at J?.1 (Pin_1), J?.3 (Pin_3): now also J?.5 (Pin_5), J?.7 (Pin_7), JP?.2, JP?.2, R?.1
- net at J?.1 (Pin_1), J?.2 (Ext), J?.3 (Pin_3)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: now also R?.1
- new net: D?.2 (A), R?.2 (x2)
- no-connect marks 4 -> 0
Other:
- moved on the sheet: J?, JP?

Commit message: Finishing Readout Schematic
Parts:
- added C2, C3, C4: 0.1uF, symbol Device:C_Small
- gave numbers to parts that had none: 27
Connections:
- net at J7.8 (Pin_8), U5.2 (IN): now also C4.1
- net at J7.6 (Pin_6), U4.2 (IN): now also C3.1
- net at J7.4 (Pin_4), U6.2 (IN): now also C2.1
- net GNDA renamed GNDD
- net GNDD: now also C2.2, C3.2, C4.2
- no-connect marks 0 -> 24
Other:
- moved on the sheet: D2, R4

Commit message: Readout Schematic in Completion
Parts:
- added C11, C12, C13: 10uF, symbol Device:C_Small
- added C3: 1uF, symbol Device:C_Small
- added C4: 10nF, symbol Device:C_Small
- added C5: 2.2uF, symbol Device:C_Small
- added Q1: DMN67D7L, Package_TO_SOT_SMD:SOT-23, symbol Transistor_FET:DMN67D7L
- added U4: LP2985-5.0, Package_TO_SOT_SMD:SOT-23-5, symbol Regulator_Linear:LP2985-5.0
- C10: renamed from C5; value C_Small -> 1u
- C6: renamed from C1; value C_Small -> 1u
- C7: renamed from C2; value 0.1uF -> 10uF
- C8: renamed from C3; value 0.1uF -> 10uF
- C9: renamed from C4; value 0.1uF -> 10uF
- R10: renamed from R8; value R_Small -> 550
- R11: renamed from R9; value R_Small -> 550
- R12: renamed from R10; value R_Small -> 500
- R5: renamed from R3; value R_Small -> 4.9k
- R6: renamed from R5; value R_Small -> 900
- R9: renamed from R7; value R_Small -> 1k
- renumbered D3 to D2, D2 to D3, D5 to D4, D6 to D5, D7 to D6, D4 to D7, R6 to R7, R4 to R8, U3 to U5, U4 to U7, U5 to U8
Connections:
- net labels added: 5V_DAC, VCC
- wire segments 122 -> 154
Other:
- moved on the sheet: D1, D3, D7, R5, R8, U6

Commit message: _
Parts:
- removed D7: LED_Small, symbol Device:LED_Small
- removed J5, J6: Conn_02x10_Odd_Even, symbol Connector_Generic:Conn_02x10_Odd_Even
- removed R9: 1k, symbol Device:R_Small
- added D2, D8: LED_Small, symbol Device:LED_Small
- added J5: Conn_02x05_Odd_Even, Connector_PinHeader_2.54mm:PinHeader_2x05_P2.54mm_Vertical, symbol Connector_Generic:Conn_02x05_Odd_Even
- added J6, J7: Conn_01x10, Connector_PinHeader_2.54mm:PinHeader_2x05_P2.54mm_Vertical, symbol Connector_Generic:Conn_01x10
- added R13: 550, symbol Device:R_Small
- added R6: 1.4k, symbol Device:R_Small
- renumbered D2 to D3, D3 to D4, D4 to D5, D5 to D6, D6 to D7, J7 to J8, R6 to R7, R7 to R8, R8 to R9
Connections:
- net labels added: BIAS1, BIAS2, BIAS3, BIAS4, BIAS[1..4], GNDA
- wire segments 154 -> 162
- no-connect marks 24 -> 6

Commit message: _
Parts:
- C10, C11, C12, C13, C3, C4, C5, C6, C7, C8, C9: footprint (none) -> Capacitor_SMD:C_0603_1608Metric_Pad1.05x0.95mm_HandSolder
- R10, R11, R12, R13, R5, R6, R7, R9: footprint (none) -> Resistor_SMD:R_0603_1608Metric_Pad1.05x0.95mm_HandSolder
Changed lines of the file:
@@
 F 0 "C6" H 6242 2246 50  0000 L CNN
 F 1 "1u" H 6242 2155 50  0000 L CNN
-F 2 "" H 6150 2200 50  0001 C CNN
+F 2 "Capacitor_SMD:C_0603_1608Metric_Pad1.05x0.95mm_HandSolder" H 6150 2200 50  0001 C CNN
 F 3 "~" H 6150 2200 50  0001 C CNN
 	1    6150 2200
@@
 F 0 "C10" H 7292 2246 50  0000 L CNN
 F 1 "1u" H 7292 2155 50  0000 L CNN
-F 2 "" H 7200 2200 50  0001 C CNN
+F 2 "Capacitor_SMD:C_0603_1608Metric_Pad1.05x0.95mm_HandSolder" H 7200 2200 50  0001 C CNN
 F 3 "~" H 7200 2200 50  0001 C CNN
 	1    7200 2200
@@
 F 0 "R9" H 6609 1546 50  0000 L CNN
 F 1 "R_Small" H 6609 1455 50  0000 L CNN
-F 2 "" H 6550 1500 50  0001 C CNN
+F 2 "Resistor_SMD:R_0603_1608Metric_Pad1.05x0.95mm_HandSolder" H 6550 1500 50  0001 C CNN
 F 3 "~" H 6550 1500 50  0001 C CNN
 	1    6550 1500
@@
 F 0 "R11" H 7809 4246 50  0000 L CNN
 F 1 "550" H 7809 4155 50  0000 L CNN
-F 2 "" H 7750 4200 50  0001 C CNN
+F 2 "Resistor_SMD:R_0603_1608Metric_Pad1.05x0.95mm_HandSolder" H 7750 4200 50  0001 C CNN
 F 3 "~" H 7750 4200 50  0001 C CNN
 	1    7750 4200
@@
 F 0 "R12" H 7809 5246 50  0000 L CNN
 F 1 "500" H 7809 5155 50  0000 L CNN
-F 2 "" H 7750 5200 50  0001 C CNN
+F 2 "Resistor_SMD:R_0603_1608Metric_Pad1.05x0.95mm_HandSolder" H 7750 5200 50  0001 C CNN
 F 3 "~" H 7750 5200 50  0001 C CNN
 	1    7750 5200
@@
 F 0 "R10" H 7809 3246 50  0000 L CNN
 F 1 "550" H 7809 3155 50  0000 L CNN
-F 2 "" H 7750 3200 50  0001 C CNN
+F 2 "Resistor_SMD:R_0603_1608Metric_Pad1.05x0.95mm_HandSolder" H 7750 3200 50  0001 C CNN
 F 3 "~" H 7750 3200 50  0001 C CNN
 	1    7750 3200
@@
 F 0 "R5" H 1959 2246 50  0000 L CNN
 F 1 "4.9k" H 1959 2155 50  0000 L CNN
-F 2 "" H 1900 2200 50  0001 C CNN
+F 2 "Resistor_SMD:R_0603_1608Metric_Pad1.05x0.95mm_HandSolder" H 1900 2200 50  0001 C CNN
 F 3 "~" H 1900 2200 50  0001 C CNN
 	1    1900 2200
@@
 F 0 "R7" H 5059 2246 50  0000 L CNN
 F 1 "900" H 5059 2155 50  0000 L CNN
-F 2 "" H 5000 2200 50  0001 C CNN
+F 2 "Resistor_SMD:R_0603_1608Metric_Pad1.05x0.95mm_HandSolder" H 5000 2200 50  0001 C CNN
 F 3 "~" H 5000 2200 50  0001 C CNN
 	1    5000 2200
@@
 F 0 "C7" H 6242 3246 50  0000 L CNN
 F 1 "10uF" H 6242 3155 50  0000 L CNN
-F 2 "" H 6150 3200 50  0001 C CNN
+F 2 "Capacitor_SMD:C_0603_1608Metric_Pad1.05x0.95mm_HandSolder" H 6150 3200 50  0001 C CNN
 F 3 "~" H 6150 3200 50  0001 C CNN
 	1    6150 3200
@@
 F 0 "C8" H 6242 4246 50  0000 L CNN
 F 1 "10uF" H 6242 4155 50  0000 L CNN
-F 2 "" H 6150 4200 50  0001 C CNN
+F 2 "Capacitor_SMD:C_0603_1608Metric_Pad1.05x0.95mm_HandSolder" H 6150 4200 50  0001 C CNN
 F 3 "~" H 6150 4200 50  0001 C CNN
 	1    6150 4200
@@
 F 0 "C9" H 6242 5246 50  0000 L CNN
 F 1 "10uF" H 6242 5155 50  0000 L CNN
-F 2 "" H 6150 5200 50  0001 C CNN
+F 2 "Capacitor_SMD:C_0603_1608Metric_Pad1.05x0.95mm_HandSolder" H 6150 5200 50  0001 C CNN
 F 3 "~" H 6150 5200 50  0001 C CNN
 	1    6150 5200
@@
 F 0 "C11" H 7692 3246 50  0000 L CNN
 F 1 "10uF" H 7692 3155 50  0000 L CNN
-F 2 "" H 7600 3200 50  0001 C CNN
+F 2 "Capacitor_SMD:C_0603_1608Metric_Pad1.05x0.95mm_HandSolder" H 7600 3200 50  0001 C CNN
 F 3 "~" H 7600 3200 50  0001 C CNN
 	1    7600 3200
@@
 F 0 "C12" H 7692 4246 50  0000 L CNN
 F 1 "10uF" H 7692 4155 50  0000 L CNN
-F 2 "" H 7600 4200 50  0001 C CNN
+F 2 "Capacitor_SMD:C_0603_1608Metric_Pad1.05x0.95mm_HandSolder" H 7600 4200 50  0001 C CNN
 F 3 "~" H 7600 4200 50  0001 C CNN
 	1    7600 4200
@@
 F 0 "C13" H 7692 5246 50  0000 L CNN
 F 1 "10uF" H 7692 5155 50  0000 L CNN
-F 2 "" H 7600 5200 50  0001 C CNN
+F 2 "Capacitor_SMD:C_0603_1608Metric_Pad1.05x0.95mm_HandSolder" H 7600 5200 50  0001 C CNN
 F 3 "~" H 7600 5200 50  0001 C CNN
 	1    7600 5200
@@
 F 0 "C3" H 1442 4546 50  0000 L CNN
 F 1 "1uF" H 1442 4455 50  0000 L CNN
-F 2 "" H 1350 4500 50  0001 C CNN
+F 2 "Capacitor_SMD:C_0603_1608Metric_Pad1.05x0.95mm_HandSolder" H 1350 4500 50  0001 C CNN
 F 3 "~" H 1350 4500 50  0001 C CNN
 	1    1350 4500
@@
 F 0 "C4" H 2392 4546 50  0000 L CNN
 F 1 "10nF" H 2392 4455 50  0000 L CNN
-F 2 "" H 2300 4500 50  0001 C CNN
+F 2 "Capacitor_SMD:C_0603_1608Metric_Pad1.05x0.95mm_HandSolder" H 2300 4500 50  0001 C CNN
 F 3 "~" H 2300 4500 50  0001 C CNN
 	1    2300 4500
@@
 F 0 "C5" H 2742 4546 50  0000 L CNN
 F 1 "2.2uF" H 2742 4455 50  0000 L CNN
-F 2 "" H 2650 4500 50  0001 C CNN
+F 2 "Capacitor_SMD:C_0603_1608Metric_Pad1.05x0.95mm_HandSolder" H 2650 4500 50  0001 C CNN
 F 3 "~" H 2650 4500 50  0001 C CNN
 	1    2650 4500
@@
 F 0 "R6" H 3109 4396 50  0000 L CNN
 F 1 "1.4k" H 3109 4305 50  0000 L CNN
-F 2 "" H 3050 4350 50  0001 C CNN
+F 2 "Resistor_SMD:R_0603_1608Metric_Pad1.05x0.95mm_HandSolder" H 3050 4350 50  0001 C CNN
 F 3 "~" H 3050 4350 50  0001 C CNN
 	1    3050 4350
@@
 F 0 "R13" V 8100 2250 50  0000 L CNN
 F 1 "550" V 8159 2255 50  0000 L CNN
-F 2 "" H 8100 2300 50  0001 C CNN
+F 2 "Resistor_SMD:R_0603_1608Metric_Pad1.05x0.95mm_HandSolder" H 8100 2300 50  0001 C CNN
 F 3 "~" H 8100 2300 50  0001 C CNN
 	1    8100 2300

Commit message: Readout Preliminary Schematic Made
Parts:
- U4: Item Cost (none) -> $0.66; MFN (none) -> LP2985A-50DBVT; Manufacturer (none) -> Texas Instruments; Supplier (none) -> Digi-Key; Supplier P/N (none) -> 296-32159-1-ND
- U5: Item Cost (none) -> $0.53; MFN (none) -> NCP718ASN180T1G; Manufacturer (none) -> ON Semiconductor; Supplier (none) -> Digi-Key; Supplier P/N (none) -> NCP718ASN180T1GOSCT-ND
- U6, U7, U8: Item Cost (none) -> $6.69; MFN (none) -> LT1963AEQ-3.3#PBF; Manufacturer (none) -> Analog Devices Inc.; Supplier (none) -> Digi-Key; Supplier P/N (none) -> LT1963AEQ-3.3#PBF-ND
Changed lines of the file:
@@
 F 2 "Package_TO_SOT_SMD:SOT-23-5" H 6900 2450 50  0001 C CNN
 F 3 "https://www.onsemi.com/pub/Collateral/NCP718-D.PDF" H 6900 2600 50  0001 C CNN
+F 4 "$0.53" H 6900 2100 50  0001 C CNN "Item Cost"
+F 5 "ON Semiconductor" H 6900 2100 50  0001 C CNN "Manufacturer"
+F 6 "NCP718ASN180T1G" H 6900 2100 50  0001 C CNN "MFN"
+F 7 "Digi-Key" H 6900 2100 50  0001 C CNN "Supplier"
+F 8 "NCP718ASN180T1GOSCT-ND" H 6900 2100 50  0001 C CNN "Supplier P/N"
 	1    6900 2100
 	1    0    0    -1
@@
 F 2 "Package_TO_SOT_SMD:TO-263-5_TabPin3" H 6900 4650 50  0001 C CNN
 F 3 "https://www.analog.com/media/en/technical-documentation/data-sheets/1963aff.pdf" H 6900 4550 50  0001 C CNN
+F 4 "$6.69" H 6900 5100 50  0001 C CNN "Item Cost"
+F 5 "LT1963AEQ-3.3#PBF" H 6900 5100 50  0001 C CNN "MFN"
+F 6 "Analog Devices Inc." H 6900 5100 50  0001 C CNN "Manufacturer"
+F 7 "Digi-Key" H 6900 5100 50  0001 C CNN "Supplier"
+F 8 "LT1963AEQ-3.3#PBF-ND" H 6900 5100 50  0001 C CNN "Supplier P/N"
 	1    6900 5100
 	1    0    0    -1
@@
 F 2 "Package_TO_SOT_SMD:TO-263-5_TabPin3" H 6900 3650 50  0001 C CNN
 F 3 "https://www.analog.com/media/en/technical-documentation/data-sheets/1963aff.pdf" H 6900 3550 50  0001 C CNN
+F 4 "$6.69" H 6900 4100 50  0001 C CNN "Item Cost"
+F 5 "LT1963AEQ-3.3#PBF" H 6900 4100 50  0001 C CNN "MFN"
+F 6 "Analog Devices Inc." H 6900 4100 50  0001 C CNN "Manufacturer"
+F 7 "Digi-Key" H 6900 4100 50  0001 C CNN "Supplier"
+F 8 "LT1963AEQ-3.3#PBF-ND" H 6900 4100 50  0001 C CNN "Supplier P/N"
 	1    6900 4100
 	1    0    0    -1
@@
 F 2 "Package_TO_SOT_SMD:TO-263-5_TabPin3" H 6900 2650 50  0001 C CNN
 F 3 "https://www.analog.com/media/en/technical-documentation/data-sheets/1963aff.pdf" H 6900 2550 50  0001 C CNN
+F 4 "$6.69" H 6900 3100 50  0001 C CNN "Item Cost"
+F 5 "Analog Devices Inc." H 6900 3100 50  0001 C CNN "Manufacturer"
+F 6 "LT1963AEQ-3.3#PBF" H 6900 3100 50  0001 C CNN "MFN"
+F 7 "Digi-Key" H 6900 3100 50  0001 C CNN "Supplier"
+F 8 "LT1963AEQ-3.3#PBF-ND" H 6900 3100 50  0001 C CNN "Supplier P/N"
 	1    6900 3100
 	1    0    0    -1
@@
 F 2 "Package_TO_SOT_SMD:SOT-23-5" H 1900 4575 50  0001 C CNN
 F 3 "http://www.ti.com/lit/ds/symlink/lp2985.pdf" H 1900 4250 50  0001 C CNN
+F 4 "$0.66" H 1900 4250 50  0001 C CNN "Item Cost"
+F 5 "Texas Instruments" H 1900 4250 50  0001 C CNN "Manufacturer"
+F 6 "LP2985A-50DBVT" H 1900 4250 50  0001 C CNN "MFN"
+F 7 "Digi-Key" H 1900 4250 50  0001 C CNN "Supplier"
+F 8 "296-32159-1-ND" H 1900 4250 50  0001 C CNN "Supplier P/N"
 	1    1900 4250
 	1    0    0    -1
@@
 Wire Wire Line
 	7700 2500 7700 2000
+Connection ~ 7700 2000
+Wire Wire Line
+	7700 2000 8000 2000
 Wire Bus Line
 	2600 5650 2600 5950
-Connection ~ 7700 2000
-Wire Wire Line
-	7700 2000 8000 2000
 $EndSCHEMATC

Commit message: Footprints Assigned
Parts:
- removed J8: Conn_02x04_Odd_Even, symbol Connector_Generic:Conn_02x04_Odd_Even
- D1, D2, D3, D4, D5, D6, D7, D8: footprint (none) -> LED_THT:LED_D3.0mm
- J4: footprint (none) -> Connector_BarrelJack:BarrelJack_Wuerth_6941xx301002; Item Cost (none) -> $0.96; MFN (none) -> 694106301002; Manufacturer (none) -> Würth Elektronik; Supplier  (none) -> Digi-Key; Supplier P/N (none) -> 732-5930-ND
- JP1, JP2: footprint (none) -> Connector_PinHeader_2.54mm:PinHeader_1x23_P2.54mm_Vertical
- renumbered U4 to U2, U5 to U3, U6 to U4, U7 to U5, U8 to U6
Connections:
- wire segments 162 -> 158
Other:
- moved on the sheet: C3, C4, C5, D1, D2, D3, J4, JP1, JP2, R5, R6, R7
