File: hardware/readout_trenz/CITIROC_1.sch (KiCad schematic (older format))
At the start: 132 parts, among them J11 BNC, J12 conn, J13 GPIO Header, U18 CITIROC1A, U19 SN74AXC2T45DCTR, U20 SN74AXC2T45DCTR, U21 NLSV8T244, U22 NLSV8T244, U23 DS90LV027A, U24 ADS7955, U25 REF5025, U26 NLSV4T244E, U9 CITIROC1A

Commit message: _
Parts:
- removed C86, C88: 4.7u, Capacitor_SMD:C_0603_1608Metric_Pad1.05x0.95mm_HandSolder, symbol Device:C_Small
- removed C87: 47u, Capacitor_SMD:C_0603_1608Metric_Pad1.05x0.95mm_HandSolder, symbol Device:C_Small
- removed C90, C91, C92, C93: .47u, Capacitor_SMD:C_0603_1608Metric_Pad1.05x0.95mm_HandSolder, symbol Device:C_Small
- removed R85, R86: 100, Resistor_SMD:R_0603_1608Metric_Pad1.05x0.95mm_HandSolder, symbol Device:R
- added C19, C20, C21, C22, C23, C24, C25, C26, C27, C28, C29, C30, C31, C32: 0.1uF, symbol Device:C_Small
- renumbered C96 to C110, C97 to C111, C98 to C112, C99 to C113, C100 to C114, C101 to C115, C102 to C116, C103 to C117, C104 to C118, C105 to C119, C106 to C120, C107 to C121, C108 to C122, C109 to C123, C110 to C124, C111 to C125, C112 to C126, C113 to C127, C114 to C128, C115 to C129, C116 to C130, C117 to C131, C118 to C132, C119 to C133, C120 to C134, C121 to C135, C122 to C136, C123 to C137, C124 to C138, C125 to C139, C126 to C140, C127 to C141, C128 to C142, C129 to C143, C130 to C144, C135 to C149, C136 to C150, C137 to C151, C138 to C152, C141 to C155, C142 to C156, C145 to C159, C146 to C160, C149 to C163, C150 to C164, C24 to C17, C25 to C18, C61 to C68, C62 to C69, C63 to C70, C64 to C71, C69 to C76, C70 to C77, C73 to C80, C74 to C81, C77 to C84, C78 to C85, C81 to C88, C82 to C89, C83 to C90, C84 to C91, C85 to C92, C89 to C93, J11 to J12, J12 to J13, J13 to J14, R103 to R100, R104 to R101, R105 to R102, R106 to R103, R60 to R59, R61 to R60, R62 to R61, R63 to R62, R64 to R63, R65 to R64, R66 to R65, R67 to R66, R68 to R67, R69 to R68, R70 to R69, R71 to R70, R72 to R71, R73 to R72, R74 to R73, R75 to R74, R76 to R75, R77 to R76, R78 to R77, R79 to R78, R80 to R79, R81 to R80, R82 to R81, R83 to R82, R84 to R83, R87 to R84, R88 to R85, R89 to R86, R90 to R87, R91 to R88, R92 to R89, R93 to R90, R94 to R91, R95 to R92, R96 to R93, R97 to R94, R98 to R95, R99 to R96, R100 to R97, R101 to R98, R102 to R99
Connections:
- wire segments 693 -> 681

Commit message: Readout Schematic in Completion
Parts:
- removed C70, C76: 0.1uF, symbol Device:C_Small
- removed U19: SN74AXC2T45DCTR, symbol readout:SN74AXC2T45DCTR
- added R? (x2): 100, Resistor_SMD:R_0603_1608Metric_Pad1.05x0.95mm_HandSolder, symbol Device:R_Small
Connections:
- net labels removed: CITIROC_IN_ONE3, CITIROC_IN_ONE4
- wire segments 681 -> 661

Commit message: _
Parts:
- added C74: 0.1uF, Capacitor_SMD:C_0603_1608Metric_Pad1.05x0.95mm_HandSolder, symbol Device:C_Small
- C19, C20, C21, C22, C23, C24, C25, C26, C27, C28, C29, C30, C31, C32, C68, C69, C77: footprint (none) -> Capacitor_SMD:C_0603_1608Metric_Pad1.05x0.95mm_HandSolder
- C70: renamed from C71; footprint (none) -> Capacitor_SMD:C_0603_1608Metric_Pad1.05x0.95mm_HandSolder
- C79: renamed from C80; footprint (none) -> Capacitor_SMD:C_0603_1608Metric_Pad1.05x0.95mm_HandSolder
- C80: renamed from C81; footprint (none) -> Capacitor_SMD:C_0603_1608Metric_Pad1.05x0.95mm_HandSolder
- C83: renamed from C84; footprint (none) -> Capacitor_SMD:C_0603_1608Metric_Pad1.05x0.95mm_HandSolder
- C84: renamed from C85; footprint (none) -> Capacitor_SMD:C_0603_1608Metric_Pad1.05x0.95mm_HandSolder
- C87: renamed from C88; footprint (none) -> Capacitor_SMD:C_0603_1608Metric_Pad1.05x0.95mm_HandSolder
- C88: renamed from C89; footprint (none) -> Capacitor_SMD:C_0603_1608Metric_Pad1.05x0.95mm_HandSolder
- C89: renamed from C90; footprint (none) -> Capacitor_SMD:C_0603_1608Metric_Pad1.05x0.95mm_HandSolder
- R100: renamed from R98; footprint (none) -> Resistor_SMD:R_0603_1608Metric_Pad1.05x0.95mm_HandSolder
- R101: renamed from R99; footprint (none) -> Resistor_SMD:R_0603_1608Metric_Pad1.05x0.95mm_HandSolder
- U20: renamed from U22; Item Cost (none) -> $1.52; MFN (none) -> NLSV8T244DTR2G; Supplier (none) -> ON Semiconductor; Supplier P/N (none) -> NLSV8T244DTR2GOSCT-ND
- gave numbers to parts that had none: 2
- renumbered C110 to C109, C111 to C110, C112 to C111, C113 to C112, C114 to C113, C115 to C114, C116 to C115, C117 to C116, C118 to C117, C119 to C118, C120 to C119, C121 to C120, C122 to C121, C123 to C122, C124 to C123, C125 to C124, C126 to C125, C127 to C126, C128 to C127, C129 to C128, C130 to C129, C131 to C130, C132 to C131, C133 to C132, C134 to C133, C135 to C134, C136 to C135, C137 to C136, C138 to C137, C139 to C138, C140 to C139, C141 to C140, C142 to C141, C143 to C142, C144 to C143, C149 to C147, C150 to C148, C151 to C149, C152 to C151, C155 to C152, C156 to C154, C159 to C157, C160 to C158, C163 to C161, C164 to C162, C91 to C90, C92 to C91, C93 to C92, R100 to R104, R101 to R105, R102 to R106, R103 to R107, R59 to R61, R60 to R62, R61 to R63, R62 to R64, R63 to R65, R64 to R66, R65 to R67, R66 to R68, R67 to R69, R68 to R70, R69 to R71, R70 to R72, R71 to R73, R72 to R74, R73 to R75, R74 to R76, R75 to R77, R76 to R78, R77 to R79, R78 to R80, R79 to R81, R80 to R82, R81 to R83, R82 to R84, R83 to R85, R84 to R86, R85 to R87, R86 to R88, R87 to R89, R88 to R90, R89 to R91, R90 to R92, R91 to R93, R92 to R94, R93 to R95, R94 to R96, R95 to R97, R96 to R98, R97 to R99, U18 to U17, U20 to U18, U21 to U19, U23 to U21, U24 to U22, U25 to U23, U26 to U24
Connections:
- net labels added: Fast_Trig0, Fast_Trig1, Fast_Trig2, Fast_Trig3, Fast_Trig[0..3], SH_Ctrl0, SH_Ctrl1, SH_Ctrl2, SH_Ctrl3, SH_Ctrl4, SH_Ctrl5, SH_Ctrl6, SH_Ctrl7, SH_Ctrl8, SH_Ctrl9, SH_Ctrl[0..24], Serial_ctrl0, Serial_ctrl1, Serial_ctrl2, Serial_ctrl3, Serial_ctrl4, Serial_ctrl5, Serial_ctrl6, Serial_ctrl7, Serial_ctrl8, Serial_ctrl[0..8], TRIG_OUT0, TRIG_OUT1, TRIG_OUT10, TRIG_OUT11, TRIG_OUT12, TRIG_OUT13, TRIG_OUT14, TRIG_OUT15, TRIG_OUT16, TRIG_OUT17, TRIG_OUT18, TRIG_OUT19, TRIG_OUT2, TRIG_OUT20, TRIG_OUT21, TRIG_OUT22, TRIG_OUT23, TRIG_OUT24, TRIG_OUT25, TRIG_OUT26, TRIG_OUT27, TRIG_OUT28, TRIG_OUT29, TRIG_OUT3, TRIG_OUT30, TRIG_OUT31, TRIG_OUT4, TRIG_OUT5, TRIG_OUT6, TRIG_OUT7, TRIG_OUT8, TRIG_OUT9, TRIG_OUT[0..31]
- net labels removed: CITIROC_IN_ONE0, CITIROC_IN_ONE1, CITIROC_IN_ONE10, CITIROC_IN_ONE11, CITIROC_IN_ONE12, CITIROC_IN_ONE13, CITIROC_IN_ONE14, CITIROC_IN_ONE15, CITIROC_IN_ONE16, CITIROC_IN_ONE17, CITIROC_IN_ONE18, CITIROC_IN_ONE19, CITIROC_IN_ONE2, CITIROC_IN_ONE20, CITIROC_IN_ONE21, CITIROC_IN_ONE22, CITIROC_IN_ONE23, CITIROC_IN_ONE24, CITIROC_IN_ONE5, CITIROC_IN_ONE6, CITIROC_IN_ONE7, CITIROC_IN_ONE8, CITIROC_IN_ONE9, CITIROC_IN_ONE[0..24], T1_0, T1_1, T1_10, T1_11, T1_12, T1_13, T1_14, T1_15, T1_16, T1_17, T1_18, T1_19, T1_2, T1_20, T1_21, T1_22, T1_23, T1_24, T1_25, T1_26, T1_27, T1_28, T1_29, T1_3, T1_30, T1_31, T1_4, T1_5, T1_6, T1_7, T1_8, T1_9, T1_[0..31]
- wire segments 661 -> 642

Commit message: Readout Preliminary Schematic Made
Parts:
- U14: renamed from U22; Manufacturer (none) -> Texas Instruments
- U17, U9: Manufacturer (none) -> Weeroc
- U18: footprint (none) -> Package_SO:SSOP-8_2.95x2.8mm_P0.65mm; Item Cost (none) -> $0.66; MFN (none) -> SN74AXC2T45DCTR; Manufacturer (none) -> Texas Instruments; Supplier (none) -> Digi-Key; Supplier P/N (none) -> 296-SN74AXC2T45DCCT-ND
- U19: footprint (none) -> Package_SO:TSSOP-20_4.4x6.5mm_P0.65mm; Item Cost (none) -> $1.52; MFN (none) -> NLSV8T244DTR2G; Manufacturer (none) -> ON Semiconductors; Supplier (none) -> Digi-Key; Supplier P/N (none) -> NLSV8T244DTR2GOSCT-ND
- U20: footprint (none) -> Package_SO:TSSOP-20_4.4x6.5mm_P0.65mm; Manufacturer (none) -> ON Semiconductors; Supplier ON Semiconductor -> Digi-Key
- U21: footprint (none) -> Package_SO:SOIC-8_3.9x4.9mm_P1.27mm; Item Cost (none) -> $1.92; MFN (none) -> DS90LV027ATM/NOPB; Manufacturer (none) -> Texas Instruments; Supplier (none) -> Digi-Key; Supplier  (none) -> Digi-Key; Supplier P/N (none) -> DS90LV027ATM/NOPB-ND
- U23: Item Cost 11.75 -> $11.75; Manufacturer (none) -> Texas Instruments
- U24: footprint (none) -> Package_SO:TSSOP-14_4.4x5mm_P0.65mm; Item Cost (none) -> $1.97; MFN (none) -> NLSV4T244EDTR2G; Manufacturer (none) -> ON Semiconductors; Supplier (none) -> Digi-Key; Supplier P/N (none) -> NLSV4T244EDTR2GOSCT-ND
Changed lines of the file:
@@
 F 5 "296-27641-1-ND" H 13750 9000 50  0001 C CNN "Supplier P/N"
 F 6 "REF5025MDTEP" H 13750 9000 50  0001 C CNN "MFN"
-F 7 "11.75" H 13750 9000 50  0001 C CNN "Item Cost"
+F 7 "$11.75" H 13750 9000 50  0001 C CNN "Item Cost"
+F 8 "Texas Instruments" H 13750 9000 50  0001 C CNN "Manufacturer"
 	1    13750 9000
 	-1   0    0    -1
@@
 	6400 7250 8950 7250
 $Comp
-L readout:ADS7955 U22
+L readout:ADS7955 U14
 U 1 1 61BCD360
 P 12350 7150
-AR Path="/60BB4A14/61BCD360" Ref="U22"  Part="1"
+AR Path="/60BB4A14/61BCD360" Ref="U14"  Part="1"
 AR Path="/60BB4C00/61BCD360" Ref="U14"  Part="1"
 F 0 "U14" H 12600 7300 50  0000 C CNN
@@
 F 6 "ADS7955SDBT" H 12350 7150 50  0001 C CNN "MFN"
 F 7 "6.74" H 12350 7150 50  0001 C CNN "Item Cost"
+F 8 "Texas Instruments" H 12350 7150 50  0001 C CNN "Manufacturer"
 	1    12350 7150
 	1    0    0    -1
@@
 F 2 "Package_QFP:LQFP-160_24x24mm_P0.5mm" H 9000 7300 50  0001 C CNN
 F 3 "http://gauss.bu.edu/svn/emphatic-doco/Docs/CITIROC1A%20-%20Datasheet%20V2.5.pdf" H 9000 7300 50  0001 C CNN
+F 4 "Weeroc" H 9600 7150 50  0001 C CNN "Manufacturer"
 	3    9600 7150
 	1    0    0    -1
@@
 F 2 "Package_QFP:LQFP-160_24x24mm_P0.5mm" H 13000 1600 50  0001 C CNN
 F 3 "http://gauss.bu.edu/svn/emphatic-doco/Docs/CITIROC1A%20-%20Datasheet%20V2.5.pdf" H 13000 1600 50  0001 C CNN
+F 4 "Weeroc" H 13600 1450 50  0001 C CNN "Manufacturer"
 	2    13600 1450
 	1    0    0    -1
@@
 F 6 "" V 4700 3400 50  0001 C CNN "Supplier"
 F 7 "" V 4700 3400 50  0001 C CNN "Supplier P/N"
+F 8 "Weeroc" H 4700 3400 50  0001 C CNN "Manufacturer"
 	1    4700 3400
 	0    1    1    0
@@
 F 0 "U16" H 15550 4625 50  0000 C CNN
 F 1 "NLSV4T244E" H 15550 4534 50  0000 C CNN
-F 2 "" H 15550 4150 50  0001 C CNN
+F 2 "Package_SO:TSSOP-14_4.4x5mm_P0.65mm" H 15550 4150 50  0001 C CNN
 F 3 "https://www.onsemi.com/pdf/datasheet/nlsv4t244e-d.pdf" H 15550 4150 50  0001 C CNN
+F 4 "$1.97" H 15550 4150 50  0001 C CNN "Item Cost"
+F 5 "ON Semiconductors" H 15550 4150 50  0001 C CNN "Manufacturer"
+F 6 "NLSV4T244EDTR2G" H 15550 4150 50  0001 C CNN "MFN"
+F 7 "Digi-Key" H 15550 4150 50  0001 C CNN "Supplier"
+F 8 "NLSV4T244EDTR2GOSCT-ND" H 15550 4150 50  0001 C CNN "Supplier P/N"
 	1    15550 4150
 	-1   0    0    -1
@@
 F 0 "U10" H 10500 2675 50  0000 C CNN
 F 1 "SN74AXC2T45DCTR" H 10500 2584 50  0000 C CNN
-F 2 "" H 10500 2300 50  0001 C CNN
+F 2 "Package_SO:SSOP-8_2.95x2.8mm_P0.65mm" H 10500 2300 50  0001 C CNN
 F 3 "https://www.ti.com/lit/ds/symlink/sn74axc2t45.pdf?ts=1624298260694&ref_url=https%253A%252F%252Fwww.ti.com%252Fstore%252Fti%252Fen%252Fp%252Fproduct%252F%253Fp%253DSN74AXC2T45DCTR" H 10500 2300 50  0001 C CNN
+F 4 "$0.66" H 10500 2300 50  0001 C CNN "Item Cost"
+F 5 "Texas Instruments" H 10500 2300 50  0001 C CNN "Manufacturer"
+F 6 "SN74AXC2T45DCTR" H 10500 2300 50  0001 C CNN "MFN"
+F 7 "Digi-Key" H 10500 2300 50  0001 C CNN "Supplier"
+F 8 "296-SN74AXC2T45DCCT-ND" H 10500 2300 50  0001 C CNN "Supplier P/N"
 	1    10500 2300
 	1    0    0    -1
@@
 F 0 "U11" H 10500 3975 50  0000 C CNN
 F 1 "NLSV8T244" H 10500 3884 50  0000 C CNN
-F 2 "" H 10500 3300 50  0001 C CNN
+F 2 "Package_SO:TSSOP-20_4.4x6.5mm_P0.65mm" H 10500 3300 50  0001 C CNN
 F 3 "https://www.onsemi.com/pdf/datasheet/nlsv8t244-d.pdf" H 10500 3300 50  0001 C CNN
+F 4 "$1.52" H 10500 3300 50  0001 C CNN "Item Cost"
+F 5 "NLSV8T244DTR2G" H 10500 3300 50  0001 C CNN "MFN"
+F 6 "ON Semiconductors" H 10500 3300 50  0001 C CNN "Manufacturer"
+F 7 "Digi-Key" H 10500 3300 50  0001 C CNN "Supplier"
+F 8 "NLSV8T244DTR2GOSCT-ND" H 10500 3300 50  0001 C CNN "Supplier P/N"
 	1    10500 3300
 	1    0    0    -1
@@
 F 0 "U12" H 10500 5475 50  0000 C CNN
 F 1 "NLSV8T244" H 10500 5384 50  0000 C CNN
-F 2 "" H 10500 4800 50  0001 C CNN
+F 2 "Package_SO:TSSOP-20_4.4x6.5mm_P0.65mm" H 10500 4800 50  0001 C CNN
 F 3 "https://www.onsemi.com/pdf/datasheet/nlsv8t244-d.pdf" H 10500 4800 50  0001 C CNN
 F 4 "$1.52" H 10500 4800 50  0001 C CNN "Item Cost"
 F 5 "NLSV8T244DTR2G" H 10500 4800 50  0001 C CNN "MFN"
-F 6 "ON Semiconductor" H 10500 4800 50  0001 C CNN "Supplier"
+F 6 "Digi-Key" H 10500 4800 50  0001 C CNN "Supplier"
 F 7 "NLSV8T244DTR2GOSCT-ND" H 10500 4800 50  0001 C CNN "Supplier P/N"
+F 8 "ON Semiconductors" H 10500 4800 50  0001 C CNN "Manufacturer"
 	1    10500 4800
 	1    0    0    -1
@@
 F 0 "U13" H 11550 2675 50  0000 C CNN
 F 1 "DS90LV027A" H 11550 2584 50  0000 C CNN
-F 2 "" H 11550 2300 50  0001 C CNN
+F 2 "Package_SO:SOIC-8_3.9x4.9mm_P1.27mm" H 11550 2300 50  0001 C CNN
 F 3 "https://www.ti.com/lit/ds/symlink/ds90lv027a.pdf?ts=1624298607733&ref_url=https%253A%252F%252Fwww.ti.com%252Fstore%252Fti%252Fen%252Fp%252Fproduct%252F%253Fp%253DDS90LV027ATM%252FNOPB%2526utm_source%253Dgoogle%2526utm_medium%253Dcpc%2526utm_campaign%253Dasc-null-null-OPN_EN-cpc-store-google-wwe%2526utm_content%253DDevice%2526ds_k%253DDS90LV027ATM%252FNOPB%2526DCM%253Dyes%2526gclid%253DEAIaIQobChMI8Je45qep8QIVV-HICh3kjQY7EAAYASAAEgIUZvD_BwE%2526gclsrc%253Daw.ds" H 11550 2300 50  0001 C CNN
+F 4 "$1.92" H 11550 2300 50  0001 C CNN "Item Cost"
+F 5 "Texas Instruments" H 11550 2300 50  0001 C CNN "Manufacturer"
+F 6 "DS90LV027ATM/NOPB" H 11550 2300 50  0001 C CNN "MFN"
+F 7 "Digi-Key" H 11550 2300 50  0001 C CNN "Supplier "
+F 8 "DS90LV027ATM/NOPB-ND" H 11550 2300 50  0001 C CNN "Supplier P/N"
+F 9 "Digi-Key" H 11550 2300 50  0001 C CNN "Supplier"
 	1    11550 2300
 	1    0    0    -1

Commit message: Footprints Assigned
Parts:
- removed J13: conn, symbol Connector_Generic:Conn_02x11_Counter_Clockwise
- removed J14: GPIO Header, symbol Connector_Generic:Conn_02x04_Odd_Even
- added TP? (x11): TestPoint_2Pole, TestPoint:TestPoint_2Pads_Pitch2.54mm_Drill0.8mm, symbol Connector:TestPoint_2Pole
- J20: renamed from J12; footprint (none) -> Readout_Board_Parts:lemo-EPB.00.250.NTN
- RV2: footprint (none) -> Potentiometer_THT:Potentiometer_ACP_CA6-H2,5_Horizontal; Item Cost (none) -> $2.41; MFN (none) -> 3296Z-1-103LF; Manufacturer (none) -> Bourns Inc.; Supplier  (none) -> Digi-Key; Supplier P/N (none) -> 3296Z-103LF-ND
- TP2: footprint (none) -> Connector_PinHeader_2.54mm:PinHeader_1x23_P2.54mm_Vertical_SMD_Pin1Left
- renumbered C109 to C115, C110 to C116, C111 to C117, C112 to C118, C113 to C119, C114 to C120, C115 to C121, C116 to C122, C117 to C123, C118 to C124, C119 to C125, C120 to C126, C121 to C127, C122 to C128, C123 to C129, C124 to C130, C125 to C131, C126 to C132, C127 to C133, C128 to C134, C129 to C135, C130 to C136, C131 to C137, C132 to C138, C133 to C139, C134 to C140, C135 to C141, C136 to C142, C137 to C143, C138 to C144, C139 to C145, C140 to C146, C141 to C147, C142 to C148, C143 to C149, C147 to C153, C148 to C154, C149 to C155, C151 to C157, C152 to C158, C154 to C160, C157 to C163, C158 to C164, C161 to C167, C162 to C168, C90 to C96, C91 to C97, C92 to C98, R94 to R100, R95 to R101, R96 to R102, R97 to R103, R98 to R104, R99 to R105, R100 to R106, R101 to R107, R102 to R108, R103 to R109, R104 to R110, R105 to R111, R106 to R112, R107 to R113, R61 to R67, R62 to R68, R63 to R69, R64 to R70, R65 to R71, R66 to R72, R67 to R73, R68 to R74, R69 to R75, R70 to R76, R71 to R77, R72 to R78, R73 to R79, R74 to R80, R75 to R81, R76 to R82, R77 to R83, R78 to R84, R79 to R85, R80 to R86, R81 to R87, R82 to R88, R83 to R89, R84 to R90, R85 to R91, R86 to R92, R87 to R93, R88 to R94, R89 to R95, R90 to R96, R91 to R97, R92 to R98, R93 to R99, U17 to U15, U18 to U16, U19 to U17, U20 to U18, U21 to U19, U14 to U20, U23 to U21, U24 to U22, U9 to U7
Connections:
- wire segments 642 -> 630
- no-connect marks 9 -> 13

Commit message: Layout Started
Parts:
- gave numbers to parts that had none: 11
- renumbered J20 to J15, TP2 to TP24

Commit message: Starting Layout
Parts:
- C115, C116, C117, C118, C119, C120, C121, C122, C123, C124, C125, C126, C127, C128, C129, C130, C131, C132, C133, C134, C135, C136, C137, C138, C139, C140, C141, C142, C143, C144, C145, C146, C147, C148, C149, C153, C154, C17, C18: value 100n -> 0.1uF; Item Cost (none) -> $0.1; MFN (none) -> 885012206046; Manufacturer (none) -> Würth Elektronik; Supplier  (none) -> Digi-Key; Supplier P/N (none) -> 732-7965-1-ND
- C155, C157, C158, C160, C163, C164: value 150p -> 150pF; Item Cost (none) -> $0.1; MFN (none) -> 885012206103; Manufacturer (none) -> Würth Elektronik; Supplier  (none) -> Digi-Key; Supplier P/N (none) -> 732-12236-1-ND
- C167, C168: value 10u -> 10uF; footprint Capacitor_SMD:C_0603_1608Metric_Pad1.05x0.95mm_HandSolder -> Capacitor_SMD:C_0805_2012Metric_Pad1.15x1.40mm_HandSolder; Item Cost (none) -> $0.18; MFN (none) -> 885012107010; Manufacturer (none) -> Würth Elektronik; Supplier  (none) -> Digi-Key; Supplier P/N (none) -> 732-7620-1-ND
- C19, C20, C21, C22, C23, C24, C25, C26, C27, C28, C29, C30, C31, C32, C68, C69, C70, C74, C77, C79, C80, C83, C84, C87, C88, C89: Item Cost (none) -> $0.1; MFN (none) -> 885012206046; Manufacturer (none) -> Würth Elektronik; Supplier  (none) -> Digi-Key; Supplier P/N (none) -> 732-7965-1-ND
- C96, C97, C98: value 1u -> 1uF; Item Cost (none) -> $0.15; MFN (none) -> 885012106010; Manufacturer (none) -> Würth Elektronik; Supplier  (none) -> Digi-Key; Supplier P/N (none) -> 732-7907-1-ND
- TP24: footprint Connector_PinHeader_2.54mm:PinHeader_1x23_P2.54mm_Vertical_SMD_Pin1Left -> Connector_PinHeader_2.54mm:PinHeader_1x02_P2.54mm_Vertical_SMD_Pin1Left
- U17, U18: footprint Package_SO:TSSOP-20_4.4x6.5mm_P0.65mm -> Package_SO:SOIC-20W_7.5x12.8mm_P1.27mm
- U22: footprint Package_SO:TSSOP-14_4.4x5mm_P0.65mm -> Package_SO:SOIC-14_3.9x8.7mm_P1.27mm
Other:
- note removed: "may not need gnd for all\nif space issue"

Commit message: -
Parts:
- J15: footprint Readout_Board_Parts:lemo-EPB.00.250.NTN -> readout_trenz:lemo-EPB.00.250.NTN
- R100: renamed from R97; value 50 -> 56; Item Cost (none) -> $0.1; MFN (none) -> CRCW060356R0FKEAC; Manufacturer (none) -> Vishay Dale; Supplier  (none) -> Digi-Key; Supplier P/N (none) -> 541-5483-1-ND
- R101: renamed from R98; value 50 -> 56; Item Cost (none) -> $0.1; MFN (none) -> CRCW060356R0FKEAC; Manufacturer (none) -> Vishay Dale; Supplier  (none) -> Digi-Key; Supplier P/N (none) -> 541-5483-1-ND
- R102: renamed from R99; Item Cost (none) -> $0.1; MFN (none) -> RC0603FR-070RL; Manufacturer (none) -> Yageo; Supplier  (none) -> Digi-Key; Supplier P/N (none) -> 311-0.0HRCT-ND
- R103: renamed from R100; Item Cost (none) -> $0.1; MFN (none) -> RC0603FR-070RL; Manufacturer (none) -> Yageo; Supplier  (none) -> Digi-Key; Supplier P/N (none) -> 311-0.0HRCT-ND
- R104: renamed from R101; Item Cost (none) -> $0.1; MFN (none) -> RC0603FR-070RL; Manufacturer (none) -> Yageo; Supplier  (none) -> Digi-Key; Supplier P/N (none) -> 311-0.0HRCT-ND
- R105: renamed from R102; Item Cost (none) -> $0.1; MFN (none) -> RC0603FR-070RL; Manufacturer (none) -> Yageo; Supplier  (none) -> Digi-Key; Supplier P/N (none) -> 311-0.0HRCT-ND
- R106: renamed from R103; Item Cost (none) -> $0.1; MFN (none) -> RC0603FR-070RL; Manufacturer (none) -> Yageo; Supplier  (none) -> Digi-Key; Supplier P/N (none) -> 311-0.0HRCT-ND
- R107: renamed from R104; Item Cost (none) -> $0.1; MFN (none) -> RC0603FR-070RL; Manufacturer (none) -> Yageo; Supplier  (none) -> Digi-Key; Supplier P/N (none) -> 311-0.0HRCT-ND
- R108: renamed from R105; Item Cost (none) -> $0.1; MFN (none) -> RC0603FR-070RL; Manufacturer (none) -> Yageo; Supplier  (none) -> Digi-Key; Supplier P/N (none) -> 311-0.0HRCT-ND
- R109: renamed from R106; value R_Small -> 10k; footprint Resistor_SMD:R_0603_1608Metric_Pad1.05x0.95mm_HandSolder -> Resistor_SMD:R_1206_3216Metric_Pad1.42x1.75mm_HandSolder; Item Cost (none) -> $0.1; MFN (none) -> CRCW120610K0FKEAC; Manufacturer (none) -> Vishay Dale; Supplier  (none) -> Digi-Key; Supplier P/N (none) -> 541-3983-1-ND
- R110: renamed from R107; value R_Small -> 10k; footprint Resistor_SMD:R_0603_1608Metric_Pad1.05x0.95mm_HandSolder -> Resistor_SMD:R_1206_3216Metric_Pad1.42x1.75mm_HandSolder; Item Cost (none) -> $0.1; MFN (none) -> CRCW120610K0FKEAC; Manufacturer (none) -> Vishay Dale; Supplier  (none) -> Digi-Key; Supplier P/N (none) -> 541-3983-1-ND
- R111: renamed from R108; Item Cost (none) -> $0.01; MFN (none) -> CR0603AFX-1000ELF; Manufacturer (none) -> Bourns Inc.; Supplier  (none) -> Digi-Key; Supplier P/N (none) -> 118-CR0603AFX-1000ELFCT-ND
- R112: renamed from R109; Item Cost (none) -> $0.01; MFN (none) -> CR0603AFX-1000ELF; Manufacturer (none) -> Bourns Inc.; Supplier  (none) -> Digi-Key; Supplier P/N (none) -> 118-CR0603AFX-1000ELFCT-ND
- R113: renamed from R110; footprint Resistor_SMD:R_0603_1608Metric_Pad1.05x0.95mm_HandSolder -> Resistor_SMD:R_0805_2012Metric_Pad1.15x1.40mm_HandSolder; Item Cost (none) -> $0.1; MFN (none) -> RC0805FR-071KL; Manufacturer (none) -> Yageo; Supplier  (none) -> Digi-Key; Supplier P/N (none) -> 311-1.00KCRCT-ND
- R114: renamed from R111; footprint Resistor_SMD:R_0603_1608Metric_Pad1.05x0.95mm_HandSolder -> Resistor_SMD:R_1206_3216Metric_Pad1.42x1.75mm_HandSolder; Item Cost (none) -> $0.1; MFN (none) -> RC1206FR-07470KL; Manufacturer (none) -> Yageo; Supplier  (none) -> Digi-Key; Supplier P/N (none) -> 311-470KFRCT-ND
- R115: renamed from R112; footprint Resistor_SMD:R_0603_1608Metric_Pad1.05x0.95mm_HandSolder -> Resistor_SMD:R_0805_2012Metric_Pad1.15x1.40mm_HandSolder; Item Cost (none) -> $0.1; MFN (none) -> RC0805FR-071KL; Manufacturer (none) -> Yageo; Supplier  (none) -> Digi-Key; Supplier P/N (none) -> 311-1.00KCRCT-ND
- R116: renamed from R113; footprint Resistor_SMD:R_0603_1608Metric_Pad1.05x0.95mm_HandSolder -> Resistor_SMD:R_0805_2012Metric_Pad1.15x1.40mm_HandSolder; Item Cost (none) -> $0.1; MFN (none) -> RC0805FR-071KL; Manufacturer (none) -> Yageo; Supplier  (none) -> Digi-Key; Supplier P/N (none) -> 311-1.00KCRCT-ND
- R70: renamed from R67; value 50 -> 56; Item Cost (none) -> $0.1; MFN (none) -> CRCW060356R0FKEAC; Manufacturer (none) -> Vishay Dale; Supplier  (none) -> Digi-Key; Supplier P/N (none) -> 541-5483-1-ND
- R71: renamed from R68; value 50 -> 56; Item Cost (none) -> $0.1; MFN (none) -> CRCW060356R0FKEAC; Manufacturer (none) -> Vishay Dale; Supplier  (none) -> Digi-Key; Supplier P/N (none) -> 541-5483-1-ND
- R72: renamed from R69; value 50 -> 56; Item Cost (none) -> $0.1; MFN (none) -> CRCW060356R0FKEAC; Manufacturer (none) -> Vishay Dale; Supplier  (none) -> Digi-Key; Supplier P/N (none) -> 541-5483-1-ND
- R73: renamed from R70; value 50 -> 56; Item Cost (none) -> $0.1; MFN (none) -> CRCW060356R0FKEAC; Manufacturer (none) -> Vishay Dale; Supplier  (none) -> Digi-Key; Supplier P/N (none) -> 541-5483-1-ND
- R74: renamed from R71; value 50 -> 56; Item Cost (none) -> $0.1; MFN (none) -> CRCW060356R0FKEAC; Manufacturer (none) -> Vishay Dale; Supplier  (none) -> Digi-Key; Supplier P/N (none) -> 541-5483-1-ND
- R75: renamed from R72; value 50 -> 56; Item Cost (none) -> $0.1; MFN (none) -> CRCW060356R0FKEAC; Manufacturer (none) -> Vishay Dale; Supplier  (none) -> Digi-Key; Supplier P/N (none) -> 541-5483-1-ND
- R76: renamed from R73; value 50 -> 56; Item Cost (none) -> $0.1; MFN (none) -> CRCW060356R0FKEAC; Manufacturer (none) -> Vishay Dale; Supplier  (none) -> Digi-Key; Supplier P/N (none) -> 541-5483-1-ND
- R77: renamed from R74; value 50 -> 56; Item Cost (none) -> $0.1; MFN (none) -> CRCW060356R0FKEAC; Manufacturer (none) -> Vishay Dale; Supplier  (none) -> Digi-Key; Supplier P/N (none) -> 541-5483-1-ND
- R78: renamed from R75; value 50 -> 56; Item Cost (none) -> $0.1; MFN (none) -> CRCW060356R0FKEAC; Manufacturer (none) -> Vishay Dale; Supplier  (none) -> Digi-Key; Supplier P/N (none) -> 541-5483-1-ND
- R79: renamed from R76; value 50 -> 56; Item Cost (none) -> $0.1; MFN (none) -> CRCW060356R0FKEAC; Manufacturer (none) -> Vishay Dale; Supplier  (none) -> Digi-Key; Supplier P/N (none) -> 541-5483-1-ND
- R80: renamed from R77; value 50 -> 56; Item Cost (none) -> $0.1; MFN (none) -> CRCW060356R0FKEAC; Manufacturer (none) -> Vishay Dale; Supplier  (none) -> Digi-Key; Supplier P/N (none) -> 541-5483-1-ND
- R81: renamed from R78; value 50 -> 56; Item Cost (none) -> $0.1; MFN (none) -> CRCW060356R0FKEAC; Manufacturer (none) -> Vishay Dale; Supplier  (none) -> Digi-Key; Supplier P/N (none) -> 541-5483-1-ND
- R82: renamed from R79; value 50 -> 56; Item Cost (none) -> $0.1; MFN (none) -> CRCW060356R0FKEAC; Manufacturer (none) -> Vishay Dale; Supplier  (none) -> Digi-Key; Supplier P/N (none) -> 541-5483-1-ND
- R83: renamed from R80; value 50 -> 56; Item Cost (none) -> $0.1; MFN (none) -> CRCW060356R0FKEAC; Manufacturer (none) -> Vishay Dale; Supplier  (none) -> Digi-Key; Supplier P/N (none) -> 541-5483-1-ND
- R84: renamed from R81; value 50 -> 56; Item Cost (none) -> $0.1; MFN (none) -> CRCW060356R0FKEAC; Manufacturer (none) -> Vishay Dale; Supplier  (none) -> Digi-Key; Supplier P/N (none) -> 541-5483-1-ND
- R85: renamed from R82; value 50 -> 56; Item Cost (none) -> $0.1; MFN (none) -> CRCW060356R0FKEAC; Manufacturer (none) -> Vishay Dale; Supplier  (none) -> Digi-Key; Supplier P/N (none) -> 541-5483-1-ND
- R86: renamed from R83; value 50 -> 56; Item Cost (none) -> $0.1; MFN (none) -> CRCW060356R0FKEAC; Manufacturer (none) -> Vishay Dale; Supplier  (none) -> Digi-Key; Supplier P/N (none) -> 541-5483-1-ND
- R87: renamed from R84; value 50 -> 56; Item Cost (none) -> $0.1; MFN (none) -> CRCW060356R0FKEAC; Manufacturer (none) -> Vishay Dale; Supplier  (none) -> Digi-Key; Supplier P/N (none) -> 541-5483-1-ND
- R88: renamed from R85; value 50 -> 56; Item Cost (none) -> $0.1; MFN (none) -> CRCW060356R0FKEAC; Manufacturer (none) -> Vishay Dale; Supplier  (none) -> Digi-Key; Supplier P/N (none) -> 541-5483-1-ND
- R89: renamed from R86; value 50 -> 56; Item Cost (none) -> $0.1; MFN (none) -> CRCW060356R0FKEAC; Manufacturer (none) -> Vishay Dale; Supplier  (none) -> Digi-Key; Supplier P/N (none) -> 541-5483-1-ND
- R90: renamed from R87; value 50 -> 56; Item Cost (none) -> $0.1; MFN (none) -> CRCW060356R0FKEAC; Manufacturer (none) -> Vishay Dale; Supplier  (none) -> Digi-Key; Supplier P/N (none) -> 541-5483-1-ND
- R91: renamed from R88; value 50 -> 56; Item Cost (none) -> $0.1; MFN (none) -> CRCW060356R0FKEAC; Manufacturer (none) -> Vishay Dale; Supplier  (none) -> Digi-Key; Supplier P/N (none) -> 541-5483-1-ND
- R92: renamed from R89; value 50 -> 56; Item Cost (none) -> $0.1; MFN (none) -> CRCW060356R0FKEAC; Manufacturer (none) -> Vishay Dale; Supplier  (none) -> Digi-Key; Supplier P/N (none) -> 541-5483-1-ND
- R93: renamed from R90; value 50 -> 56; Item Cost (none) -> $0.1; MFN (none) -> CRCW060356R0FKEAC; Manufacturer (none) -> Vishay Dale; Supplier  (none) -> Digi-Key; Supplier P/N (none) -> 541-5483-1-ND
- R94: renamed from R91; value 50 -> 56; Item Cost (none) -> $0.1; MFN (none) -> CRCW060356R0FKEAC; Manufacturer (none) -> Vishay Dale; Supplier  (none) -> Digi-Key; Supplier P/N (none) -> 541-5483-1-ND
- R95: renamed from R92; value 50 -> 56; Item Cost (none) -> $0.1; MFN (none) -> CRCW060356R0FKEAC; Manufacturer (none) -> Vishay Dale; Supplier  (none) -> Digi-Key; Supplier P/N (none) -> 541-5483-1-ND
- R96: renamed from R93; value 50 -> 56; Item Cost (none) -> $0.1; MFN (none) -> CRCW060356R0FKEAC; Manufacturer (none) -> Vishay Dale; Supplier  (none) -> Digi-Key; Supplier P/N (none) -> 541-5483-1-ND
- R97: renamed from R94; value 50 -> 56; Item Cost (none) -> $0.1; MFN (none) -> CRCW060356R0FKEAC; Manufacturer (none) -> Vishay Dale; Supplier  (none) -> Digi-Key; Supplier P/N (none) -> 541-5483-1-ND
- R98: renamed from R95; value 50 -> 56; Item Cost (none) -> $0.1; MFN (none) -> CRCW060356R0FKEAC; Manufacturer (none) -> Vishay Dale; Supplier  (none) -> Digi-Key; Supplier P/N (none) -> 541-5483-1-ND
- R99: renamed from R96; value 50 -> 56; Item Cost (none) -> $0.1; MFN (none) -> CRCW060356R0FKEAC; Manufacturer (none) -> Vishay Dale; Supplier  (none) -> Digi-Key; Supplier P/N (none) -> 541-5483-1-ND
- renumbered C115 to C116, C116 to C117, C117 to C118, C118 to C119, C119 to C120, C120 to C121, C121 to C122, C122 to C123, C123 to C124, C124 to C125, C125 to C126, C126 to C127, C127 to C128, C128 to C129, C129 to C130, C130 to C131, C131 to C132, C132 to C133, C133 to C134, C134 to C135, C135 to C136, C136 to C137, C137 to C138, C138 to C139, C139 to C140, C140 to C141, C141 to C142, C142 to C143, C143 to C144, C144 to C145, C145 to C146, C146 to C147, C147 to C148, C148 to C149, C149 to C150, C153 to C154, C154 to C155, C155 to C156, C157 to C158, C158 to C159, C160 to C161, C163 to C164, C164 to C165, C167 to C168, C168 to C169, C96 to C97, C97 to C98, C98 to C99
Connections:
- wire segments 630 -> 629
