File: hardware/onboard_amp/amp_norm.sch (KiCad schematic (older format))
At the start: 45 parts, among them J1 Coaxial, J2 Coaxial, J3 Coaxial, J4 Coaxial, J5 Conn_01x04, J6 Mating_Conn, J7 2x32_Odd_Even, J8 Mating_Conn, J9 2x32_Odd_Even, U1 THS4304D, U2 THS4304D, U3 THS4304D, U4 THS4304D

Commit message: test
Parts:
- removed U1, U2, U3, U4: THS4304D, Package_SO:SOIC-8_3.9x4.9mm_P1.27mm, symbol amp_norm-rescue:THS4304D
- added C17, C18, C19, C20, C21, C22, C23, C24: 6.8 uF, Capacitor_SMD:C_1206_3216Metric, symbol Device:CP1
- added U1, U2, U3, U4: THS3201, Package_SO:SO-8_3.9x4.9mm_P1.27mm, symbol amp_norm-rescue:THS3201
- J1, J2, J3, J4: footprint Breakout_Board_Parts:lemo-EPB.00.250.NTN -> mod:lemo-EPB.00.250.NTN
- R1, R2, R3, R4: value 50 -> 51.1
- R10, R11, R12, R9: value 1k -> 464
Connections:
- net -VCC: now also C18.2, C20.2, C22.2, C24.2, U1.4 (-), U2.4 (-), U3.4 (-), U4.4 (-)
- net GND: now also C17.2, C18.1, C19.2, C20.1, C21.2, C22.1, C23.2, C24.1
- net SIG1: now also U1.3 (+)
- net SIG2: now also U2.3 (+)
- net SIG3: now also U3.3 (+)
- net SIG4: now also J8.63 (Pin_63), U4.3 (+); no longer J9.34 (Pin_34), J9.36 (Pin_36), J9.38 (Pin_38), J9.40 (Pin_40), J9.42 (Pin_42), J9.44 (Pin_44), J9.46 (Pin_46), J9.48 (Pin_48), J9.50 (Pin_50), J9.52 (Pin_52), J9.54 (Pin_54), J9.56 (Pin_56), J9.58 (Pin_58), J9.60 (Pin_60), J9.62 (Pin_62), J9.64 (Pin_64)
- net VCC: now also C17.1, C19.1, C21.1, C23.1, U1.7 (+), U2.7 (+), U3.7 (+), U4.7 (+)
- net at R11.1, R15.2: now also U3.6
- net at R11.2, R3.1: now also U3.2 (-)
- net at R1.1, R9.2: now also U1.2 (-)
- net at R13.2, R9.1: now also U1.6
- net at R12.2, R4.1: now also U4.2 (-)
- net at R12.1, R16.2: now also U4.6
- net at R10.2, R2.1: now also U2.2 (-)
- net at R10.1, R14.2: now also U2.6
- net at J9.33 (Pin_33): no longer J8.33 (Pin_33)
- net at J9.35 (Pin_35): no longer J8.35 (Pin_35)
- net at J9.37 (Pin_37): no longer J8.37 (Pin_37)
- net at J9.39 (Pin_39): no longer J8.39 (Pin_39)
- net at J9.41 (Pin_41): no longer J8.41 (Pin_41)
- net at J9.43 (Pin_43): no longer J8.43 (Pin_43)
- net at J9.45 (Pin_45): no longer J8.45 (Pin_45)
- net at J9.47 (Pin_47): no longer J8.47 (Pin_47)
- net at J9.49 (Pin_49): no longer J8.49 (Pin_49)
- net at J9.51 (Pin_51): no longer J8.51 (Pin_51)
- net at J9.53 (Pin_53): no longer J8.53 (Pin_53)
- net at J9.55 (Pin_55): no longer J8.55 (Pin_55)
- net at J9.57 (Pin_57): no longer J8.57 (Pin_57)
- net at J9.59 (Pin_59): no longer J8.59 (Pin_59)
- net at J9.61 (Pin_61): no longer J8.61 (Pin_61)
- net at J9.63 (Pin_63): no longer J8.63 (Pin_63)
- no-connect marks 66 -> 113
Other:
- moved on the sheet: C10, C2, C9, J5, J8, J9

Commit message: Updates
Parts:
- removed J1: Coaxial, mod:lemo-EPB.00.250.NTN, symbol amp_norm-rescue:Conn_Coaxial-Connector-Breakout_Board-rescue
- added J1: Conn_Coaxial, mod:lemo-EPB.00.250.NTN, symbol Connector:Conn_Coaxial
- J2, J3, J4: value Coaxial -> Conn_Coaxial; symbol amp_norm-rescue:Conn_Coaxial-Connector-Breakout_Board-rescue -> Connector:Conn_Coaxial
- U1, U2, U3, U4: symbol amp_norm-rescue:THS3201 -> amplib:THS3201
Connections:
- net GND: now also J1.2 (Ext)
- net at R13.1: now also J1.1 (In)
Changed lines of the file:
@@
 Wire Wire Line
 	2400 1700 2900 1700
-$Comp
-L power:GND #PWR09
-U 1 1 60EAFF26
-P 3550 1900
-F 0 "#PWR09" H 3550 1650 50  0001 C CNN
-F 1 "GND" H 3555 1727 50  0000 C CNN
-F 2 "" H 3550 1900 50  0001 C CNN
-F 3 "" H 3550 1900 50  0001 C CNN
-	1    3550 1900
-	1    0    0    -1
-$EndComp
-$Comp
-L amp_norm-rescue:Conn_Coaxial-Connector-Breakout_Board-rescue J1
-U 1 1 60EAFF2C
-P 3550 1700
-F 0 "J1" H 3650 1675 50  0000 L CNN
-F 1 "Coaxial" H 3650 1584 50  0000 L CNN
-F 2 "mod:lemo-EPB.00.250.NTN" H 3550 1700 50  0001 C CNN
-F 3 "" H 3550 1700 50  0001 C CNN
-	1    3550 1700
-	1    0    0    -1
-$EndComp
 Wire Wire Line
 	3200 1700 3350 1700
@@
 $EndComp
 $Comp
-L amp_norm-rescue:THS3201 U1
+L amplib:THS3201 U1
 U 1 1 60EA1133
 P 2100 1700
@@
 $EndComp
 $Comp
-L amp_norm-rescue:Conn_Coaxial-Connector-Breakout_Board-rescue J2
+L Connector:Conn_Coaxial J2
 U 1 1 60FE5466
 P 3550 3350
 F 0 "J2" H 3650 3325 50  0000 L CNN
-F 1 "Coaxial" H 3650 3234 50  0000 L CNN
+F 1 "Conn_Coaxial" H 3650 3234 50  0000 L CNN
 F 2 "mod:lemo-EPB.00.250.NTN" H 3550 3350 50  0001 C CNN
 F 3 "" H 3550 3350 50  0001 C CNN
@@
 Connection ~ 2900 3350
 $Comp
-L amp_norm-rescue:THS3201 U2
+L amplib:THS3201 U2
 U 1 1 60FE5498
 P 2100 3350
@@
 $EndComp
 $Comp
-L amp_norm-rescue:Conn_Coaxial-Connector-Breakout_Board-rescue J3
+L Connector:Conn_Coaxial J3
 U 1 1 61048AA0
 P 3550 4950
 F 0 "J3" H 3650 4925 50  0000 L CNN
-F 1 "Coaxial" H 3650 4834 50  0000 L CNN
+F 1 "Conn_Coaxial" H 3650 4834 50  0000 L CNN
 F 2 "mod:lemo-EPB.00.250.NTN" H 3550 4950 50  0001 C CNN
 F 3 "" H 3550 4950 50  0001 C CNN
@@
 Connection ~ 2900 4950
 $Comp
-L amp_norm-rescue:THS3201 U3
+L amplib:THS3201 U3
 U 1 1 61048AD2
 P 2100 4950
@@
 $EndComp
 $Comp
-L amp_norm-rescue:Conn_Coaxial-Connector-Breakout_Board-rescue J4
+L Connector:Conn_Coaxial J4
 U 1 1 61048B22
 P 3550 6600
 F 0 "J4" H 3650 6575 50  0000 L CNN
-F 1 "Coaxial" H 3650 6484 50  0000 L CNN
+F 1 "Conn_Coaxial" H 3650 6484 50  0000 L CNN
 F 2 "mod:lemo-EPB.00.250.NTN" H 3550 6600 50  0001 C CNN
 F 3 "" H 3550 6600 50  0001 C CNN
@@
 Connection ~ 2900 6600
 $Comp
-L amp_norm-rescue:THS3201 U4
+L amplib:THS3201 U4
 U 1 1 61048B54
 P 2100 6600
@@
 	1    0    0    -1
 $EndComp
+$Comp
+L Connector:Conn_Coaxial J1
+U 1 1 60EA8C8D
+P 3550 1700
+F 0 "J1" H 3650 1675 50  0000 L CNN
+F 1 "Conn_Coaxial" H 3650 1584 50  0000 L CNN
+F 2 "mod:lemo-EPB.00.250.NTN" H 3550 1700 50  0001 C CNN
+F 3 " ~" H 3550 1700 50  0001 C CNN
+	1    3550 1700
+	1    0    0    -1
+$EndComp
+$Comp
+L power:GND #PWR09
+U 1 1 60ECF4FB
+P 3550 1900
+F 0 "#PWR09" H 3550 1650 50  0001 C CNN
+F 1 "GND" H 3555 1727 50  0000 C CNN
+F 2 "" H 3550 1900 50  0001 C CNN
+F 3 "" H 3550 1900 50  0001 C CNN
+	1    3550 1900
+	1    0    0    -1
+$EndComp

Commit message: Amplifier layout
Parts:
- J5: footprint Connector_PinHeader_2.54mm:PinHeader_1x04_P2.54mm_Vertical_SMD_Pin1Left -> Connector_PinHeader_2.54mm:PinHeader_1x04_P2.54mm_Vertical
Connections:
- net SIG1: now also J7.1 (Pin_1), J7.11 (Pin_11), J7.13 (Pin_13), J7.15 (Pin_15), J7.17 (Pin_17), J7.19 (Pin_19), J7.21 (Pin_21), J7.23 (Pin_23), J7.25 (Pin_25), J7.27 (Pin_27), J7.29 (Pin_29), J7.3 (Pin_3), J7.31 (Pin_31), J7.5 (Pin_5), J7.7 (Pin_7), J7.9 (Pin_9); no longer J7.10 (Pin_10), J7.12 (Pin_12), J7.14 (Pin_14), J7.16 (Pin_16), J7.18 (Pin_18), J7.2 (Pin_2), J7.20 (Pin_20), J7.22 (Pin_22), J7.24 (Pin_24), J7.26 (Pin_26), J7.28 (Pin_28), J7.30 (Pin_30), J7.32 (Pin_32), J7.4 (Pin_4), J7.6 (Pin_6), J7.8 (Pin_8)
- net SIG2: now also J7.33 (Pin_33), J7.35 (Pin_35), J7.37 (Pin_37), J7.39 (Pin_39), J7.41 (Pin_41), J7.43 (Pin_43), J7.45 (Pin_45), J7.47 (Pin_47), J7.49 (Pin_49), J7.51 (Pin_51), J7.53 (Pin_53), J7.55 (Pin_55), J7.57 (Pin_57), J7.59 (Pin_59), J7.61 (Pin_61), J7.63 (Pin_63); no longer J7.34 (Pin_34), J7.36 (Pin_36), J7.38 (Pin_38), J7.40 (Pin_40), J7.42 (Pin_42), J7.44 (Pin_44), J7.46 (Pin_46), J7.48 (Pin_48), J7.50 (Pin_50), J7.52 (Pin_52), J7.54 (Pin_54), J7.56 (Pin_56), J7.58 (Pin_58), J7.60 (Pin_60), J7.62 (Pin_62), J7.64 (Pin_64)
- net at J6.1 (Pin_1): now also J7.2 (Pin_2); no longer J7.1 (Pin_1)
- net at J6.11 (Pin_11): now also J7.12 (Pin_12); no longer J7.11 (Pin_11)
- net at J6.13 (Pin_13): now also J7.14 (Pin_14); no longer J7.13 (Pin_13)
- net at J6.15 (Pin_15): now also J7.16 (Pin_16); no longer J7.15 (Pin_15)
- net at J6.17 (Pin_17): now also J7.18 (Pin_18); no longer J7.17 (Pin_17)
- net at J6.19 (Pin_19): now also J7.20 (Pin_20); no longer J7.19 (Pin_19)
- net at J6.21 (Pin_21): now also J7.22 (Pin_22); no longer J7.21 (Pin_21)
- net at J6.23 (Pin_23): now also J7.24 (Pin_24); no longer J7.23 (Pin_23)
- net at J6.25 (Pin_25): now also J7.26 (Pin_26); no longer J7.25 (Pin_25)
- net at J6.27 (Pin_27): now also J7.28 (Pin_28); no longer J7.27 (Pin_27)
- net at J6.29 (Pin_29): now also J7.30 (Pin_30); no longer J7.29 (Pin_29)
- net at J6.3 (Pin_3): now also J7.4 (Pin_4); no longer J7.3 (Pin_3)
- net at J6.31 (Pin_31): now also J7.32 (Pin_32); no longer J7.31 (Pin_31)
- net at J6.33 (Pin_33): now also J7.34 (Pin_34); no longer J7.33 (Pin_33)
- net at J6.35 (Pin_35): now also J7.36 (Pin_36); no longer J7.35 (Pin_35)
- net at J6.37 (Pin_37): now also J7.38 (Pin_38); no longer J7.37 (Pin_37)
- net at J6.39 (Pin_39): now also J7.40 (Pin_40); no longer J7.39 (Pin_39)
- net at J6.41 (Pin_41): now also J7.42 (Pin_42); no longer J7.41 (Pin_41)
- net at J6.43 (Pin_43): now also J7.44 (Pin_44); no longer J7.43 (Pin_43)
- net at J6.45 (Pin_45): now also J7.46 (Pin_46); no longer J7.45 (Pin_45)
- net at J6.47 (Pin_47): now also J7.48 (Pin_48); no longer J7.47 (Pin_47)
- net at J6.49 (Pin_49): now also J7.50 (Pin_50); no longer J7.49 (Pin_49)
- net at J6.5 (Pin_5): now also J7.6 (Pin_6); no longer J7.5 (Pin_5)
- net at J6.51 (Pin_51): now also J7.52 (Pin_52); no longer J7.51 (Pin_51)
- net at J6.53 (Pin_53): now also J7.54 (Pin_54); no longer J7.53 (Pin_53)
- net at J6.55 (Pin_55): now also J7.56 (Pin_56); no longer J7.55 (Pin_55)
- net at J6.57 (Pin_57): now also J7.58 (Pin_58); no longer J7.57 (Pin_57)
- net at J6.59 (Pin_59): now also J7.60 (Pin_60); no longer J7.59 (Pin_59)
- net at J6.61 (Pin_61): now also J7.62 (Pin_62); no longer J7.61 (Pin_61)
- net at J6.63 (Pin_63): now also J7.64 (Pin_64); no longer J7.63 (Pin_63)
- net at J6.7 (Pin_7): now also J7.8 (Pin_8); no longer J7.7 (Pin_7)
- net at J6.9 (Pin_9): now also J7.10 (Pin_10); no longer J7.9 (Pin_9)
Changed lines of the file:
@@
 Text Label 6150 6800 2    50   ~ 0
 VCC
-Text Label 7300 2750 2    50   ~ 0
-SIG2
-Wire Wire Line
-	8700 2750 8600 2750
-Connection ~ 8700 2750
-Wire Wire Line
-	8600 2750 8500 2750
-Connection ~ 8600 2750
-Wire Wire Line
-	8500 2750 8400 2750
-Connection ~ 8500 2750
-Wire Wire Line
-	8400 2750 8300 2750
-Connection ~ 8400 2750
-Wire Wire Line
-	8300 2750 8200 2750
-Connection ~ 8300 2750
-Wire Wire Line
-	8200 2750 8100 2750
-Connection ~ 8200 2750
-Wire Wire Line
-	8100 2750 8000 2750
-Connection ~ 8100 2750
-Wire Wire Line
-	8000 2750 7900 2750
-Connection ~ 8000 2750
-Wire Wire Line
-	7900 2750 7800 2750
-Connection ~ 7900 2750
-Wire Wire Line
-	7800 2750 7700 2750
-Connection ~ 7800 2750
-Wire Wire Line
-	7700 2750 7600 2750
-Connection ~ 7700 2750
-Wire Wire Line
-	7600 2750 7500 2750
-Connection ~ 7600 2750
-Wire Wire Line
-	7500 2750 7400 2750
-Connection ~ 7500 2750
-Wire Wire Line
-	7400 2750 7300 2750
-Connection ~ 7400 2750
-Wire Wire Line
-	8800 2750 8700 2750
-Wire Wire Line
-	10300 2750 10400 2750
-Connection ~ 10300 2750
-Wire Wire Line
-	10200 2750 10300 2750
-Connection ~ 10200 2750
-Wire Wire Line
-	10100 2750 10200 2750
-Connection ~ 10100 2750
-Wire Wire Line
-	10000 2750 10100 2750
-Connection ~ 10000 2750
-Wire Wire Line
-	9900 2750 10000 2750
-Connection ~ 9900 2750
-Wire Wire Line
-	9800 2750 9900 2750
-Connection ~ 9800 2750
-Wire Wire Line
-	9700 2750 9800 2750
-Connection ~ 9700 2750
-Wire Wire Line
-	9600 2750 9700 2750
-Connection ~ 9600 2750
-Wire Wire Line
-	9500 2750 9600 2750
-Connection ~ 9500 2750
-Wire Wire Line
-	9400 2750 9500 2750
-Connection ~ 9400 2750
-Wire Wire Line
-	9300 2750 9400 2750
-Connection ~ 9300 2750
-Wire Wire Line
-	9200 2750 9300 2750
-Connection ~ 9200 2750
-Wire Wire Line
-	9100 2750 9200 2750
-Connection ~ 9100 2750
-Wire Wire Line
-	9000 2750 9100 2750
-Connection ~ 9000 2750
-Wire Wire Line
-	8900 2750 9000 2750
-$Comp
-L Connector_Generic:Conn_02x32_Odd_Even J7
-U 1 1 60E62E77
-P 8900 2450
-F 0 "J7" V 8904 763 50  0000 R CNN
-F 1 "2x32_Odd_Even" V 8995 763 50  0000 R CNN
-F 2 "Connector_PinHeader_2.00mm:PinHeader_2x32_P2.00mm_Vertical_SMD" H 8900 2450 50  0001 C CNN
-F 3 "~" H 8900 2450 50  0001 C CNN
-	1    8900 2450
-	0    1    1    0
-$EndComp
-Text Label 10400 2750 0    50   ~ 0
-SIG1
 $Comp
 L Connector_Generic:Conn_02x32_Odd_Even J6
@@
 	0    1    -1   0
 $EndComp
-Wire Wire Line
-	10400 1750 10400 2250
-Wire Wire Line
-	10300 1750 10300 2250
-Wire Wire Line
-	10200 1750 10200 2250
-Wire Wire Line
-	10100 2250 10100 1750
-Wire Wire Line
-	10000 1750 10000 2250
-Wire Wire Line
-	9900 1750 9900 2250
-Wire Wire Line
-	9800 1750 9800 2250
-Wire Wire Line
-	9700 2250 9700 1750
-Wire Wire Line
-	9600 1750 9600 2250
-Wire Wire Line
-	9500 1750 9500 2250
-Wire Wire Line
-	9400 1750 9400 2250
-Wire Wire Line
-	9300 2250 9300 1750
-Wire Wire Line
-	9200 1750 9200 2250
-Wire Wire Line
-	9100 1750 9100 2250
-Wire Wire Line
-	9000 1750 9000 2250
-Wire Wire Line
-	8900 2250 8900 1750
-Wire Wire Line
-	8800 1750 8800 2250
-Wire Wire Line
-	8700 1750 8700 2250
-Wire Wire Line
-	8600 1750 8600 2250
-Wire Wire Line
-	8500 2250 8500 1750
-Wire Wire Line
-	8400 1750 8400 2250
-Wire Wire Line
-	8300 1750 8300 2250
-Wire Wire Line
-	8200 1750 8200 2250
-Wire Wire Line
-	8100 2250 8100 1750
-Wire Wire Line
-	8000 1750 8000 2250
-Wire Wire Line
-	7900 1750 7900 2250
-Wire Wire Line
-	7800 1750 7800 2250
-Wire Wire Line
-	7700 2250 7700 1750
-Wire Wire Line
-	7600 1750 7600 2250
-Wire Wire Line
-	7500 1750 7500 2250
-Wire Wire Line
-	7400 1750 7400 2250
 Wire Wire Line
 	7300 2250 7300 1750
@@
 F 0 "J5" H 6430 6892 50  0000 L CNN
 F 1 "Conn_01x04" H 6430 6801 50  0000 L CNN
-F 2 "Connector_PinHeader_2.54mm:PinHeader_1x04_P2.54mm_Vertical_SMD_Pin1Left" H 6350 6900 50  0001 C CNN
+F 2 "Connector_PinHeader_2.54mm:PinHeader_1x04_P2.54mm_Vertical" H 6350 6900 50  0001 C CNN
 F 3 "~" H 6350 6900 50  0001 C CNN
 	1    6350 6900
@@
 	1    0    0    -1
 $EndComp
+Wire Wire Line
+	7700 2250 7700 1750
+Wire Wire Line
+	10400 1750 10400 2250
+Wire Wire Line
+	10300 1750 10300 2250
+Wire Wire Line
+	7600 1750 7600 2250
+Wire Wire Line
+	10200 1750 10200 2250
+Wire Wire Line
+	10100 2250 10100 1750
+Wire Wire Line
+	10000 1750 10000 2250
+Wire Wire Line
+	9900 1750 9900 2250
+Wire Wire Line
+	9800 1750 9800 2250
+Wire Wire Line
+	9700 2250 9700 1750
+Wire Wire Line
+	9600 1750 9600 2250
+Wire Wire Line
+	9500 1750 9500 2250
+Wire Wire Line
+	9400 1750 9400 2250
+Wire Wire Line
+	9300 2250 9300 1750
+Wire Wire Line
+	7500 1750 7500 2250
+Wire Wire Line
+	9200 1750 9200 2250
+Wire Wire Line
+	9000 1750 9000 2250
+Wire Wire Line
+	8900 2250 8900 1750
+Wire Wire Line
+	8800 1750 8800 2250
+Wire Wire Line
+	8700 1750 8700 2250
+Wire Wire Line
+	8500 2250 8500 1750
+Wire Wire Line
+	8400 1750 8400 2250
+Wire Wire Line
+	8300 1750 8300 2250
+Wire Wire Line
+	7400 1750 7400 2250
+Wire Wire Line
+	8200 1750 8200 2250
+Wire Wire Line
+	8100 2250 8100 1750
+Wire Wire Line
+	8000 1750 8000 2250
+Wire Wire Line
+	7900 1750 7900 2250
+Wire Wire Line
+	7800 1750 7800 2250
+Wire Wire Line
+	8600 1750 8600 2250
+Wire Wire Line
+	9100 1750 9100 2250
+Text Label 10400 2750 0    50   ~ 0
+SIG1
+Text Label 7300 2750 2    50   ~ 0
+SIG2
+Wire Wire Line
+	8800 2750 8700 2750
+Connection ~ 8700 2750
+Wire Wire Line
+	8700 2750 8600 2750
+Wire Wire Line
+	8600 2750 8500 2750
+Connection ~ 8500 2750
+Wire Wire Line
+	8500 2750 8400 2750
+Wire Wire Line
+	8400 2750 8300 2750
+Connection ~ 8400 2750
+Connection ~ 8300 2750
+Wire Wire Line
+	8300 2750 8200 2750
+Wire Wire Line
+	8200 2750 8100 2750
+Connection ~ 8200 2750
+Connection ~ 8100 2750
+Wire Wire Line
+	8100 2750 8000 2750
+Wire Wire Line
+	8000 2750 7900 2750
+Connection ~ 8000 2750
+Connection ~ 7900 2750
+Wire Wire Line
+	7900 2750 7800 2750
+Wire Wire Line
+	7800 2750 7700 2750
+Connection ~ 7800 2750
+Connection ~ 7700 2750
+Wire Wire Line
+	7700 2750 7600 2750
+Wire Wire Line
+	7600 2750 7500 2750
+Connection ~ 7600 2750
+Connection ~ 7500 2750
+Wire Wire Line
+	7500 2750 7400 2750
+Wire Wire Line
+	7400 2750 7300 2750
+Connection ~ 7400 2750
+Wire Wire Line
+	10300 2750 10400 2750
+Connection ~ 10300 2750
+Connection ~ 10200 2750
+Wire Wire Line
+	10200 2750 10300 2750
+Wire Wire Line
+	10100 2750 10200 2750
+Connection ~ 10100 2750
+Connection ~ 10000 2750
+Wire Wire Line
+	10000 2750 10100 2750
+Wire Wire Line
+	9900 2750 10000 2750
+Connection ~ 9900 2750
+Connection ~ 9800 2750
+Wire Wire Line
+	9800 2750 9900 2750
+Wire Wire Line
+	9700 2750 9800 2750
+Connection ~ 9700 2750
+Connection ~ 9600 2750
+Wire Wire Line
+	9600 2750 9700 2750
+Wire Wire Line
+	9500 2750 9600 2750
+Connection ~ 9500 2750
+Connection ~ 9400 2750
+Wire Wire Line
+	9400 2750 9500 2750
+Wire Wire Line
+	9300 2750 9400 2750
+Connection ~ 9300 2750
+Connection ~ 9200 2750
+Wire Wire Line
+	9200 2750 9300 2750
+Wire Wire Line
+	9100 2750 9200 2750
+Wire Wire Line
+	9000 2750 9100 2750
+Wire Wire Line
+	8900 2750 9000 2750
+Connection ~ 9000 2750
+Connection ~ 8600 2750
+Connection ~ 9100 2750
+$Comp
+L Connector_Generic:Conn_02x32_Odd_Even J7
+U 1 1 60E62E77
+P 8900 2550
+F 0 "J7" V 8904 863 50  0000 R CNN
+F 1 "2x32_Odd_Even" V 8995 863 50  0000 R CNN
+F 2 "Connector_PinHeader_2.00mm:PinHeader_2x32_P2.00mm_Vertical_SMD" H 8900 2550 50  0001 C CNN
+F 3 "~" H 8900 2550 50  0001 C CNN
+	1    8900 2550
+	0    1    -1   0
+$EndComp
 $EndSCHEMATC

Commit message: 2 amp version
Parts:
- removed C1, C2, C3, C4: 100 pF, Capacitor_SMD:C_1206_3216Metric, symbol Device:C
- removed C10, C11, C12, C9: 0.1 uF, Capacitor_SMD:C_1206_3216Metric, symbol Device:C
- removed C17, C18, C19, C20: 6.8 uF, Capacitor_SMD:C_1206_3216Metric, symbol Device:CP1
- removed J1, J2: Conn_Coaxial, mod:lemo-EPB.00.250.NTN, symbol Connector:Conn_Coaxial
- removed J6: Mating_Conn, Connector_PinSocket_2.00mm:PinSocket_2x32_P2.00mm_Vertical_SMD, symbol Connector_Generic:Conn_02x32_Odd_Even
- removed J7: 2x32_Odd_Even, Connector_PinHeader_2.00mm:PinHeader_2x32_P2.00mm_Vertical_SMD, symbol Connector_Generic:Conn_02x32_Odd_Even
- removed R1, R2: 51.1, Resistor_SMD:R_1206_3216Metric, symbol Device:R
- removed R10, R9: 464, Resistor_SMD:R_1206_3216Metric, symbol Device:R
- removed R13, R14, R5, R6: 50, Resistor_SMD:R_1206_3216Metric, symbol Device:R
- removed U1, U2: THS3201, Package_SO:SO-8_3.9x4.9mm_P1.27mm, symbol amplib:THS3201
- renumbered C5 to C1, C22 to C10, C23 to C11, C24 to C12, C6 to C2, C7 to C3, C8 to C4, C13 to C5, C14 to C6, C15 to C7, C16 to C8, C21 to C9, J3 to J1, J4 to J2, J8 to J3, J9 to J4, R3 to R1, R4 to R2, R7 to R3, R8 to R4, R11 to R5, R12 to R6, R15 to R7, R16 to R8, U3 to U1, U4 to U2
Connections:
- no-connect marks 113 -> 81
Other:
- moved on the sheet: C1, C10, C11, C12, C2, C3, C4, C5, C6, C7, C8, C9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

Commit message: vcc update
Parts:
- J4: footprint Connector_PinHeader_2.00mm:PinHeader_2x32_P2.00mm_Vertical_SMD -> Connector_PinHeader_2.00mm:PinHeader_2x32_P2.00mm_Vertical
Connections:
- net -VCC: now also J5.3 (Pin_3); no longer J5.2 (Pin_2)
- net GND: now also J5.2 (Pin_2), J5.4 (Pin_4)
- no-connect marks 81 -> 79
Changed lines of the file:
@@
 Comment4 ""
 $EndDescr
-NoConn ~ 9900 4950
-NoConn ~ 9900 5050
-Text Label 9900 4850 2    50   ~ 0
+Text Label 9900 4950 2    50   ~ 0
 -VCC
 Text Label 9900 4750 2    50   ~ 0
@@
 F 0 "J4" V 8904 1063 50  0000 R CNN
 F 1 "2x32_Odd_Even" V 8995 1063 50  0000 R CNN
-F 2 "Connector_PinHeader_2.00mm:PinHeader_2x32_P2.00mm_Vertical_SMD" H 8900 2750 50  0001 C CNN
+F 2 "Connector_PinHeader_2.00mm:PinHeader_2x32_P2.00mm_Vertical" H 8900 2750 50  0001 C CNN
 F 3 "~" H 8900 2750 50  0001 C CNN
 	1    8900 2750
@@
 	1    0    0    -1
 $EndComp
+$Comp
+L power:GND #PWR0101
+U 1 1 60EF4D19
+P 9900 4850
+F 0 "#PWR0101" H 9900 4600 50  0001 C CNN
+F 1 "GND" V 9905 4722 50  0000 R CNN
+F 2 "" H 9900 4850 50  0001 C CNN
+F 3 "" H 9900 4850 50  0001 C CNN
+	1    9900 4850
+	0    1    1    0
+$EndComp
+$Comp
+L power:GND #PWR0102
+U 1 1 60EF501F
+P 9900 5050
+F 0 "#PWR0102" H 9900 4800 50  0001 C CNN
+F 1 "GND" V 9905 4922 50  0000 R CNN
+F 2 "" H 9900 5050 50  0001 C CNN
+F 3 "" H 9900 5050 50  0001 C CNN
+	1    9900 5050
+	0    1    1    0
+$EndComp
 $EndSCHEMATC

Commit message: keepout
Parts:
- R3, R4, R7, R8: value 50 -> 49.9
Changed lines of the file:
@@
 P 1700 2200
 F 0 "R3" H 1770 2246 50  0000 L CNN
-F 1 "50" H 1770 2155 50  0000 L CNN
+F 1 "49.9" H 1770 2155 50  0000 L CNN
 F 2 "Resistor_SMD:R_1206_3216Metric" V 1630 2200 50  0001 C CNN
 F 3 "~" H 1700 2200 50  0001 C CNN
@@
 P 3050 2750
 F 0 "R7" V 2843 2750 50  0000 C CNN
-F 1 "50" V 2934 2750 50  0000 C CNN
+F 1 "49.9" V 2934 2750 50  0000 C CNN
 F 2 "Resistor_SMD:R_1206_3216Metric" V 2980 2750 50  0001 C CNN
 F 3 "~" H 3050 2750 50  0001 C CNN
@@
 P 1700 3850
 F 0 "R4" H 1770 3896 50  0000 L CNN
-F 1 "50" H 1770 3805 50  0000 L CNN
+F 1 "49.9" H 1770 3805 50  0000 L CNN
 F 2 "Resistor_SMD:R_1206_3216Metric" V 1630 3850 50  0001 C CNN
 F 3 "~" H 1700 3850 50  0001 C CNN
@@
 P 3050 4400
 F 0 "R8" V 2843 4400 50  0000 C CNN
-F 1 "50" V 2934 4400 50  0000 C CNN
+F 1 "49.9" V 2934 4400 50  0000 C CNN
 F 2 "Resistor_SMD:R_1206_3216Metric" V 2980 4400 50  0001 C CNN
 F 3 "~" H 3050 4400 50  0001 C CNN
