File: hardware/onboard_amp/amp_norm.sch (KiCad schematic (older format))
At the start: 27 parts, among them J1 Conn_Coaxial, J2 Conn_Coaxial, J3 Mating_Conn, J4 2x32_Odd_Even, J5 Conn_01x04, U1 THS3201, U2 THS3201

Commit message: SMD
Parts:
- removed J4: 2x32_Odd_Even, Connector_PinHeader_2.00mm:PinHeader_2x32_P2.00mm_Vertical, symbol Connector_Generic:Conn_02x32_Odd_Even
- added J4: Conn_02x16_Odd_Even, Connector_PinHeader_2.00mm:PinHeader_2x16_P2.00mm_Vertical_SMD, symbol Connector_Generic:Conn_02x16_Odd_Even
Connections:
- net SIG3: now also J4.1 (Pin_1), J4.11 (Pin_11), J4.13 (Pin_13), J4.15 (Pin_15), J4.17 (Pin_17), J4.19 (Pin_19), J4.21 (Pin_21), J4.23 (Pin_23), J4.25 (Pin_25), J4.27 (Pin_27), J4.29 (Pin_29), J4.3 (Pin_3), J4.31 (Pin_31), J4.5 (Pin_5), J4.7 (Pin_7), J4.9 (Pin_9)
- net at J3.1 (Pin_1): now also J4.2 (Pin_2)
- net at J3.11 (Pin_11): now also J4.12 (Pin_12)
- net at J3.13 (Pin_13): now also J4.14 (Pin_14)
- net at J3.15 (Pin_15): now also J4.16 (Pin_16)
- net at J3.17 (Pin_17): now also J4.18 (Pin_18)
- net at J3.19 (Pin_19): now also J4.20 (Pin_20)
- net at J3.21 (Pin_21): now also J4.22 (Pin_22)
- net at J3.23 (Pin_23): now also J4.24 (Pin_24)
- net at J3.25 (Pin_25): now also J4.26 (Pin_26)
- net at J3.27 (Pin_27): now also J4.28 (Pin_28)
- net at J3.29 (Pin_29): now also J4.30 (Pin_30)
- net at J3.3 (Pin_3): now also J4.4 (Pin_4)
- net at J3.31 (Pin_31): now also J4.32 (Pin_32)
- net at J3.5 (Pin_5): now also J4.6 (Pin_6)
- net at J3.7 (Pin_7): now also J4.8 (Pin_8)
- net at J3.9 (Pin_9): now also J4.10 (Pin_10)
- no-connect marks 79 -> 47
Changed lines of the file:
@@
 Wire Wire Line
 	10400 2050 10400 2550
-$Comp
-L Connector_Generic:Conn_02x32_Odd_Even J4
-U 1 1 6104FD7C
-P 8900 2750
-F 0 "J4" V 8904 1063 50  0000 R CNN
-F 1 "2x32_Odd_Even" V 8995 1063 50  0000 R CNN
-F 2 "Connector_PinHeader_2.00mm:PinHeader_2x32_P2.00mm_Vertical" H 8900 2750 50  0001 C CNN
-F 3 "~" H 8900 2750 50  0001 C CNN
-	1    8900 2750
-	0    1    1    0
-$EndComp
-Wire Wire Line
-	10400 3050 10300 3050
-Connection ~ 9000 3050
-Wire Wire Line
-	9000 3050 8900 3050
-Connection ~ 9100 3050
-Wire Wire Line
-	9100 3050 9000 3050
-Connection ~ 9200 3050
-Wire Wire Line
-	9200 3050 9100 3050
-Connection ~ 9300 3050
-Wire Wire Line
-	9300 3050 9200 3050
-Connection ~ 9400 3050
-Wire Wire Line
-	9400 3050 9300 3050
-Connection ~ 9500 3050
-Wire Wire Line
-	9500 3050 9400 3050
-Connection ~ 9600 3050
-Wire Wire Line
-	9600 3050 9500 3050
-Connection ~ 9700 3050
-Wire Wire Line
-	9700 3050 9600 3050
-Connection ~ 9800 3050
-Wire Wire Line
-	9800 3050 9700 3050
-Connection ~ 9900 3050
-Wire Wire Line
-	9900 3050 9800 3050
-Connection ~ 10000 3050
-Wire Wire Line
-	10000 3050 9900 3050
-Connection ~ 10100 3050
-Wire Wire Line
-	10100 3050 10000 3050
-Connection ~ 10200 3050
-Wire Wire Line
-	10200 3050 10100 3050
-Connection ~ 10300 3050
-Wire Wire Line
-	10300 3050 10200 3050
 Text Label 10400 3050 0    50   ~ 0
 SIG3
@@
 	0    1    -1   0
 $EndComp
-NoConn ~ 8800 3050
-NoConn ~ 8700 3050
-NoConn ~ 8600 3050
-NoConn ~ 8500 3050
-NoConn ~ 8400 3050
-NoConn ~ 8300 3050
-NoConn ~ 8200 3050
-NoConn ~ 8100 3050
-NoConn ~ 8000 3050
-NoConn ~ 7900 3050
-NoConn ~ 7800 3050
-NoConn ~ 7700 3050
-NoConn ~ 7600 3050
-NoConn ~ 7500 3050
-NoConn ~ 7400 3050
-NoConn ~ 7300 3050
 NoConn ~ 7400 2050
 NoConn ~ 7500 2050
@@
 NoConn ~ 8700 2050
 NoConn ~ 8800 2050
-NoConn ~ 8800 2550
-NoConn ~ 8700 2550
-NoConn ~ 8600 2550
-NoConn ~ 8500 2550
-NoConn ~ 8400 2550
-NoConn ~ 8300 2550
-NoConn ~ 8200 2550
-NoConn ~ 8100 2550
-NoConn ~ 8000 2550
-NoConn ~ 7900 2550
-NoConn ~ 7800 2550
-NoConn ~ 7700 2550
-NoConn ~ 7600 2550
-NoConn ~ 7500 2550
-NoConn ~ 7400 2550
-NoConn ~ 7300 2550
 $Comp
 L Device:C C5
@@
 	0    1    1    0
 $EndComp
+Wire Wire Line
+	8900 3050 9000 3050
+$Comp
+L Connector_Generic:Conn_02x16_Odd_Even J4
+U 1 1 60F08B30
+P 9700 2850
+F 0 "J4" V 9704 1963 50  0000 R CNN
+F 1 "Conn_02x16_Odd_Even" V 9795 1963 50  0000 R CNN
+F 2 "Connector_PinHeader_2.00mm:PinHeader_2x16_P2.00mm_Vertical_SMD" H 9700 2850 50  0001 C CNN
+F 3 "~" H 9700 2850 50  0001 C CNN
+	1    9700 2850
+	0    1    -1   0
+$EndComp
+Connection ~ 9000 3050
+Wire Wire Line
+	9000 3050 9100 3050
+Connection ~ 9100 3050
+Wire Wire Line
+	9100 3050 9200 3050
+Connection ~ 9200 3050
+Wire Wire Line
+	9200 3050 9300 3050
+Connection ~ 9300 3050
+Wire Wire Line
+	9300 3050 9400 3050
+Connection ~ 9400 3050
+Wire Wire Line
+	9400 3050 9500 3050
+Connection ~ 9500 3050
+Wire Wire Line
+	9500 3050 9600 3050
+Connection ~ 9600 3050
+Wire Wire Line
+	9600 3050 9700 3050
+Connection ~ 9700 3050
+Wire Wire Line
+	9700 3050 9800 3050
+Connection ~ 9800 3050
+Wire Wire Line
+	9800 3050 9900 3050
+Connection ~ 9900 3050
+Wire Wire Line
+	9900 3050 10000 3050
+Connection ~ 10000 3050
+Wire Wire Line
+	10000 3050 10100 3050
+Connection ~ 10100 3050
+Wire Wire Line
+	10100 3050 10200 3050
+Connection ~ 10200 3050
+Wire Wire Line
+	10200 3050 10300 3050
+Connection ~ 10300 3050
+Wire Wire Line
+	10300 3050 10400 3050
 $EndSCHEMATC

Commit message: GND
Connections:
- net GND: now also J3.10 (Pin_10), J3.12 (Pin_12), J3.14 (Pin_14), J3.16 (Pin_16), J3.18 (Pin_18), J3.2 (Pin_2), J3.20 (Pin_20), J3.22 (Pin_22), J3.24 (Pin_24), J3.26 (Pin_26), J3.28 (Pin_28), J3.30 (Pin_30), J3.32 (Pin_32), J3.34 (Pin_34), J3.36 (Pin_36), J3.38 (Pin_38), J3.4 (Pin_4), J3.40 (Pin_40), J3.42 (Pin_42), J3.44 (Pin_44), J3.46 (Pin_46), J3.48 (Pin_48), J3.50 (Pin_50), J3.52 (Pin_52), J3.54 (Pin_54), J3.56 (Pin_56), J3.58 (Pin_58), J3.6 (Pin_6), J3.60 (Pin_60), J3.62 (Pin_62), J3.64 (Pin_64), J3.8 (Pin_8)
- no-connect marks 47 -> 15
Changed lines of the file:
@@
 	1    0    0    -1
 $EndComp
-NoConn ~ 10400 1550
-NoConn ~ 10300 1550
-NoConn ~ 10200 1550
-NoConn ~ 10100 1550
-NoConn ~ 10000 1550
-NoConn ~ 9900 1550
-NoConn ~ 9800 1550
-NoConn ~ 9700 1550
-NoConn ~ 9600 1550
-NoConn ~ 9500 1550
-NoConn ~ 9400 1550
-NoConn ~ 9300 1550
-NoConn ~ 9200 1550
-NoConn ~ 9100 1550
-NoConn ~ 9000 1550
-NoConn ~ 8900 1550
-NoConn ~ 8800 1550
-NoConn ~ 8700 1550
-NoConn ~ 8600 1550
-NoConn ~ 8500 1550
-NoConn ~ 8400 1550
-NoConn ~ 8300 1550
-NoConn ~ 8200 1550
-NoConn ~ 8100 1550
-NoConn ~ 8000 1550
-NoConn ~ 7900 1550
-NoConn ~ 7800 1550
-NoConn ~ 7700 1550
-NoConn ~ 7600 1550
-NoConn ~ 7500 1550
-NoConn ~ 7400 1550
-NoConn ~ 7300 1550
 Wire Wire Line
 	8900 2550 8900 2050
@@
 Wire Wire Line
 	10300 3050 10400 3050
+Wire Wire Line
+	10400 1550 10300 1550
+Connection ~ 7400 1550
+Wire Wire Line
+	7400 1550 7300 1550
+Connection ~ 7500 1550
+Wire Wire Line
+	7500 1550 7400 1550
+Connection ~ 7600 1550
+Wire Wire Line
+	7600 1550 7500 1550
+Connection ~ 7700 1550
+Wire Wire Line
+	7700 1550 7600 1550
+Connection ~ 7800 1550
+Wire Wire Line
+	7800 1550 7700 1550
+Connection ~ 7900 1550
+Wire Wire Line
+	7900 1550 7800 1550
+Connection ~ 8000 1550
+Wire Wire Line
+	8000 1550 7900 1550
+Connection ~ 8100 1550
+Wire Wire Line
+	8100 1550 8000 1550
+Connection ~ 8200 1550
+Wire Wire Line
+	8200 1550 8100 1550
+Connection ~ 8300 1550
+Wire Wire Line
+	8300 1550 8200 1550
+Connection ~ 8400 1550
+Wire Wire Line
+	8400 1550 8300 1550
+Connection ~ 8500 1550
+Wire Wire Line
+	8500 1550 8400 1550
+Connection ~ 8600 1550
+Wire Wire Line
+	8600 1550 8500 1550
+Connection ~ 8700 1550
+Wire Wire Line
+	8700 1550 8600 1550
+Connection ~ 8800 1550
+Wire Wire Line
+	8800 1550 8700 1550
+Connection ~ 8900 1550
+Wire Wire Line
+	8900 1550 8800 1550
+Connection ~ 9000 1550
+Wire Wire Line
+	9000 1550 8900 1550
+Connection ~ 9100 1550
+Wire Wire Line
+	9100 1550 9000 1550
+Connection ~ 9200 1550
+Wire Wire Line
+	9200 1550 9100 1550
+Connection ~ 9300 1550
+Wire Wire Line
+	9300 1550 9200 1550
+Connection ~ 9400 1550
+Wire Wire Line
+	9400 1550 9300 1550
+Connection ~ 9500 1550
+Wire Wire Line
+	9500 1550 9400 1550
+Connection ~ 9600 1550
+Wire Wire Line
+	9600 1550 9500 1550
+Connection ~ 9700 1550
+Wire Wire Line
+	9700 1550 9600 1550
+Connection ~ 9800 1550
+Wire Wire Line
+	9800 1550 9700 1550
+Connection ~ 9900 1550
+Wire Wire Line
+	9900 1550 9800 1550
+Connection ~ 10000 1550
+Wire Wire Line
+	10000 1550 9900 1550
+Connection ~ 10100 1550
+Wire Wire Line
+	10100 1550 10000 1550
+Connection ~ 10200 1550
+Wire Wire Line
+	10200 1550 10100 1550
+Connection ~ 10300 1550
+Wire Wire Line
+	10300 1550 10200 1550
+$Comp
+L power:GND #PWR0103
+U 1 1 60F3435A
+P 10400 1550
+F 0 "#PWR0103" H 10400 1300 50  0001 C CNN
+F 1 "GND" V 10405 1422 50  0000 R CNN
+F 2 "" H 10400 1550 50  0001 C CNN
+F 3 "" H 10400 1550 50  0001 C CNN
+	1    10400 1550
+	0    -1   -1   0
+$EndComp
+Connection ~ 10400 1550
 $EndSCHEMATC
