File: hardware/readout/96Chan.sch (KiCad schematic (older format))
At the start: 0 parts

Commit message: working on final schem
Changed lines of the file:
@@
 F3 "SIPM[0..31]" I L 4000 1600 50
 F4 "CCTL[0..7]" I L 4000 1750 50
+F5 "D_PROBE" O R 5150 2100 50
+F6 "A_PROBE" O R 5150 1900 50
 $EndSheet
 $Sheet
@@
 F3 "SIPM[0..31]" I L 4000 2950 50
 F4 "CCTL[0..7]" I L 4000 3100 50
+F5 "D_PROBE" O R 5150 3450 50
+F6 "A_PROBE" O R 5150 3250 50
 $EndSheet
 $Sheet
@@
 F3 "SIPM[0..31]" I L 4000 4300 50
 F4 "CCTL[0..7]" I L 4000 4450 50
+F5 "D_PROBE" O R 5150 4850 50
+F6 "A_PROBE" O R 5150 4650 50
 $EndSheet
 Wire Bus Line
