File: hardware/readout/bias.sch (KiCad schematic (older format))
At the start: 0 parts

Commit message: schematic update
Parts:
- added C? (x2): 0.1 uF, Capacitor_SMD:C_1206_3216Metric, symbol Device:C
- added D? (x2): LED, LED_THT:LED_D4.0mm, symbol Device:LED
- added JP? (x3): Jumper, Connector_PinHeader_2.54mm:PinHeader_1x02_P2.54mm_Vertical, symbol Device:Jumper
- added R? (x2): 150, Resistor_SMD:R_1206_3216Metric, symbol Device:R_US
- added R? (x2): 10K, Resistor_SMD:R_1206_3216Metric, symbol Device:R_US
- added R? (x2): 4.7k, symbol Device:R_US
- added SW?: SW_SPDT, A7585-test-board:SW_DIP_SPSTx01_Slide_9.78x4.72mm_W7.62mm_P2.54mm, symbol Switch:SW_SPDT
- added U?: A7585D, A7585-test-board:A7585D_Board, symbol A7585-test-board_Library:A7585D
Connections:
- net labels added: +1V8, +3.3V, GND, I2C_SCL, I2C_SDA, UART_RX_5V, UART_TX_5V, VCC, VSS
- wire segments 1 -> 54
Other:
- note added: "1: HV output is enabled\n0: HV output is disabled\n"
- note added: "I/V monitor 0-5V"
- note added: "I2C address 1111xx\nJumper in = 1\nIdentified at power on"
- note added: "Use either I2C (1.8V)\nOr UART (5V)"
- note added: "VDD is 1.8V to 5V for I2C\n"
- note added: "VSS is 6V to 28V"
- note removed: "SiPM Bias voltage generator\n"

Commit message: working on schematic
Parts:
- removed JP? (x2): Jumper, Connector_PinHeader_2.54mm:PinHeader_1x02_P2.54mm_Vertical, symbol Device:Jumper
- added C1063, C1067, C1069, C1070, C1072, C1073, C1074: 0.1uF, symbol Device:C_Small
- added C1066, C1068: 10uF, symbol Device:C_Small
- added C1071: 1uF, symbol Device:C_Small
- added R607, R608, R609, R610, R612, R613, R614, R615: DNP, symbol Device:R_Small_US
- added R611: 0R, symbol Device:R_Small_US
- added R616, R617, R618, R619, R620, R621, R624: 10k, symbol Device:R_Small_US
- added U44, U45: 74AXP1T34, symbol readout:74AXP1T34
- added U46: AD7291, Package_CSP:LFCSP-20-1EP_4x4mm_P0.5mm_EP2.6x2.6mm_ThermalVias, symbol readout:AD7291
- C1064, C1065: renamed from C?; footprint Capacitor_SMD:C_1206_3216Metric -> (none)
- D2, D3: renamed from D?; footprint LED_THT:LED_D4.0mm -> (none)
- R603, R604, R605, R606: renamed from R?; footprint Resistor_SMD:R_1206_3216Metric -> (none)
- gave numbers to parts that had none: 5
Connections:
- net labels added: +5V, T0, T1, T2, T3, T4, T5, T6, T7, T8, T[0..8], UART_RX, UART_TX
- net labels removed: UART_RX_5V, UART_TX_5V, VCC
- wire segments 54 -> 151
- no-connect marks 0 -> 5
Other:
- note added: "Monitor temp sensor\nwith ADC channel 2"
- note added: "Spare ADC inputs\n(GND if unused)\n"
- note added: "Temperature sensor input\nInstall only one resistor\nto select SiPM board\n\nDefault = middle board"
- note removed: "I2C address 1111xx\nJumper in = 1\nIdentified at power on"
- note removed: "Use either I2C (1.8V)\nOr UART (5V)"
