File: hardware/readout/readout96.sch (KiCad schematic (older format))
At the start: 3 parts

Commit message: schematic in progress
Connections:
- net labels added: CTRL[0..3]
Other:
- note added: "EMPHATIC readout board\n96 channel readout group -- 1 of 6"
Changed lines of the file:
@@
 $Descr A4 11693 8268
 encoding utf-8
-Sheet 8 35
+Sheet 8 38
 Title ""
 Date ""
@@
 F6 "MGT_TX_N[0..3]" O R 9150 4050 50
 F7 "GPIO[0..15]" O L 7750 4550 50
+F8 "CTRL[0..3]" O R 9150 4550 50
 $EndSheet
 Text Label 7650 3950 2    50   ~ 0
@@
 	5500 4300 5500 5400
 Connection ~ 5500 4300
-Wire Bus Line
-	9750 2800 9750 3950
-Wire Bus Line
-	9950 2900 9950 4050
-Wire Bus Line
-	5500 2450 5500 4300
-Wire Bus Line
-	2900 2300 2900 5400
-Wire Bus Line
-	6800 2900 6800 4050
-Wire Bus Line
-	7000 2800 7000 3950
 Text Notes 4700 1800 2    75   ~ 0
 3x CITIROC ASIC\n32 Channels each
 Text Notes 8800 1900 2    75   ~ 0
 Trenz TE0714\nFPGA Module
+Wire Bus Line
+	9150 4550 9950 4550
+Text HLabel 9950 4550 2    50   BiDi ~ 0
+CTRL[0..3]
+Wire Bus Line
+	9750 2800 9750 3950
+Wire Bus Line
+	9950 2900 9950 4050
+Wire Bus Line
+	5500 2450 5500 4300
+Wire Bus Line
+	6800 2900 6800 4050
+Wire Bus Line
+	7000 2800 7000 3950
+Wire Bus Line
+	2900 2300 2900 5400
+Text Notes 7100 6800 0    75   ~ 0
+EMPHATIC readout board\n96 channel readout group -- 1 of 6
 $EndSCHEMATC

Commit message: working on schematic
Parts:
- added C175, C176, C177, C178, C179, C180: 0.1uF, symbol Device:C_Small
- added U7: FXL4245, symbol readout:FXL4245
- added U8, U9: NLSV4T244MU, symbol readout:NLSV4T244MU
- gave numbers to parts that had none: 3
Connections:
- net labels added: +1V8, +3.3V, CTL0, CTL1, CTL2, CTL3, CTL[0..3], CTRL[0..11], GND, GPIO0, GPIO1, GPIO2, GPIO3
- net labels removed: CTRL[0..3], GPIO[0..3]
- wire segments 26 -> 97
Other:
- note added: "CTRL exported to\nsheet above"
- note added: "GPIO used on this sheet only"
