File: hardware/examples/LED_Pulser/_autosave-LED_Pulser.sch (KiCad schematic (older format))
At the start: 64 parts, among them J1 Conn_Coaxial, J10 Conn_01x01, J11 Conn_01x01, J12 Conn_01x01, J13 Conn_01x01, J14 Conn_01x01, J15 Conn_01x01, J16 Conn_01x01, J17 Conn_01x01, J18 Conn_01x01, J19 Conn_01x01, J2 Conn_01x01, J20 Conn_01x01, J21 Conn_01x01, J22 Conn_01x01, J23 Conn_01x01, J24 Conn_01x01, J25 Conn_01x01, J26 Conn_01x01, J27 Conn_01x01, J28 Conn_01x01, J29 Conn_01x01, J3 Conn_01x01, J30 Conn_01x01, J31 Conn_01x01, J32 Conn_01x01, J33 Conn_01x01, J34 Conn_01x01, J35 Conn_01x01, J36 Conn_01x01, J37 Conn_01x01, J38 Conn_01x01, J39 Conn_01x01, J4 Conn_01x01, J40 Conn_01x01, J41 Conn_01x01, J42 Conn_Coaxial_Power, J5 Conn_01x01, J6 Conn_01x01, J7 Conn_01x01, J8 Conn_01x01, J9 Conn_01x01, Q1 2N3904, U1 LM385Z-2.5, U2 TLV2371P, U3 74LVCH2T45DC, U4 Raspberry_pi_pico

Commit message: LED Pulser V2.1
Parts:
- RV1: symbol Device:R_POT_US -> LED_Pulser-rescue:R_POT_US-Device
